File: usb_fsls.kicad_sch (KiCad schematic)
At the start: 15 parts, among them J2 USB_C_Receptacle_USB2.0, U13 STUSB03E, U8 T8Q144xx

Commit message: Fixed V1.0 errata
- added feedback resistor for ulpi transceiver clock oscillator
- removed SS_N connection
Parts:
- renumbered C14 to C46, C17 to C47, C23 to C55, C13 to C56, C14 to C58, R3 to R38, R3 to R39, R9 to R51
