File: trion-8-test.kicad_pcb (KiCad board)
At the start: 4 copper layers, 39.5 x 80 mm, 186 parts, among them J1 USB_C_Receptacle_USB2.0, J2 FT_JTAG, J3 T8_JTAG, J4 USB_C_Receptacle_USB2.0, J5 USB_C_Receptacle_USB2.0, Q1 SSM3K37MFV, SW1 Reset, U1 FXL5T244, U10 USB3343, U12 RT8096B, U13 STUSB03E, U2 FT2232HL, U3 93LCxxAxxOT, U4 TLV75801PDBV, U5 TSX339IPT, U6 RT8096B, U7 2N7001T, U8 T8Q144xx, U9 AT25SF081-SSHD-X, X1 ECS-2520MV-120-CM, X2 ECS-2520MV-120-CM, Y1 26MHz

Commit message: Fixed V1.0 errata
- added feedback resistor for ulpi transceiver clock oscillator
- removed SS_N connection
Parts:
- added R73: 1M, Resistor_SMD:R_0603_1608Metric, F.Cu at (61.4, 95.9)
- R19: value 27k4 -> 27k
- U9: value AT25SF081-SSHD-X -> AT25FF081A-SSHN-B
- moved C52 1.45 mm to (59.9, 95.9)
- moved C47 1.03 mm to (60.1, 98.4), turned to 0 degrees
Connections:
- U1 pad 9: /FT-USB-JTAG/SS_N -> unconnected-(U1-B4-Pad9)
Routing:
- net /FT-USB-JTAG/SS_N: track 13.8 -> 0.00 mm
- net GND: track 250.9 -> 254.4 mm, vias 173 -> 174
- net Net-(U10-REFCLK/XI): track 5.37 -> 8.11 mm
- net Net-(U10-XO): track 3.50 -> 4.95 mm

Commit message: sdram layout done - COMPLETE REWORK NEEDED
cannot mix LVDS and GPIO banks due to too different timing
Parts:
- removed C11, C14, C16, C19, C20, C24, C25, C26, C46, C58: 100n, Capacitor_SMD:C_0603_1608Metric
- removed C15, C18, C56: 4u7, Capacitor_SMD:C_0805_2012Metric
- removed C17, C47: 10n, Capacitor_SMD:C_0603_1608Metric
- removed C23, C55: 1u, Capacitor_SMD:C_0805_2012Metric
- removed J1, J5: USB_C_Receptacle_USB2.0, proj_footprints:USB_C_Receptacle_Molex_2171790001_16P_TopMnt_Horizontal
- removed J2: FT_JTAG, Connector_PinHeader_2.00mm:PinHeader_2x07_P2.00mm_Vertical
- removed L2: 600Ohm@100MHz, Inductor_SMD:L_0603_1608Metric
- removed R1, R14, R15, R17, R2, R3, R38, R39, R55: 10k, Resistor_SMD:R_0603_1608Metric
- removed R10: 45k3, Resistor_SMD:R_0603_1608Metric
- removed R11, R18: 20k0, Resistor_SMD:R_0603_1608Metric
- removed R12: 35k7, Resistor_SMD:R_0603_1608Metric
- removed R13: 30k9, Resistor_SMD:R_0603_1608Metric
- removed R16: 8k06, Resistor_SMD:R_0603_1608Metric
- removed R19: 27k, Resistor_SMD:R_0603_1608Metric
- removed R20: 100k, Resistor_SMD:R_0603_1608Metric
- removed R21, R25, R26, R27, R28, R29, R51, R9: 1M, Resistor_SMD:R_0603_1608Metric
- removed R4: 2k, Resistor_SMD:R_0603_1608Metric
- removed R5: 1k, Resistor_SMD:R_0603_1608Metric
- removed R52, R53, R7, R8: 5k1, Resistor_SMD:R_0603_1608Metric
- removed R54: 1k5, Resistor_SMD:R_0603_1608Metric
- removed R6: 12k, Resistor_SMD:R_0603_1608Metric
- removed U13: STUSB03E, Package_DFN_QFN:TQFN-16-1EP_3x3mm_P0.5mm_EP1.6x1.6mm
- removed U2: FT2232HL, Package_QFP:LQFP-64_10x10mm_P0.5mm
- removed U3: 93LCxxAxxOT, Package_TO_SOT_SMD:SOT-23-6
- removed U4: TLV75801PDBV, Package_TO_SOT_SMD:SOT-23-5
- removed U5: TSX339IPT, Package_SO:TSSOP-14_4.4x5mm_P0.65mm
- removed U7: 2N7001T, Package_TO_SOT_SMD:SOT-353_SC-70-5
- removed X1: ECS-2520MV-120-CM, Oscillator:Oscillator_SMD_ECS_2520MV-xxx-xx-4Pin_2.5x2.0mm
- C1, C12, C2, C4, C9: moved to B.Cu
- C10: value 100n -> 4u7; footprint Capacitor_SMD:C_0603_1608Metric -> Capacitor_SMD:C_0805_2012Metric
- C13: value 4u7 -> 100n; footprint Capacitor_SMD:C_0805_2012Metric -> Capacitor_SMD:C_0603_1608Metric
- C35, C36, C6, C8, R30: moved to F.Cu
- U1: value FXL5T244 -> MT48LC16M16A2P; footprint Package_DFN_QFN:DHVQFN-14-1EP_2.5x3mm_P0.5mm_EP1x1.5mm -> Package_SO:TSOP-II-54_22.2x10.16mm_P0.8mm; moved to B.Cu
- moved C4 48.6 mm to (101.1, 99.5), turned to 90 degrees
- moved C6 47.8 mm to (95.9, 91.5), turned to 0 degrees
- moved C7 43.1 mm to (85.4, 88.3)
- moved H3 41.3 mm to (62.7, 105.7)
- moved C2 40.4 mm to (101.1, 106.3)
- moved C10 39.9 mm to (85.8, 96.2), turned to 90 degrees
- moved U1 39.0 mm to (93.6, 98.7), turned to 0 degrees
- moved L1 38.2 mm to (97.7, 111.1), turned to 180 degrees
- moved C5 36.6 mm to (86.1, 101.8)
- moved C8 36.0 mm to (96.0, 96.7), turned to 0 degrees
- moved C3 35.1 mm to (65.9, 101.7), turned to -90 degrees
- moved C13 32.1 mm to (85.4, 98.7), turned to 180 degrees
- moved X2 31.1 mm to (68.3, 101.6), turned to 90 degrees
- moved H2 29.3 mm to (96.5, 118.2)
- moved C12 23.0 mm to (88.6, 110.9)
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Connections:
- C1 pad 1: +3V3 -> Net-(C1-Pad1)
- C10 pad 1: GND -> +3V3
- C10 pad 2: Net-(U2-VREGOUT) -> GND
- C12 pad 1: GND -> +3V3
- C12 pad 2: Net-(U2-VREGOUT) -> GND
- C13 pad 1: Net-(U2-VPHY) -> +3V3
- C2 pad 1: +3V3 -> Net-(C1-Pad1)
- C4 pad 1: Net-(U2-~{RESET}) -> Net-(C1-Pad1)
- C48 pad 1: Net-(U10-VBAT) -> +5V
- C5 pad 1: +3V3 -> Net-(C1-Pad1)
- C9 pad 1: Net-(U2-VREGOUT) -> Net-(C1-Pad1)
- J4 pad A4: Net-(U10-VBAT) -> +5V
- J4 pad A9: Net-(U10-VBAT) -> +5V
- J4 pad B4: Net-(U10-VBAT) -> +5V
- J4 pad B9: Net-(U10-VBAT) -> +5V
- L1 pad 1: +3V3 -> Net-(C1-Pad1)
- L1 pad 2: Net-(U2-VPLL) -> +3V3
- R22 pad 2: Net-(U8H-GPIOR_149_CBUS2) -> /sdram/CSb
- R23 pad 2: Net-(U8H-GPIOR_150_CBUS1) -> /sdram/RASb
- R30 pad 2: Net-(U8H-GPIOR_158_TEST_N) -> /sdram/A8
- R46 pad 1: Net-(U10-VBAT) -> +5V
- U1 pad 10: /FT-USB-JTAG/CRESET_N -> /sdram/DQ5
- U1 pad 11: /FT-USB-JTAG/TCK -> /sdram/DQ6
- U1 pad 12: /FT-USB-JTAG/TDI -> GND
- U1 pad 13: /FT-USB-JTAG/TMS -> /sdram/DQ7
- U1 pad 14: VS -> +3V3
- U1 pad 15: unconnected-(U1-PAD-Pad15) -> /sdram/DQML
- U1 pad 2: /FT-USB-JTAG/FT_TMS -> /sdram/DQ0
- U1 pad 3: /FT-USB-JTAG/FT_TDI -> Net-(C1-Pad1)
- U1 pad 4: /FT-USB-JTAG/FT_TCK -> /sdram/DQ1
- U1 pad 5: /FT-USB-JTAG/FT_CRESET_N -> /sdram/DQ2
- U1 pad 6: /FT-USB-JTAG/FT_SS_N -> GND
- U1 pad 7: GND -> /sdram/DQ3
- U1 pad 8: GND -> /sdram/DQ4
- U1 pad 9: unconnected-(U1-B4-Pad9) -> Net-(C1-Pad1)
- U10 pad 16: Net-(U10-VBAT) -> +5V
- U8 pad 100: /LED/LED0 -> /LED/LED5
- U8 pad 101: unconnected-(U8F-GPIOR_112_CDI23-Pad101) -> /LED/LED4
- U8 pad 102: unconnected-(U8F-GPIOR_105_CDI24-Pad102) -> /LED/LED3
- U8 pad 103: unconnected-(U8F-GPIOR_104_CDI25-Pad103) -> /LED/LED2
- U8 pad 105: unconnected-(U8F-GPIOR_95_CDI26-Pad105) -> /LED/LED1
- U8 pad 106: unconnected-(U8F-GPIOR_94_CDI27-Pad106) -> /LED/LED0
- U8 pad 132: unconnected-(U8D-GPIOL_74_PLLIN0-Pad132) -> Net-(U8D-GPIOL_74_PLLIN0)
- U8 pad 135: /usb_fsls/FSLS_OEb -> unconnected-(U8D-GPIOL_72_EXTFB0_CDI14-Pad135)
- U8 pad 136: /usb_fsls/FSLS_RSEL -> unconnected-(U8D-GPIOL_71_NSTATUS-Pad136)
- U8 pad 137: /usb_fsls/FSLS_SUS -> unconnected-(U8D-GPIOL_70_CBSEL0-Pad137)
- U8 pad 138: /usb_fsls/FSLS_CON -> unconnected-(U8D-GPIOL_69_CBSEL1-Pad138)
- U8 pad 139: /usb_fsls/FSLS_VM -> unconnected-(U8D-GPIOL_68-Pad139)
- U8 pad 140: /usb_fsls/FSLS_VP -> unconnected-(U8D-GPIOL_67_CDI13-Pad140)
- U8 pad 141: /usb_fsls/FSLS_RCV -> unconnected-(U8D-GPIOL_65-Pad141)
- U8 pad 142: /usb_fsls/FSLS_SPD -> unconnected-(U8D-GPIOL_66_CDI12-Pad142)
- U8 pad 144: /usb_fsls/FSLS_VBUSDET -> unconnected-(U8D-GPIOL_64-Pad144)
- U8 pad 38: unconnected-(U8J-GPIOB_TXP00-Pad38) -> /sdram/DQ0
- U8 pad 39: unconnected-(U8J-GPIOB_TXN00-Pad39) -> /sdram/DQ15
- U8 pad 40: unconnected-(U8J-GPIOB_TXP02-Pad40) -> /sdram/DQ1
- U8 pad 41: unconnected-(U8J-GPIOB_TXN02-Pad41) -> /sdram/DQ14
- U8 pad 42: unconnected-(U8J-GPIOB_TXP04-Pad42) -> /sdram/DQ2
- U8 pad 43: unconnected-(U8J-GPIOB_TXN04-Pad43) -> /sdram/DQ13
- U8 pad 45: unconnected-(U8J-GPIOB_TXP06-Pad45) -> /sdram/DQ3
- U8 pad 46: unconnected-(U8J-GPIOB_TXN06-Pad46) -> /sdram/DQ12
- U8 pad 47: unconnected-(U8J-GPIOB_TXP09-Pad47) -> /sdram/DQ4
- U8 pad 48: unconnected-(U8J-GPIOB_TXN09-Pad48) -> /sdram/DQ5
- U8 pad 53: unconnected-(U8J-GPIOB_TXP11-Pad53) -> /sdram/DQ11
- U8 pad 54: unconnected-(U8J-GPIOB_TXN11-Pad54) -> /sdram/DQ10
- U8 pad 55: unconnected-(U8I-GPIOB_RXP00-Pad55) -> /sdram/DQ9
- U8 pad 56: unconnected-(U8I-GPIOB_RXN00-Pad56) -> /sdram/DQ6
- U8 pad 58: unconnected-(U8I-GPIOB_RXP02-Pad58) -> /sdram/DQ8
- U8 pad 59: unconnected-(U8I-GPIOB_RXN02-Pad59) -> /sdram/DQMH
- U8 pad 60: unconnected-(U8I-GPIOB_RXN03-Pad60) -> /sdram/CLK
- U8 pad 61: unconnected-(U8I-GPIOB_RXP03-Pad61) -> /sdram/DQ7
- U8 pad 65: unconnected-(U8I-GPIOB_RXN07-Pad65) -> /sdram/DQML
- U8 pad 66: unconnected-(U8I-GPIOB_RXP07-Pad66) -> /sdram/WEb
- U8 pad 67: unconnected-(U8I-GPIOB_RXP10-Pad67) -> /sdram/CASb
- U8 pad 68: unconnected-(U8I-GPIOB_RXN10-Pad68) -> /sdram/CKE
- U8 pad 69: unconnected-(U8I-GPIOB_RXN12_EXTFB0-Pad69) -> /sdram/A12
- U8 pad 70: unconnected-(U8I-GPIOB_RXP12_EXTFB0-Pad70) -> /sdram/A11
- U8 pad 71: unconnected-(U8I-GPIOB_CLKP0-Pad71) -> /sdram/A9
- U8 pad 72: unconnected-(U8I-GPIOB_CLKN0-Pad72) -> /sdram/A7
- U8 pad 74: Net-(U8H-GPIOR_158_TEST_N) -> /sdram/A8
- U8 pad 75: Net-(U8H-GPIOR_157_PLLIN) -> /sdram/A6
- U8 pad 76: /bank_1a_cfg/GPIOR_155 -> /sdram/A4
- U8 pad 77: unconnected-(U8H-GPIOR_154-Pad77) -> /sdram/A5
- U8 pad 79: Net-(U8H-GPIOR_150_CBUS1) -> /sdram/RASb
- U8 pad 80: Net-(U8H-GPIOR_149_CBUS2) -> /sdram/CSb
- U8 pad 81: unconnected-(U8G-GPIOR_139-Pad81) -> /sdram/BA0
- U8 pad 82: /LED/LED7 -> /sdram/A3
- U8 pad 83: /LED/LED6 -> /sdram/A2
- U8 pad 84: /LED/LED5 -> /sdram/A1
- U8 pad 86: unconnected-(U8G-GPIOR_133_CDI18-Pad86) -> /sdram/A0
- U8 pad 87: /LED/LED4 -> /sdram/A10
- U8 pad 89: unconnected-(U8G-GPIOR_129_CTRL10-Pad89) -> /sdram/BA1
- U8 pad 90: /LED/LED3 -> unconnected-(U8G-GPIOR_128_CTRL11-Pad90)
- U8 pad 92: /LED/LED2 -> unconnected-(U8G-GPIOR_125_CLK10-Pad92)
- U8 pad 98: unconnected-(U8F-GPIOR_117_CTRL14-Pad98) -> /LED/LED7
- U8 pad 99: /LED/LED1 -> /LED/LED6
- X2 pad 3: Net-(U8H-GPIOR_157_PLLIN) -> Net-(U8D-GPIOL_74_PLLIN0)
Routing:
- net GND: track 254.4 -> 183.4 mm, vias 174 -> 148
- net Net-(C1-Pad1): track 0.00 -> 51.0 mm, vias 0 -> 4
- net Net-(U2-VREGOUT): track 37.0 -> 0.00 mm, vias 2 -> 0
- net VS: track 35.5 -> 0.00 mm, vias 4 -> 0
- net /FT-USB-JTAG/JTAG_VREF: track 31.4 -> 0.00 mm
- net Net-(U10-VBAT): track 27.8 -> 0.00 mm, vias 4 -> 0
- net Net-(J1-SHIELD): track 22.8 -> 0.00 mm
- net +5V: track 76.2 -> 98.6 mm, vias 7 -> 13
- net Net-(J5-SHIELD): track 20.8 -> 0.00 mm
- net Net-(U13-VBUS): track 18.7 -> 0.00 mm
- net Net-(J3-Pin_7): track 35.2 -> 16.6 mm
- net Net-(J3-Pin_11): track 33.4 -> 15.3 mm
- net Net-(J3-Pin_9): track 31.2 -> 14.7 mm
- net /sdram/A8: track 0.00 -> 16.1 mm, vias 0 -> 1
- net /FT-USB-JTAG/FT_CRESET_N: track 15.6 -> 0.00 mm, vias 1 -> 0
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Other:
- board size 39.5 x 80 mm -> 46 x 51.5 mm
- board text added: "RSTb"
- board text added: "SSb"
- board text added: "Trion-SDRAM-Test V1.0"
- board text removed: "CRESET_N"
- board text removed: "SS_N"
- board text removed: "Trion-Test V1.0"

Commit message: layout finished; passed all checks...
Parts:
- added C11: 100n, Capacitor_SMD:C_0603_1608Metric, F.Cu at (78.4, 108.1)
- added C14: 100n, Capacitor_SMD:C_0603_1608Metric, F.Cu at (82.1, 108.0)
- added C15: 100n, Capacitor_SMD:C_0603_1608Metric, B.Cu at (69.3, 103.0)
- added R1: 10k, Resistor_SMD:R_0603_1608Metric, F.Cu at (75.7, 109.7)
- C10, C13, C39, C40, C41, C42, C57, C59, C68, C7, C70: moved to F.Cu
- C35, C36, C6, C8, L1: moved to B.Cu
- moved C3 36.4 mm to (96.6, 82.1), turned to 90 degrees
- moved C9 34.3 mm to (66.0, 97.8), turned to 90 degrees
- moved L1 33.0 mm to (66.2, 101.1), turned to -90 degrees
- moved X2 32.6 mm to (94.3, 81.9), turned to 180 degrees
- moved C2 25.4 mm to (83.6, 88.0), turned to 180 degrees
- moved C4 24.8 mm to (79.2, 87.9), turned to 180 degrees
- moved C68 23.0 mm to (67.3, 109.6), turned to 180 degrees
- moved C10 22.0 mm to (65.2, 103.8), turned to 180 degrees
- moved C13 17.8 mm to (69.0, 105.6)
- moved C71 17.4 mm to (77.5, 83.7)
- moved C64 16.6 mm to (90.5, 100.7), turned to 90 degrees
- moved U1 15.6 mm to (78.4, 95.4), turned to 90 degrees
- moved C72 15.2 mm to (80.1, 111.3), turned to 180 degrees
- moved C69 14.9 mm to (76.7, 109.2), turned to -90 degrees
- moved C67 14.8 mm to (90.3, 104.1), turned to 180 degrees
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Connections:
- D2 pad 1: /LED/LED0 -> LED0
- D3 pad 1: /LED/LED1 -> LED1
- D4 pad 1: /LED/LED2 -> LED2
- D5 pad 1: /LED/LED3 -> LED3
- D6 pad 1: /LED/LED4 -> LED4
- D7 pad 1: /LED/LED5 -> LED5
- D8 pad 1: /LED/LED6 -> LED6
- D9 pad 1: /LED/LED7 -> LED7
- R22 pad 2: /sdram/CSb -> LED4
- R23 pad 2: /sdram/RASb -> LED5
- R24 pad 2: Net-(U8H-GPIOR_151_CBUS0) -> LED6
- R30 pad 2: /sdram/A8 -> LED7
- R49 pad 1: /ulpi/ULPI_RSTb -> ULPI_RSTb
- U1 pad 2: /sdram/DQ0 -> SDRAM_DQ0
- U1 pad 29: /sdram/A4 -> SDRAM_A4
- U1 pad 30: /sdram/A5 -> SDRAM_A5
- U10 pad 24: /ulpi/ULPI_STP -> ULPI_STP
- U8 pad 10: unconnected-(U8C-GPIOL_32_CTRL4_CDI7-Pad10) -> /sdram/WEb
- U8 pad 100: /LED/LED5 -> /sdram/A12
- U8 pad 101: /LED/LED4 -> /sdram/A11
- U8 pad 102: /LED/LED3 -> /sdram/A9
- U8 pad 103: /LED/LED2 -> /sdram/A8
- U8 pad 105: /LED/LED1 -> /sdram/A7
- U8 pad 106: /LED/LED0 -> /sdram/A6
- U8 pad 109: unconnected-(U8E-GPIOR_88_CDI28-Pad109) -> SDRAM_A5
- U8 pad 11: unconnected-(U8C-GPIOL_31_CLK7_CDI6-Pad11) -> /sdram/DQML
- U8 pad 110: unconnected-(U8E-GPIOR_87_CDI29-Pad110) -> SDRAM_A4
- U8 pad 131: /ulpi/ULPI_STP -> /sdram/A10
- U8 pad 132: Net-(U8D-GPIOL_74_PLLIN0) -> ULPI_STP
- U8 pad 134: /ulpi/ULPI_RSTb -> /sdram/A1
- U8 pad 135: unconnected-(U8D-GPIOL_72_EXTFB0_CDI14-Pad135) -> /sdram/A2
- U8 pad 136: unconnected-(U8D-GPIOL_71_NSTATUS-Pad136) -> /sdram/A3
- U8 pad 137: unconnected-(U8D-GPIOL_70_CBSEL0-Pad137) -> /sdram/A0
- U8 pad 138: unconnected-(U8D-GPIOL_69_CBSEL1-Pad138) -> ULPI_RSTb
- U8 pad 14: unconnected-(U8B-GPIOL_25_CLK1-Pad14) -> /sdram/DQ7
- U8 pad 15: unconnected-(U8B-GPIOL_24_CLK0-Pad15) -> /sdram/DQ6
- U8 pad 16: unconnected-(U8B-GPIOL_22_CTRL2-Pad16) -> /sdram/DQ5
- U8 pad 17: unconnected-(U8B-GPIOL_21_CTRL1_CDI5-Pad17) -> /sdram/DQ4
- U8 pad 18: unconnected-(U8B-GPIOL_20_CTRL0_CDI4-Pad18) -> /sdram/DQ3
- U8 pad 19: unconnected-(U8B-GPIOL_13_CDI3-Pad19) -> /sdram/DQ2
- U8 pad 20: unconnected-(U8B-GPIOL_12_CDI2-Pad20) -> /sdram/DQ1
- U8 pad 3: unconnected-(U8C-GPIOL_53_CDI10-Pad3) -> /sdram/BA1
- U8 pad 33: unconnected-(U8A-GPIOL_05_CSO-Pad33) -> SDRAM_DQ0
- U8 pad 38: /sdram/DQ0 -> unconnected-(U8J-GPIOB_TXP00-Pad38)
- U8 pad 39: /sdram/DQ15 -> unconnected-(U8J-GPIOB_TXN00-Pad39)
- U8 pad 4: unconnected-(U8C-GPIOL_54_CDI11-Pad4) -> /sdram/BA0
- U8 pad 40: /sdram/DQ1 -> unconnected-(U8J-GPIOB_TXP02-Pad40)
- U8 pad 41: /sdram/DQ14 -> unconnected-(U8J-GPIOB_TXN02-Pad41)
- U8 pad 42: /sdram/DQ2 -> unconnected-(U8J-GPIOB_TXP04-Pad42)
- U8 pad 43: /sdram/DQ13 -> unconnected-(U8J-GPIOB_TXN04-Pad43)
- U8 pad 45: /sdram/DQ3 -> unconnected-(U8J-GPIOB_TXP06-Pad45)
- U8 pad 46: /sdram/DQ12 -> unconnected-(U8J-GPIOB_TXN06-Pad46)
- U8 pad 47: /sdram/DQ4 -> unconnected-(U8J-GPIOB_TXP09-Pad47)
- U8 pad 48: /sdram/DQ5 -> unconnected-(U8J-GPIOB_TXN09-Pad48)
- U8 pad 53: /sdram/DQ11 -> unconnected-(U8J-GPIOB_TXP11-Pad53)
- U8 pad 54: /sdram/DQ10 -> unconnected-(U8J-GPIOB_TXN11-Pad54)
- U8 pad 55: /sdram/DQ9 -> unconnected-(U8I-GPIOB_RXP00-Pad55)
- U8 pad 56: /sdram/DQ6 -> unconnected-(U8I-GPIOB_RXN00-Pad56)
- U8 pad 58: /sdram/DQ8 -> unconnected-(U8I-GPIOB_RXP02-Pad58)
- U8 pad 59: /sdram/DQMH -> unconnected-(U8I-GPIOB_RXN02-Pad59)
- U8 pad 6: unconnected-(U8C-GPIOL_46-Pad6) -> /sdram/CSb
- U8 pad 60: /sdram/CLK -> unconnected-(U8I-GPIOB_RXN03-Pad60)
- U8 pad 61: /sdram/DQ7 -> unconnected-(U8I-GPIOB_RXP03-Pad61)
- U8 pad 65: /sdram/DQML -> unconnected-(U8I-GPIOB_RXN07-Pad65)
- U8 pad 66: /sdram/WEb -> unconnected-(U8I-GPIOB_RXP07-Pad66)
- U8 pad 67: /sdram/CASb -> unconnected-(U8I-GPIOB_RXP10-Pad67)
- U8 pad 68: /sdram/CKE -> unconnected-(U8I-GPIOB_RXN10-Pad68)
- U8 pad 69: /sdram/A12 -> unconnected-(U8I-GPIOB_RXN12_EXTFB0-Pad69)
- U8 pad 7: unconnected-(U8C-GPIOL_41_CDI9-Pad7) -> /sdram/RASb
- U8 pad 70: /sdram/A11 -> unconnected-(U8I-GPIOB_RXP12_EXTFB0-Pad70)
- U8 pad 71: /sdram/A9 -> unconnected-(U8I-GPIOB_CLKP0-Pad71)
- U8 pad 72: /sdram/A7 -> unconnected-(U8I-GPIOB_CLKN0-Pad72)
- U8 pad 74: /sdram/A8 -> LED7
- U8 pad 75: /sdram/A6 -> Net-(U8H-GPIOR_157_PLLIN)
- U8 pad 76: /sdram/A4 -> /sdram/DQ15
- U8 pad 77: /sdram/A5 -> /sdram/DQ14
- U8 pad 78: Net-(U8H-GPIOR_151_CBUS0) -> LED6
- U8 pad 79: /sdram/RASb -> LED5
- U8 pad 8: unconnected-(U8C-GPIOL_40_CDI8-Pad8) -> /sdram/CASb
- U8 pad 80: /sdram/CSb -> LED4
- U8 pad 81: /sdram/BA0 -> /sdram/DQ13
- U8 pad 82: /sdram/A3 -> LED3
- U8 pad 83: /sdram/A2 -> LED2
- U8 pad 84: /sdram/A1 -> LED1
- U8 pad 86: /sdram/A0 -> /sdram/DQ12
- U8 pad 87: /sdram/A10 -> /sdram/DQ11
- U8 pad 89: /sdram/BA1 -> /sdram/DQ10
- U8 pad 90: unconnected-(U8G-GPIOR_128_CTRL11-Pad90) -> /sdram/DQ9
- U8 pad 92: unconnected-(U8G-GPIOR_125_CLK10-Pad92) -> LED0
- U8 pad 93: unconnected-(U8F-GPIOR_123_CLK12_CDI20-Pad93) -> /sdram/DQ8
- U8 pad 97: unconnected-(U8F-GPIOR_122_CLK13_CDI21-Pad97) -> /sdram/DQMH
- U8 pad 98: /LED/LED7 -> /sdram/CLK
- U8 pad 99: /LED/LED6 -> /sdram/CKE
- X2 pad 3: Net-(U8D-GPIOL_74_PLLIN0) -> Net-(U8H-GPIOR_157_PLLIN)
Routing:
- net +1V2: track 35.8 -> 58.6 mm, vias 42 -> 38
- net +3V3: track 102.0 -> 122.9 mm, vias 67 -> 56
- net /LED/LED7: track 14.5 -> 0.00 mm
- net /LED/LED6: track 13.5 -> 0.00 mm
- net /sdram/A5: track 13.4 -> 0.00 mm, vias 1 -> 0
- net /sdram/A4: track 12.8 -> 0.00 mm, vias 1 -> 0
- net /LED/LED5: track 12.4 -> 0.00 mm
- net /LED/LED4: track 11.2 -> 0.00 mm
- net LED2: track 0.00 -> 10.7 mm
- net /ulpi/ULPI_STP: track 10.3 -> 0.00 mm
- net ULPI_STP: track 0.00 -> 10.3 mm
- net /LED/LED3: track 10.1 -> 0.00 mm
- net LED1: track 0.00 -> 9.62 mm
- net LED7: track 0.00 -> 9.57 mm, vias 0 -> 2
- net /LED/LED1: track 9.42 -> 0.00 mm
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- added copper zone on In2.Cu, net +1V2
- removed copper zone on B.Cu, net +1V2
