File: trion-8-test.kicad_pcb (KiCad board)
At the start: 4 copper layers, 39.5 x 80 mm, 187 parts, among them J1 USB_C_Receptacle_USB2.0, J2 FT_JTAG, J3 T8_JTAG, J4 USB_C_Receptacle_USB2.0, J5 USB_C_Receptacle_USB2.0, Q1 SSM3K37MFV, SW1 Reset, U1 FXL5T244, U10 USB3343, U12 RT8096B, U13 STUSB03E, U2 FT2232HL, U3 93LCxxAxxOT, U4 TLV75801PDBV, U5 TSX339IPT, U6 RT8096B, U7 2N7001T, U8 T8Q144xx, U9 AT25FF081A-SSHN-B, X1 ECS-2520MV-120-CM, X2 ECS-2520MV-120-CM, Y1 26MHz

Commit message: updated R20 to 1M (100k proved to strong a pull-down)
Parts:
- R20: value 100k -> 1M
Changed lines of the file:
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@@
         (effects (font (size 1 1) (thickness 0.15)) (justify mirror))
     )
-    (fp_text value "100k" (at 0 -1.43) (layer "B.Fab")
+    (fp_text value "1M" (at 0 -1.43) (layer "B.Fab")
         (effects (font (size 1 1) (thickness 0.15)) (justify mirror))
     )
