File: trion-8-test.kicad_pcb (KiCad board)
At the start: 4 copper layers, 46 x 51.5 mm, 130 parts, among them J3 T8_JTAG, J4 USB_C_Receptacle_USB2.0, Q1 SSM3K37MFV, SW1 Reset, U1 MT48LC16M16A2P, U10 USB3343, U12 RT8096B, U6 RT8096B, U8 T8Q144xx, U9 AT25FF081A-SSHN-B, X2 ECS-2520MV-120-CM, Y1 26MHz

Commit message: rerouted some SDRAM pins to 139,140,141,142,144
Preparation for moving ULPI to free up some DDIO pins
on the other side of the package...
Parts:
- moved C15 1.30 mm to (68.5, 104.0), turned to -90 degrees
- moved C66 0.19 mm to (75.0, 104.2)
Connections:
- U8 pad 131: /sdram/A10 -> unconnected-(U8D-GPIOL_75_PLLIN1-Pad131)
- U8 pad 134: /sdram/A1 -> unconnected-(U8D-GPIOL_73_EXTFB1_CDI15-Pad134)
- U8 pad 135: /sdram/A2 -> unconnected-(U8D-GPIOL_72_EXTFB0_CDI14-Pad135)
- U8 pad 136: /sdram/A3 -> unconnected-(U8D-GPIOL_71_NSTATUS-Pad136)
- U8 pad 137: /sdram/A0 -> unconnected-(U8D-GPIOL_70_CBSEL0-Pad137)
- U8 pad 139: unconnected-(U8D-GPIOL_68-Pad139) -> /sdram/A1
- U8 pad 140: unconnected-(U8D-GPIOL_67_CDI13-Pad140) -> /sdram/A2
- U8 pad 141: unconnected-(U8D-GPIOL_65-Pad141) -> /sdram/A3
- U8 pad 142: unconnected-(U8D-GPIOL_66_CDI12-Pad142) -> /sdram/A10
- U8 pad 144: unconnected-(U8D-GPIOL_64-Pad144) -> /sdram/A0
Routing:
- net /sdram/A1: track 3.34 -> 6.48 mm
- net /sdram/A10: track 6.82 -> 4.24 mm
- net +1V2: track 58.6 -> 60.3 mm
- net /sdram/A0: track 6.25 -> 4.99 mm
- net /sdram/BA1: track 6.40 -> 7.35 mm
- net GND: track 185.3 -> 184.4 mm, vias 131 -> 130

Commit message: added ethernet phy
Parts:
- added C16: 100n, Capacitor_SMD:C_0603_1608Metric, F.Cu at (117.2, 88.4)
- added C17: 100n, Capacitor_SMD:C_0603_1608Metric, F.Cu at (116.6, 97.8)
- added C18: 100n, Capacitor_SMD:C_0603_1608Metric, F.Cu at (100.0, 82.0)
- added C19: 100n, Capacitor_SMD:C_0603_1608Metric, F.Cu at (119.4, 88.9)
- added C20: 100n, Capacitor_SMD:C_0603_1608Metric, B.Cu at (127.9, 91.3)
- added C23: 4u7, Capacitor_SMD:C_0805_2012Metric, B.Cu at (106.0, 83.2)
- added C24: 100n, Capacitor_SMD:C_0603_1608Metric, F.Cu at (102.1, 94.8)
- added C25: 100n, Capacitor_SMD:C_0603_1608Metric, B.Cu at (103.7, 93.6)
- added C26: 100n, Capacitor_SMD:C_0603_1608Metric, F.Cu at (106.3, 85.0)
- added C46: 4u7, Capacitor_SMD:C_0805_2012Metric, F.Cu at (116.9, 86.4)
- added C47: 100n, Capacitor_SMD:C_0603_1608Metric, F.Cu at (113.9, 90.4)
- added C55: 100n, Capacitor_SMD:C_0603_1608Metric, B.Cu at (111.1, 91.1)
- added C56: 100n, Capacitor_SMD:C_0603_1608Metric, F.Cu at (123.1, 82.4)
- added C58: 1n, Capacitor_SMD:C_0603_1608Metric, F.Cu at (132.0, 82.3)
- added C60: 1n, Capacitor_SMD:C_0603_1608Metric, F.Cu at (131.9, 101.6)
- added C73: 100n, Capacitor_SMD:C_0603_1608Metric, F.Cu at (124.9, 101.5)
- added C74: 100n, Capacitor_SMD:C_0603_1608Metric, F.Cu at (104.0, 119.7)
- added C75: 100n, Capacitor_SMD:C_0603_1608Metric, F.Cu at (132.0, 119.5)
- added D11: LED, LED_SMD:LED_0603_1608Metric, F.Cu at (141.1, 82.3)
- added J1: RJ45_Amphenol_RJMG1BD3B8K1ANR, Connector_RJ:RJ45_Amphenol_RJMG1BD3B8K1ANR, F.Cu at (125.2, 96.3)
- added J2: T8_JTAG, Connector_PinHeader_2.00mm:PinHeader_2x07_P2.00mm_Vertical, F.Cu at (117.8, 102.1)
- added J5: ETH GPIO, Connector_PinHeader_2.54mm:PinHeader_2x10_P2.54mm_Vertical, F.Cu at (106.6, 78.1)
- added J6: FPGA GPIO, Connector_PinHeader_2.54mm:PinHeader_2x10_P2.54mm_Vertical, F.Cu at (106.6, 120.9)
- added J7: FPGA_B3_GPIO, Connector_PinHeader_2.54mm:PinHeader_2x04_P2.54mm_Vertical, F.Cu at (93.5, 78.0)
- added JP1: 2k2, proj_footprints:J_0603_I, F.Cu at (107.3, 79.9)
- added JP2: 2k2, proj_footprints:J_0603_I, F.Cu at (107.3, 81.1)
- added JP3: 2k2, proj_footprints:J_0603_L, B.Cu at (104.4, 88.6)
- added JP4: 2k2, proj_footprints:J_0603_L, B.Cu at (108.0, 94.8)
- added JP5: 2k2, proj_footprints:J_0603_L, B.Cu at (101.7, 89.0)
- added L2: 600Ohm@100MHz, Inductor_SMD:L_0603_1608Metric, F.Cu at (114.2, 87.4)
- added R10: 0, Resistor_SMD:R_0603_1608Metric, F.Cu at (101.3, 88.7)
- added R11: 2k2, Resistor_SMD:R_0603_1608Metric, B.Cu at (101.2, 90.1)
- added R12: 2k2, Resistor_SMD:R_0603_1608Metric, B.Cu at (106.4, 89.9)
- added R17: 2k2, Resistor_SMD:R_0603_1608Metric, F.Cu at (115.2, 81.4)
- added R18: 2k2, Resistor_SMD:R_0603_1608Metric, F.Cu at (116.7, 81.4)
- added R19: 2k2, Resistor_SMD:R_0603_1608Metric, F.Cu at (118.2, 81.4)
- added R2: 50, Resistor_SMD:R_0603_1608Metric, F.Cu at (115.9, 94.7)
- added R21: 1k5, Resistor_SMD:R_0603_1608Metric, F.Cu at (108.5, 84.3)
- added R25: 2k2, Resistor_SMD:R_0603_1608Metric, B.Cu at (100.5, 93.1)
- added R26: 2k2, Resistor_SMD:R_0603_1608Metric, B.Cu at (105.8, 93.6)
- added R27: 2k2, Resistor_SMD:R_0603_1608Metric, B.Cu at (101.2, 91.6)
- added R28: 2k2, Resistor_SMD:R_0603_1608Metric, B.Cu at (106.3, 91.4)
- added R3: 50, Resistor_SMD:R_0603_1608Metric, F.Cu at (117.3, 94.7)
- added R4: 50, Resistor_SMD:R_0603_1608Metric, F.Cu at (117.4, 90.7)
- added R5: 50, Resistor_SMD:R_0603_1608Metric, F.Cu at (115.9, 90.7)
- added R53: 4k87, Resistor_SMD:R_0603_1608Metric, B.Cu at (111.0, 89.6)
- added R54: 0, Resistor_SMD:R_0603_1608Metric, F.Cu at (114.2, 97.5)
- added R55: 10k, Resistor_SMD:R_0603_1608Metric, F.Cu at (103.6, 103.1)
- added R6: 680, Resistor_SMD:R_0603_1608Metric, F.Cu at (135.7, 82.3)
- added R7: 680, Resistor_SMD:R_0603_1608Metric, F.Cu at (135.8, 101.5)
- added R8: 1k, Resistor_SMD:R_0603_1608Metric, F.Cu at (138.2, 82.0)
- added R9: 0, Resistor_SMD:R_0603_1608Metric, F.Cu at (99.0, 87.1)
- added U2: dp83640, Package_QFP:LQFP-48_7x7mm_P0.5mm, F.Cu at (108.0, 91.0)
- added X1: ECS-2520MV-120-CM, Oscillator:Oscillator_SMD_ECS_2520MV-xxx-xx-4Pin_2.5x2.0mm, F.Cu at (99.9, 84.2)
- moved H2 40.8 mm to (137.3, 118.5)
- moved H4 40.0 mm to (137.5, 78.0)
- moved C49 1.50 mm to (59.9, 94.0)
- moved C51 1.50 mm to (64.3, 91.3)
- moved C52 1.50 mm to (59.9, 97.7)
- moved C53 1.50 mm to (63.5, 100.1)
- moved R73 1.50 mm to (61.3, 97.7)
- moved U10 1.50 mm to (64.0, 93.2)
- moved Y1 1.50 mm to (63.6, 97.6)
- moved C48 1.50 mm to (62.0, 92.8)
- moved R46 1.50 mm to (59.7, 92.6)
- moved R47 1.50 mm to (59.9, 95.5)
- moved C50 1.23 mm to (66.0, 94.7)
- moved R49 1.22 mm to (63.6, 101.9), turned to 180 degrees
- moved R48 0.60 mm to (66.2, 100.8)
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Connections:
- R30 pad 2: LED7 -> /sdram/DQ15
- U1 pad 35: /sdram/A11 -> A11
- U1 pad 36: /sdram/A12 -> A12
- U1 pad 37: /sdram/CKE -> CKE
- U10 pad 1: /ulpi/ULPI_DIR -> ULPI_DIR
- U10 pad 2: /ulpi/ULPI_CLK -> ULPI_CLK
- U10 pad 3: /ulpi/ULPI_NXT -> ULPI_NXT
- U8 pad 100: /sdram/A12 -> /sdram/DQ8
- U8 pad 101: /sdram/A11 -> /sdram/DQMH
- U8 pad 111: /ulpi/ULPI_D7 -> A12
- U8 pad 112: /ulpi/ULPI_D6 -> A11
- U8 pad 113: /ulpi/ULPI_D5 -> CKE
- U8 pad 114: /ulpi/ULPI_D4 -> /ulpi/ULPI_D7
- U8 pad 115: /ulpi/ULPI_D3 -> /ulpi/ULPI_D6
- U8 pad 116: /ulpi/ULPI_D2 -> /ulpi/ULPI_D5
- U8 pad 117: /ulpi/ULPI_D1 -> /ulpi/ULPI_D4
- U8 pad 118: /ulpi/ULPI_D0 -> /ulpi/ULPI_D3
- U8 pad 119: /ulpi/ULPI_NXT -> /ulpi/ULPI_D2
- U8 pad 123: /ulpi/ULPI_CLK -> /ulpi/ULPI_D1
- U8 pad 124: /ulpi/ULPI_DIR -> /ulpi/ULPI_D0
- U8 pad 131: unconnected-(U8D-GPIOL_75_PLLIN1-Pad131) -> ULPI_NXT
- U8 pad 132: ULPI_STP -> ULPI_CLK
- U8 pad 134: unconnected-(U8D-GPIOL_73_EXTFB1_CDI15-Pad134) -> ULPI_DIR
- U8 pad 135: unconnected-(U8D-GPIOL_72_EXTFB0_CDI14-Pad135) -> ULPI_STP
- U8 pad 36: unconnected-(U8J-REF_RES-Pad36) -> FPGA_GPIO_0
- U8 pad 38: unconnected-(U8J-GPIOB_TXP00-Pad38) -> FPGA_GPIO_1
- U8 pad 39: unconnected-(U8J-GPIOB_TXN00-Pad39) -> FPGA_GPIO_2
- U8 pad 40: unconnected-(U8J-GPIOB_TXP02-Pad40) -> FPGA_GPIO_3
- U8 pad 41: unconnected-(U8J-GPIOB_TXN02-Pad41) -> FPGA_GPIO_4
- U8 pad 42: unconnected-(U8J-GPIOB_TXP04-Pad42) -> FPGA_GPIO_5
- U8 pad 43: unconnected-(U8J-GPIOB_TXN04-Pad43) -> FPGA_GPIO_6
- U8 pad 45: unconnected-(U8J-GPIOB_TXP06-Pad45) -> FPGA_GPIO_7
- U8 pad 46: unconnected-(U8J-GPIOB_TXN06-Pad46) -> ETH0_RSTb
- U8 pad 47: unconnected-(U8J-GPIOB_TXP09-Pad47) -> ETH0_MDIO
- U8 pad 48: unconnected-(U8J-GPIOB_TXN09-Pad48) -> ETH0_MDC
- U8 pad 53: unconnected-(U8J-GPIOB_TXP11-Pad53) -> ETH0_PWRDWN_IRQ
- U8 pad 54: unconnected-(U8J-GPIOB_TXN11-Pad54) -> ETH0_TXD_3
- U8 pad 55: unconnected-(U8I-GPIOB_RXP00-Pad55) -> ETH0_TXD_2
- U8 pad 56: unconnected-(U8I-GPIOB_RXN00-Pad56) -> ETH0_TXD_1
- U8 pad 58: unconnected-(U8I-GPIOB_RXP02-Pad58) -> ETH0_TXD_0
- U8 pad 59: unconnected-(U8I-GPIOB_RXN02-Pad59) -> ETH0_TX_EN
- U8 pad 60: unconnected-(U8I-GPIOB_RXN03-Pad60) -> ETH0_RXD_0
- U8 pad 61: unconnected-(U8I-GPIOB_RXP03-Pad61) -> ETH0_RXD_1
- U8 pad 65: unconnected-(U8I-GPIOB_RXN07-Pad65) -> ETH0_RXD_2
- U8 pad 66: unconnected-(U8I-GPIOB_RXP07-Pad66) -> ETH0_RXD_3
- U8 pad 67: unconnected-(U8I-GPIOB_RXP10-Pad67) -> ETH0_COL
- U8 pad 68: unconnected-(U8I-GPIOB_RXN10-Pad68) -> ETH0_RX_ER
- U8 pad 69: unconnected-(U8I-GPIOB_RXN12_EXTFB0-Pad69) -> ETH0_CRS_DV
- U8 pad 70: unconnected-(U8I-GPIOB_RXP12_EXTFB0-Pad70) -> ETH0_RX_DV
- U8 pad 71: unconnected-(U8I-GPIOB_CLKP0-Pad71) -> ETH0_RX_CLK
- U8 pad 72: unconnected-(U8I-GPIOB_CLKN0-Pad72) -> ETH0_GPIO_9
- U8 pad 74: LED7 -> /sdram/DQ15
- U8 pad 76: /sdram/DQ15 -> LED7
- U8 pad 89: /sdram/DQ10 -> FPGA_B3_IO_2
- U8 pad 90: /sdram/DQ9 -> FPGA_B3_IO_1
- U8 pad 93: /sdram/DQ8 -> FPGA_B3_IO_0
- U8 pad 97: /sdram/DQMH -> /sdram/DQ10
- U8 pad 99: /sdram/CKE -> /sdram/DQ9
Routing:
- net GND: track 184.4 -> 249.3 mm, vias 130 -> 176
- net +3V3: track 122.9 -> 182.6 mm, vias 56 -> 82
- net ETH0_LED_ACT: track 0.00 -> 55.2 mm, vias 0 -> 2
- net ETH0_GPIO_9: track 0.00 -> 42.1 mm, vias 0 -> 2
- net FPGA_GPIO_7: track 0.00 -> 41.1 mm
- net Net-(C56-Pad1): track 0.00 -> 39.7 mm
- net FPGA_GPIO_6: track 0.00 -> 38.2 mm
- net FPGA_GPIO_5: track 0.00 -> 36.2 mm
- net ETH0_LED_SPEED: track 0.00 -> 35.1 mm, vias 0 -> 2
- net ETH0_LED_LINK: track 0.00 -> 34.8 mm, vias 0 -> 2
- net FPGA_GPIO_4: track 0.00 -> 32.7 mm
- net FPGA_GPIO_3: track 0.00 -> 29.8 mm
- net ETH0_RDP: track 0.00 -> 28.9 mm
- net FPGA_B3_IO_2: track 0.00 -> 28.2 mm
- net ETH0_RDN: track 0.00 -> 27.7 mm
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Other:
- board size 46 x 51.5 mm -> 86 x 51.5 mm
- board text added: "3V3"
- board text added: "REF"
- board text added: "RST"
- board text added: "Trion-SDRAM-Test V2.0"
- board text removed: "Trion-SDRAM-Test V1.0"

Commit message: PCB: updated silkscreen
Enabled LED labeling, added some labels for connector pins
Other:
- board text added: "1"
- board text added: "14"
- board text added: "19"
- board text added: "2"
- board text added: "20"
- board text added: "4"
- board text added: "8"
Changed lines of the file:
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@@
     (property "ki_keywords" "LED diode")
     (attr smd)
-    (fp_text reference "D6" (at 0 -1.43 90) (layer "F.SilkS") hide
-        (effects (font (size 1 1) (thickness 0.15)))
+    (fp_text reference "D6" (at 1.7415 0.025 180) (layer "F.SilkS")
+        (effects (font (size 0.8 0.8) (thickness 0.1)))
     )
     (fp_text value "LED" (at 0 1.43 90) (layer "F.Fab")
@@
     (property "ki_keywords" "LED diode")
     (attr smd)
-    (fp_text reference "D9" (at 0 -1.43 90) (layer "F.SilkS") hide
-        (effects (font (size 1 1) (thickness 0.15)))
+    (fp_text reference "D9" (at 1.7765 -0.005 180) (layer "F.SilkS")
+        (effects (font (size 0.8 0.8) (thickness 0.1)))
     )
     (fp_text value "LED" (at 0 1.43 90) (layer "F.Fab")
@@
     (property "ki_keywords" "LED diode")
     (attr smd)
-    (fp_text reference "D5" (at 0 -1.43 90) (layer "F.SilkS") hide
-        (effects (font (size 1 1) (thickness 0.15)))
+    (fp_text reference "D5" (at 1.738 0.013 180) (layer "F.SilkS")
+        (effects (font (size 0.8 0.8) (thickness 0.1)))
     )
     (fp_text value "LED" (at 0 1.43 90) (layer "F.Fab")
@@
     (property "ki_keywords" "LED diode")
     (attr smd)
-    (fp_text reference "D4" (at 0 -1.43 90) (layer "F.SilkS") hide
-        (effects (font (size 1 1) (thickness 0.15)))
+    (fp_text reference "D4" (at 1.7385 0.033 180) (layer "F.SilkS")
+        (effects (font (size 0.8 0.8) (thickness 0.1)))
     )
     (fp_text value "LED" (at 0 1.43 90) (layer "F.Fab")
@@
     (property "ki_keywords" "LED diode")
     (attr smd)
-    (fp_text reference "D3" (at 0 -1.43 90) (layer "F.SilkS") hide
-        (effects (font (size 1 1) (thickness 0.15)))
+    (fp_text reference "D3" (at 1.768 0.022 180) (layer "F.SilkS")
+        (effects (font (size 0.8 0.8) (thickness 0.1)))
     )
     (fp_text value "LED" (at 0 1.43 90) (layer "F.Fab")
@@
     (property "ki_keywords" "LED diode")
     (attr smd)
-    (fp_text reference "D8" (at 0 -1.43 90) (layer "F.SilkS") hide
-        (effects (font (size 1 1) (thickness 0.15)))
+    (fp_text reference "D8" (at 1.7955 0.015 180) (layer "F.SilkS")
+        (effects (font (size 0.8 0.8) (thickness 0.1)))
     )
     (fp_text value "LED" (at 0 1.43 90) (layer "F.Fab")
@@
     (property "ki_keywords" "connector")
     (attr through_hole)
-    (fp_text reference "J7" (at 1.79 -1.96 90) (layer "F.SilkS")
+    (fp_text reference "J7" (at 2.707 -1.995 90) (layer "F.SilkS")
         (effects (font (size 1 1) (thickness 0.15)))
     )
@@
     (property "ki_keywords" "LED diode")
     (attr smd)
-    (fp_text reference "D2" (at 0 -1.43 90) (layer "F.SilkS") hide
-        (effects (font (size 1 1) (thickness 0.15)))
+    (fp_text reference "D2" (at 1.797 0.012 180) (layer "F.SilkS")
+        (effects (font (size 0.8 0.8) (thickness 0.1)))
     )
     (fp_text value "LED" (at 0 1.43 90) (layer "F.Fab")
@@
     (property "ki_keywords" "LED diode")
     (attr smd)
-    (fp_text reference "D7" (at 0 -1.43 90) (layer "F.SilkS") hide
-        (effects (font (size 1 1) (thickness 0.15)))
+    (fp_text reference "D7" (at 1.7755 0.034 180) (layer "F.SilkS")
+        (effects (font (size 0.8 0.8) (thickness 0.1)))
     )
     (fp_text value "LED" (at 0 1.43 90) (layer "F.Fab")
@@
     (effects (font (size 0.8 0.8) (thickness 0.1)) (justify left bottom))
   )
+  (gr_text "1" (at 119.547 101.948) (layer "F.SilkS")
+    (effects (font (size 0.8 0.8) (thickness 0.1)) (justify bottom))
+  )
+  (gr_text "20" (at 131.693 75.768) (layer "F.SilkS")
+    (effects (font (size 0.8 0.8) (thickness 0.1)) (justify bottom))
+  )
+  (gr_text "2" (at 93.442 73.885) (layer "F.SilkS")
+    (effects (font (size 0.8 0.8) (thickness 0.1)) (justify bottom))
+  )
   (gr_text "GND" (at 102.27 122.32) (layer "F.SilkS")
     (effects (font (size 0.8 0.8) (thickness 0.1)) (justify left bottom))
@@
     (effects (font (size 0.8 0.8) (thickness 0.153) bold) (justify left bottom))
   )
+  (gr_text "19\n" (at 131.693 78.755) (layer "F.SilkS")
+    (effects (font (size 0.8 0.8) (thickness 0.1)) (justify bottom))
+  )
   (gr_text "RSTb" (at 92.68 117.18 270) (layer "F.SilkS")
     (effects (font (size 0.8 0.8) (thickness 0.1)) (justify left bottom))
   )
+  (gr_text "14" (at 78.065 123.375) (layer "F.SilkS")
+    (effects (font (size 0.8 0.8) (thickness 0.1)) (justify bottom))
+  )
   (gr_text "TCK" (at 95.48 117.405 270) (layer "F.SilkS")
     (effects (font (size 0.8 0.8) (thickness 0.1)) (justify left bottom))
   )
+  (gr_text "1" (at 104.52 78.711) (layer "F.SilkS")
+    (effects (font (size 0.8 0.8) (thickness 0.1)) (justify bottom))
+  )
+  (gr_text "2" (at 117.653 106.421) (layer "F.SilkS")
+    (effects (font (size 0.8 0.8) (thickness 0.1)) (justify bottom))
+  )
   (gr_text "TDI" (at 93.63 117.405 270) (layer "F.SilkS")
     (effects (font (size 0.8 0.8) (thickness 0.1)) (justify left bottom))
@@
     (effects (font (size 0.8 0.8) (thickness 0.1)) (justify left bottom))
   )
+  (gr_text "2" (at 106.615 116.573) (layer "F.SilkS")
+    (effects (font (size 0.8 0.8) (thickness 0.1)) (justify bottom))
+  )
   (gr_text "SSb\n" (at 91.705 117.205 270) (layer "F.SilkS")
     (effects (font (size 0.8 0.8) (thickness 0.1)) (justify left bottom))
@@
     (effects (font (size 0.8 0.8) (thickness 0.1)) (justify left bottom))
   )
+  (gr_text "2" (at 106.598 73.824) (layer "F.SilkS")
+    (effects (font (size 0.8 0.8) (thickness 0.1)) (justify bottom))
+  )
   (gr_text "GND" (at 130.7938 122.232) (layer "F.SilkS")
     (effects (font (size 0.8 0.8) (thickness 0.1)) (justify left bottom))
   )
+  (gr_text "2" (at 89.905 123.402) (layer "F.SilkS")
+    (effects (font (size 0.8 0.8) (thickness 0.1)) (justify bottom))
+  )
   (gr_text "TCK" (at 109.783 100.68 90) (layer "F.SilkS")
     (effects (font (size 0.8 0.8) (thickness 0.153) bold) (justify left bottom))
@@
     (effects (font (size 0.8 0.8) (thickness 0.153) bold) (justify left bottom))
   )
+  (gr_text "14" (at 105.813 106.394) (layer "F.SilkS")
+    (effects (font (size 0.8 0.8) (thickness 0.1)) (justify bottom))
+  )
+  (gr_text "4" (at 87.952 123.425) (layer "F.SilkS")
+    (effects (font (size 0.8 0.8) (thickness 0.1)) (justify bottom))
+  )
+  (gr_text "4" (at 115.7 106.444) (layer "F.SilkS")
+    (effects (font (size 0.8 0.8) (thickness 0.1)) (justify bottom))
+  )
+  (gr_text "4" (at 109.094 116.573) (layer "F.SilkS")
+    (effects (font (size 0.8 0.8) (thickness 0.1)) (justify bottom))
+  )
+  (gr_text "8\n" (at 101.083 73.824) (layer "F.SilkS")
+    (effects (font (size 0.8 0.8) (thickness 0.1)) (justify bottom))
+  )
+  (gr_text "1" (at 92.809 80.501) (layer "F.SilkS")
+    (effects (font (size 0.8 0.8) (thickness 0.1)) (justify bottom))
+  )
   (gr_text "TDO" (at 94.555 117.405 270) (layer "F.SilkS")
     (effects (font (size 0.8 0.8) (thickness 0.1)) (justify left bottom))
@@
     (effects (font (size 0.8 0.8) (thickness 0.1)) (justify left bottom))
   )
+  (gr_text "20" (at 129.381 116.624) (layer "F.SilkS")
+    (effects (font (size 0.8 0.8) (thickness 0.1)) (justify bottom))
+  )
   (gr_text "TDO" (at 111.875 100.68 90) (layer "F.SilkS")

Commit message: Added GPS receiver; increased board size
including battery supply; made board bigger
and added edge connectors for ETH GPIO, PPS
and antenna.
Parts:
- removed D10, D6, D7, D8, D9: LED, LED_SMD:LED_0603_1608Metric
- removed J7: FPGA_B3_GPIO, Connector_PinHeader_2.54mm:PinHeader_2x04_P2.54mm_Vertical
- removed R54: 0, Resistor_SMD:R_0603_1608Metric
- removed R55: 10k, Resistor_SMD:R_0603_1608Metric
- removed R64: 1k, Resistor_SMD:R_0603_1608Metric
- added BT1: Battery_Cell, battery:bh-3034-74-combined, B.Cu at (140.6, 95.8)
- added C76: 100n, Capacitor_SMD:C_0603_1608Metric, F.Cu at (114.4, 132.6)
- added C77: 50p, Capacitor_SMD:C_0603_1608Metric, F.Cu at (112.2, 131.9)
- added C78: 50p, Capacitor_SMD:C_0603_1608Metric, F.Cu at (111.0, 117.2)
- added C79: 100n, Capacitor_SMD:C_0603_1608Metric, F.Cu at (106.5, 121.4)
- added C80: 100n, Capacitor_SMD:C_0603_1608Metric, F.Cu at (112.5, 117.1)
- added C81: 4u7, Capacitor_SMD:C_0805_2012Metric, F.Cu at (106.3, 123.2)
- added C82: 50p, Capacitor_SMD:C_0603_1608Metric, F.Cu at (108.8, 117.8)
- added C83: 4u7, Capacitor_SMD:C_0805_2012Metric, F.Cu at (149.8, 115.5)
- added D12: D, Diode_SMD:D_SOD-323F, F.Cu at (148.8, 109.5)
- added D13: ~, Diode_SMD:D_SOD-882, F.Cu at (109.7, 133.0)
- added J10: PPS, proj_footprints:LEMO+SMA_molex_732515460, F.Cu at (128.7, 134.9)
- added J11: IO1, proj_footprints:LEMO+SMA_molex_732515460, F.Cu at (100.8, 65.2)
- added J12: IO2, proj_footprints:LEMO+SMA_molex_732515460, F.Cu at (110.8, 65.2)
- added J13: IO3, proj_footprints:LEMO+SMA_molex_732515460, F.Cu at (120.8, 65.2)
- added J14: IO4, proj_footprints:LEMO+SMA_molex_732515460, F.Cu at (130.8, 65.2)
- added J15: IO8, proj_footprints:LEMO+SMA_molex_732515460, F.Cu at (140.8, 65.2)
- added J16: CLK, proj_footprints:LEMO+SMA_molex_732515460, F.Cu at (150.8, 65.2)
- added J8: Antenna, proj_footprints:SMA Molex 732515460, F.Cu at (110.0, 138.3)
- added J9: Geofnc, Connector_PinSocket_2.54mm:PinSocket_1x02_P2.54mm_Vertical, F.Cu at (121.6, 135.8)
- added JP6: Jumper_2_Bridged, Connector_PinHeader_2.54mm:PinHeader_1x02_P2.54mm_Vertical, F.Cu at (117.8, 131.7)
- added JP7: Jumper_3_Bridged12, Connector_PinHeader_2.54mm:PinHeader_1x03_P2.54mm_Vertical, F.Cu at (152.7, 110.4)
- added L8: 100n, Inductor_SMD:L_0402_1005Metric, F.Cu at (110.5, 131.7)
- added R13: 210, Resistor_SMD:R_0603_1608Metric, F.Cu at (115.2, 134.9)
- added R14: 2k2, Resistor_SMD:R_0603_1608Metric, F.Cu at (120.1, 129.2)
- added R15: 2k2, Resistor_SMD:R_0603_1608Metric, F.Cu at (120.1, 127.7)
- added R16: 0, Resistor_SMD:R_0603_1608Metric, F.Cu at (115.5, 112.3)
- added R20: 0, Resistor_SMD:R_0603_1608Metric, F.Cu at (115.7, 113.8)
- added R29: 0, Resistor_SMD:R_0603_1608Metric, F.Cu at (117.5, 116.0)
- added R38: 0, Resistor_SMD:R_0603_1608Metric, F.Cu at (116.0, 116.0)
- added R39: 10k, Resistor_SMD:R_0603_1608Metric, F.Cu at (80.2, 115.5)
- added R51: 1k, Resistor_SMD:R_0603_1608Metric, F.Cu at (76.6, 71.8)
- added U3: LC76G, proj_footprints:lc76g, F.Cu at (113.3, 124.5)
- added U4: TS5A63157DBV, Package_TO_SOT_SMD:SOT-23-6, F.Cu at (148.8, 112.2)
- D1, D2, D3, D4, D5: value LED -> LED_Dual_RAG; footprint LED_SMD:LED_0603_1608Metric -> proj_footprints:LED_Wuerth_Sideview
- D11: value LED -> LED-GRN
- H1, H2, H3, H4: value Foot -> Foot FF-13-P3.5X5.5B
- J2: value T8_JTAG -> GPS_GPIO; footprint Connector_PinHeader_2.00mm:PinHeader_2x07_P2.00mm_Vertical -> Connector_PinHeader_2.54mm:PinHeader_2x04_P2.54mm_Vertical
- SW1: value Reset -> Reconfig; footprint Button_Switch_SMD:SW_SPST_PTS810 -> proj_footprints:SW_SPST_PTS810_and_PTS841
- U1: value MT48LC16M16A2P -> NDS36PT5-16ET
- U8: value T8Q144xx -> T20Q144xx
- X1, X2: value ECS-2520MV-120-CM -> ECS-2520MV-250-CM
- moved D11 58.2 mm to (154.1, 139.1), turned to 0 degrees
- moved R8 55.5 mm to (154.1, 135.2), turned to 0 degrees
- moved R6 53.6 mm to (153.8, 132.8), turned to -90 degrees
- moved C58 51.6 mm to (153.8, 129.0), turned to -90 degrees
- moved D1 50.8 mm to (80.0, 62.2), turned to 180 degrees
- moved C56 48.5 mm to (153.6, 120.1), turned to 90 degrees
- moved R72 41.9 mm to (76.6, 73.3), turned to 180 degrees
- moved R36 39.3 mm to (73.6, 72.2), turned to 0 degrees
- moved C19 39.3 mm to (147.4, 116.5), turned to 0 degrees
- moved Q1 38.1 mm to (74.2, 73.9)
- moved C45 38.1 mm to (64.7, 131.5), turned to 90 degrees
- moved C20 37.6 mm to (144.8, 124.9), turned to -90 degrees
- moved J6 37.0 mm to (73.6, 137.6)
- moved C75 37.0 mm to (99.0, 136.2)
- moved C74 37.0 mm to (70.9, 136.4)
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Connections:
- D1 pad 1: Net-(D1-K) -> Net-(D1-K1)
- D2 pad 1: LED0 -> Net-(D2-K1)
- D2 pad 2: Net-(D2-A) -> +3V3
- D3 pad 1: LED1 -> Net-(D3-K1)
- D3 pad 2: Net-(D3-A) -> +3V3
- D4 pad 1: LED2 -> Net-(D4-K1)
- D4 pad 2: Net-(D4-A) -> +3V3
- D5 pad 1: LED3 -> Net-(D5-K1)
- D5 pad 2: Net-(D5-A) -> +3V3
- J2 pad 1: unconnected-(J2-Pin_1-Pad1) -> GND
- J2 pad 2: GND -> Net-(J2-Pin_2)
- J2 pad 3: Net-(J2-Pin_3) -> GND
- J2 pad 4: GND -> Net-(J2-Pin_4)
- J2 pad 5: ETH0_TDI -> GND
- J2 pad 6: GND -> GPS_PPS
- J2 pad 7: ETH0_TDO -> GND
- J2 pad 8: GND -> +3V3
- J5 pad 16: GND -> ETH0_GPIO_10
- Q1 pad 3: Net-(D10-K) -> Net-(Q1-D)
- R57 pad 1: Net-(D2-A) -> LED0
- R57 pad 2: +3V3 -> Net-(D1-K2)
- R65 pad 1: Net-(D3-A) -> LED1
- R65 pad 2: +3V3 -> Net-(D1-K1)
- R66 pad 1: Net-(D4-A) -> LED2
- R66 pad 2: +3V3 -> Net-(D2-K2)
- R67 pad 1: Net-(D5-A) -> LED3
- R67 pad 2: +3V3 -> Net-(D2-K1)
- R68 pad 1: Net-(D6-A) -> LED4
- R68 pad 2: +3V3 -> Net-(D3-K2)
- R69 pad 1: Net-(D7-A) -> LED5
- R69 pad 2: +3V3 -> Net-(D3-K1)
- R70 pad 1: Net-(D8-A) -> LED6
- R70 pad 2: +3V3 -> Net-(D4-K2)
- R71 pad 1: Net-(D9-A) -> LED7
- R71 pad 2: +3V3 -> Net-(D4-K1)
- R72 pad 1: Net-(D10-A) -> Net-(D5-K2)
- R72 pad 2: +3V3 -> Net-(Q1-D)
- SW1 pad 1: Net-(J3-Pin_3) -> GND
- SW1 pad 2: GND -> Net-(J3-Pin_3)
- U12 pad 5: unconnected-(U12-PG-Pad5) -> POWER_GOOD
- U2 pad 10: ETH0_TMS -> unconnected-(U2-TMS-Pad10)
- U2 pad 11: ETH0_TRSTb -> unconnected-(U2-TRST#-Pad11)
- U2 pad 12: ETH0_TDI -> GPS_PPS
- U2 pad 5: ETH0_TXD_2 -> unconnected-(U2-TXD_2-Pad5)
- U2 pad 8: ETH0_TCK -> unconnected-(U2-TCK-Pad8)
- U2 pad 9: ETH0_TDO -> ETH0_GPIO_10
- U8 pad 42: FPGA_GPIO_5 -> UART_RX
- U8 pad 43: FPGA_GPIO_6 -> UART_TX
- U8 pad 45: FPGA_GPIO_7 -> GPS_PPS
- U8 pad 54: ETH0_TXD_3 -> FPGA_GPIO_5
- U8 pad 55: ETH0_TXD_2 -> FPGA_GPIO_6
- U8 pad 65: ETH0_RXD_2 -> FPGA_GPIO_7
- U8 pad 66: ETH0_RXD_3 -> GPS_RSTb
- U8 pad 89: FPGA_B3_IO_2 -> ETH0_GPIO_1
- U8 pad 90: FPGA_B3_IO_1 -> ETH0_GPIO_2
- U8 pad 93: FPGA_B3_IO_0 -> ETH0_CLK_OUT
Routing:
- net GPS_PPS: track 0.00 -> 80.9 mm
- net ETH0_CLK_OUT: track 22.8 -> 97.4 mm, vias 0 -> 2
- net POWER_GOOD: track 0.00 -> 73.7 mm, vias 0 -> 2
- net ETH0_LED_SPEED: track 35.1 -> 90.9 mm
- net Net-(D12-K): track 0.00 -> 54.6 mm, vias 0 -> 2
- net ETH0_LED_LINK: track 34.8 -> 89.1 mm
- net ETH0_LED_ACT: track 55.2 -> 108.4 mm
- net Net-(BT1-+): track 0.00 -> 50.0 mm
- net ETH0_GPIO_2: track 23.8 -> 67.5 mm, vias 1 -> 3
- net Net-(Q1-G): track 5.93 -> 49.6 mm
- net ETH0_TDP: track 16.4 -> 59.5 mm
- net ETH0_TDN: track 18.2 -> 60.1 mm
- net GND: track 249.3 -> 289.6 mm, vias 176 -> 206
- net GPS_RSTb: track 0.00 -> 39.6 mm, vias 0 -> 2
- net ETH0_GPIO_1: track 22.6 -> 61.5 mm, vias 1 -> 2
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Other:
- board size 86 x 51.5 mm -> 100 x 80 mm
- board text added: "CLK"
- board text added: "Gnd"
- board text added: "IO1"
- board text added: "IO10"
- board text added: "IO2"
- board text added: "IO3"
- board text added: "IO4"
- board text added: "IO8"
- board text added: "IO9"
- board text added: "Tic-Nic V2.0"
- board text added: "X"
- board text removed: "8"
- board text removed: "REF"
- board text removed: "RST"
- board text removed: "Trion-SDRAM-Test V2.0"
