File: FT-USB-JTAG.kicad_sch (KiCad schematic)
At the start: 60 parts, among them J1 USB_C_Receptacle_USB2.0, J2 FT_JTAG, U1 FXL5T244, U2 FT2232HL, U3 93LCxxAxxOT, U4 TLV75801PDBV, U5 TSX339IPT, U7 2N7001T, X1 ECS-2520MV-120-CM

Commit message: Fixed V1.0 errata
- added feedback resistor for ulpi transceiver clock oscillator
- removed SS_N connection
Connections:
- net SS_N: no longer U1.9 (B4)
- no-connect marks 34 -> 36
Other:
- note added: "Note: could use a 4x buffer; for SS_N a buffer with OE control is required (requires a software modification to the programmer as well)."
Changed lines of the file:
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@@
   (no_connect (at 177.8 120.015))
   (no_connect (at 177.8 53.975))
+  (no_connect (at 248.285 92.71))
   (no_connect (at 177.8 109.855))
   (no_connect (at 177.8 99.695))
@@
   (no_connect (at 177.8 117.475))
   (no_connect (at 177.8 76.835))
+  (no_connect (at 238.76 92.71))
   (no_connect (at 177.8 79.375))
   (no_connect (at 177.8 114.935))
@@
     (stroke (width 0) (type default))
   )
+  (text "Note: could use a 4x buffer; for SS_N\na buffer with OE control is required\n(requires a software modification to\nthe programmer as well)."
+    (at 242.57 104.14 0)
+    (effects (font (size 1.27 1.27)) (justify left bottom))
+  )
   (label "FT_USB_N" (at 116.84 66.675 180) (fields_autoplaced)
     (effects (font (size 1.27 1.27)) (justify right bottom))
@@
     (effects (font (size 1.27 1.27)) (justify right bottom))
   )
-  (label "SS_N" (at 238.76 92.71 0) (fields_autoplaced)
+  (label "SS_N" (at 248.285 92.71 0) (fields_autoplaced)
     (effects (font (size 1.27 1.27)) (justify left bottom))
   )

Commit message: updated R20 to 1M (100k proved to strong a pull-down)
Parts:
- R20: value 100k -> 1M
Changed lines of the file:
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@@
       (effects (font (size 1.27 1.27)) (justify right))
     )
-    (property "Value" "100k" (at 66.6171 148.3614 0)
+    (property "Value" "1M" (at 66.6171 148.3614 0)
       (effects (font (size 1.27 1.27)) (justify right))
     )
