File: ulpi.kicad_sch (KiCad schematic)
At the start: 19 parts, among them J2 USB_C_Receptacle_USB2.0, U16 USB3343, U8 T8Q144xx, Y1 26MHz

Commit message: Fixed V1.0 errata
- added feedback resistor for ulpi transceiver clock oscillator
- removed SS_N connection
Parts:
- added R73: 1M, Resistor_SMD:R_0603_1608Metric, symbol Device:R_Small
- renumbered C2 to C52, C3 to C53, C17 to C54, C14 to C59, R9 to R50
Connections:
- net at C52.1, U16.20 (XO), Y1.1: now also R73.1
- net at C53.1, U16.21 (REFCLK/XI), Y1.3: now also R73.2
Other:
- note removed: "ERRATA: 1meg Resistor across Crystal missing!"
- moved on the sheet: C52, C53, Y1

Commit message: sdram layout done - COMPLETE REWORK NEEDED
cannot mix LVDS and GPIO banks due to too different timing
Parts:
- added C3: 100n, Capacitor_SMD:C_0603_1608Metric, symbol Device:C_Small
- added unit 4 of U8
- added X2: ECS-2520MV-120-CM, Oscillator:Oscillator_SMD_ECS_2520MV-xxx-xx-4Pin_2.5x2.0mm, symbol Oscillator:ECS-2520MV-xxx-xx
Connections:
- net +3V3: now also C3.1, U8.143 (VCCIO1E), X2.1 (Tri-State), X2.4 (VDD)
- net GND: now also C3.2, X2.2 (GND)
- net ULPI_RSTb: now also U8.134 (GPIOL_73_EXTFB1_CDI15)
- net ULPI_STP: now also U8.131 (GPIOL_75_PLLIN1)
- net +5V: now reaches C100.1, J2.A4 (VBUS), J2.A9 (VBUS), J2.B4 (VBUS), J2.B9 (VBUS), R?.1, U16.16 (VBAT)
- new net: U8.132 (GPIOL_74_PLLIN0), X2.3 (OUT)
- no-connect marks 4 -> 13
Other:
- moved on the sheet: C100, C52, C54, C91, J2, R50, R73, R?, U16, U8E, Y1

Commit message: layout finished; passed all checks...
Parts:
- removed C3: 100n, Capacitor_SMD:C_0603_1608Metric, symbol Device:C_Small
- removed unit 4 of U8
- removed X2: ECS-2520MV-120-CM, Oscillator:Oscillator_SMD_ECS_2520MV-xxx-xx-4Pin_2.5x2.0mm, symbol Oscillator:ECS-2520MV-xxx-xx
Connections:
- net SDRAM_A5: now reaches U8.109 (GPIOR_88_CDI28)
- net SDRAM_A4: now reaches U8.110 (GPIOR_87_CDI29)
- no-connect marks 13 -> 2

Commit message: added ethernet phy
Connections:
- net ULPI_CLK: no longer U8.123 (GPIOR_77_PLLIN1)
- net ULPI_D0: now also U8.124 (GPIOR_76_PLLIN0); no longer U8.118 (GPIOR_79_EXTFB1_CDI30)
- net ULPI_D1: now also U8.123 (GPIOR_77_PLLIN1); no longer U8.117 (GPIOR_80)
- net ULPI_D2: now also U8.119 (GPIOR_78_EXTFB0_CDI31); no longer U8.116 (GPIOR_81_MREFCLK)
- net ULPI_D3: now also U8.118 (GPIOR_79_EXTFB1_CDI30); no longer U8.115 (GPIOR_82)
- net ULPI_D4: now also U8.117 (GPIOR_80); no longer U8.114 (GPIOR_83)
- net ULPI_D5: now also U8.116 (GPIOR_81_MREFCLK); no longer U8.113 (GPIOR_84)
- net ULPI_D6: now also U8.115 (GPIOR_82); no longer U8.112 (GPIOR_86)
- net ULPI_D7: now also U8.114 (GPIOR_83); no longer U8.111 (GPIOR_85)
- net ULPI_DIR: no longer U8.124 (GPIOR_76_PLLIN0)
- net ULPI_NXT: no longer U8.119 (GPIOR_78_EXTFB0_CDI31)
- new net A11: U8.112 (GPIOR_86)
- new net A12: U8.111 (GPIOR_85)
- new net CKE: U8.113 (GPIOR_84)
Changed lines of the file:
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@@
     (stroke (width 0) (type default))
   )
-  (wire (pts (xy 165.1 152.4) (xy 187.96 152.4))
+  (wire (pts (xy 165.1 152.4) (xy 198.12 152.4))
     (stroke (width 0) (type default))
   )
-  (wire (pts (xy 165.1 127) (xy 187.96 127))
+  (wire (pts (xy 165.1 127) (xy 198.12 127))
     (stroke (width 0) (type default))
   )
@@
     (stroke (width 0) (type default))
   )
-  (wire (pts (xy 165.1 154.94) (xy 187.96 154.94))
+  (wire (pts (xy 165.1 154.94) (xy 198.12 154.94))
     (stroke (width 0) (type default))
   )
@@
     (stroke (width 0) (type default))
   )
-  (wire (pts (xy 165.1 149.86) (xy 187.96 149.86))
+  (wire (pts (xy 165.1 149.86) (xy 198.12 149.86))
     (stroke (width 0) (type default))
   )
@@
     (stroke (width 0) (type default))
   )
-  (label "ULPI_D0" (at 201.93 48.26 180) (fields_autoplaced)
+  (label "ULPI_D0" (at 201.93 40.64 180) (fields_autoplaced)
     (effects (font (size 1.27 1.27)) (justify right bottom))
   )
@@
     (effects (font (size 1.27 1.27)) (justify left bottom))
   )
-  (label "ULPI_D1" (at 201.93 50.8 180) (fields_autoplaced)
+  (label "ULPI_D1" (at 201.93 43.18 180) (fields_autoplaced)
     (effects (font (size 1.27 1.27)) (justify right bottom))
   )
-  (label "ULPI_D5" (at 262.89 43.18 0) (fields_autoplaced)
-    (effects (font (size 1.27 1.27)) (justify left bottom))
+  (label "ULPI_D5" (at 201.93 53.34 180) (fields_autoplaced)
+    (effects (font (size 1.27 1.27)) (justify right bottom))
   )
-  (label "ULPI_DIR" (at 187.96 149.86 0) (fields_autoplaced)
-    (effects (font (size 1.27 1.27)) (justify left bottom))
-  )
-  (label "ULPI_D4" (at 262.89 40.64 0) (fields_autoplaced)
-    (effects (font (size 1.27 1.27)) (justify left bottom))
+  (label "ULPI_D4" (at 201.93 50.8 180) (fields_autoplaced)
+    (effects (font (size 1.27 1.27)) (justify right bottom))
   )
   (label "ULPI_USB_P" (at 99.06 132.08 0) (fields_autoplaced)
     (effects (font (size 1.27 1.27)) (justify left bottom))
   )
-  (label "ULPI_D3" (at 201.93 55.88 180) (fields_autoplaced)
+  (label "ULPI_D3" (at 201.93 48.26 180) (fields_autoplaced)
     (effects (font (size 1.27 1.27)) (justify right bottom))
   )
-  (label "ULPI_NXT" (at 201.93 45.72 180) (fields_autoplaced)
+  (label "ULPI_D6" (at 201.93 55.88 180) (fields_autoplaced)
     (effects (font (size 1.27 1.27)) (justify right bottom))
-  )
-  (label "ULPI_D6" (at 262.89 48.26 0) (fields_autoplaced)
-    (effects (font (size 1.27 1.27)) (justify left bottom))
   )
   (label "ULPI_D3" (at 187.96 137.16 0) (fields_autoplaced)
     (effects (font (size 1.27 1.27)) (justify left bottom))
   )
-  (label "ULPI_D2" (at 201.93 53.34 180) (fields_autoplaced)
+  (label "ULPI_D2" (at 201.93 45.72 180) (fields_autoplaced)
     (effects (font (size 1.27 1.27)) (justify right bottom))
   )
@@
     (effects (font (size 1.27 1.27)) (justify left bottom))
   )
-  (label "ULPI_D7" (at 262.89 45.72 0) (fields_autoplaced)
+  (label "ULPI_D7" (at 262.89 40.64 0) (fields_autoplaced)
     (effects (font (size 1.27 1.27)) (justify left bottom))
-  )
-  (label "ULPI_CLK" (at 187.96 127 0) (fields_autoplaced)
-    (effects (font (size 1.27 1.27)) (justify left bottom))
-  )
-  (label "ULPI_DIR" (at 201.93 40.64 180) (fields_autoplaced)
-    (effects (font (size 1.27 1.27)) (justify right bottom))
   )
   (label "ULPI_D6" (at 187.96 144.78 0) (fields_autoplaced)
@@
   )
   (label "ULPI_D7" (at 187.96 147.32 0) (fields_autoplaced)
-    (effects (font (size 1.27 1.27)) (justify left bottom))
-  )
-  (label "ULPI_CLK" (at 201.93 43.18 180) (fields_autoplaced)
-    (effects (font (size 1.27 1.27)) (justify right bottom))
-  )
-  (label "ULPI_NXT" (at 187.96 154.94 0) (fields_autoplaced)
     (effects (font (size 1.27 1.27)) (justify left bottom))
   )
@@
     )
   )
+  (global_label "A12" (shape input) (at 262.89 45.72 0) (fields_autoplaced)
+    (effects (font (size 1.27 1.27)) (justify left))
+    (property "Intersheetrefs" "${INTERSHEET_REFS}" (at 269.3828 45.72 0)
+      (effects (font (size 1.27 1.27)) (justify left) hide)
+    )
+  )
+  (global_label "A11" (shape input) (at 262.89 48.26 0) (fields_autoplaced)
+    (effects (font (size 1.27 1.27)) (justify left))
+    (property "Intersheetrefs" "${INTERSHEET_REFS}" (at 269.3828 48.26 0)
+      (effects (font (size 1.27 1.27)) (justify left) hide)
+    )
+  )
+  (global_label "ULPI_NXT" (shape input) (at 198.12 154.94 0) (fields_autoplaced)
+    (effects (font (size 1.27 1.27)) (justify left))
+    (property "Intersheetrefs" "${INTERSHEET_REFS}" (at 209.8138 154.94 0)
+      (effects (font (size 1.27 1.27)) (justify left) hide)
+    )
+  )
+  (global_label "CKE" (shape input) (at 262.89 43.18 0) (fields_autoplaced)
+    (effects (font (size 1.27 1.27)) (justify left))
+    (property "Intersheetrefs" "${INTERSHEET_REFS}" (at 269.5642 43.18 0)
+      (effects (font (size 1.27 1.27)) (justify left) hide)
+    )
+  )
   (global_label "SDRAM_A4" (shape output) (at 262.89 50.8 0) (fields_autoplaced)
     (effects (font (size 1.27 1.27)) (justify left))
@@
     )
   )
-  (global_label "ULPI_STP" (shape input) (at 187.96 152.4 0) (fields_autoplaced)
+  (global_label "ULPI_STP" (shape input) (at 198.12 152.4 0) (fields_autoplaced)
     (effects (font (size 1.27 1.27)) (justify left))
-    (property "Intersheetrefs" "${INTERSHEET_REFS}" (at 199.5933 152.4 0)
+    (property "Intersheetrefs" "${INTERSHEET_REFS}" (at 209.7533 152.4 0)
       (effects (font (size 1.27 1.27)) (justify left) hide)
     )
+  )
+  (global_label "ULPI_DIR" (shape input) (at 198.12 149.86 0) (fields_autoplaced)
+    (effects (font (size 1.27 1.27)) (justify left))
+    (property "Intersheetrefs" "${INTERSHEET_REFS}" (at 209.451 149.86 0)
+      (effects (font (size 1.27 1.27)) (justify left) hide)
+    )
+  )
+  (global_label "ULPI_CLK" (shape input) (at 198.12 127 0) (fields_autoplaced)
+    (effects (font (size 1.27 1.27)) (justify left))
+    (property "Intersheetrefs" "${INTERSHEET_REFS}" (at 209.8743 127 0)
+      (effects (font (size 1.27 1.27)) (justify left) hide)
+    )

Commit message: Some BOM clarifications and updates
Parts:
- U8: value T8Q144xx -> T20Q144xx
Changed lines of the file:
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@@
       (effects (font (size 1.27 1.27)))
     )
-    (property "Value" "T8Q144xx" (at 232.41 62.5643 0)
+    (property "Value" "T20Q144xx" (at 232.41 62.5643 0)
       (effects (font (size 1.27 1.27)))
     )

Commit message: Added Manufacturer + Part info for most components.
Parts:
- C100, C91: Manufacturer (none) -> TDK; Part (none) -> CGA3E3X5R1H105K080AB
- C100, C59: Manufacturer (none) -> Samsung; Part (none) -> CL10B104KB8NFN
- C52, C53: Manufacturer (none) -> Any; Part (none) -> 10p-603
- C54: Manufacturer (none) -> Any; Part (none) -> 10n-603
- U16: Manufacturer (none) -> Microchip; Part (none) -> USB3343-CP
- U8: Manufacturer (none) -> Efinix; Part (none) -> T20Q144C4
Changed lines of the file:
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@@
+      (effects (font (size 1.27 1.27)) hide)
+    )
+    (property "Manufacturer" "TDK" (at 149.86 99.06 0)
+      (effects (font (size 1.27 1.27)) hide)
+    )
+    (property "Part" "CGA3E3X5R1H105K080AB" (at 149.86 99.06 0)
       (effects (font (size 1.27 1.27)) hide)
     )
@@
       (effects (font (size 1.27 1.27)) hide)
     )
+    (property "Manufacturer" "Any" (at 38.1 151.13 0)
+      (effects (font (size 1.27 1.27)) hide)
+    )
+    (property "Part" "10n-603" (at 38.1 151.13 0)
+      (effects (font (size 1.27 1.27)) hide)
+    )
     (pin "1")
     (pin "2")
@@
       (effects (font (size 1.27 1.27)) hide)
     )
-    (property "Part" "" (at 122.555 109.22 0)
-      (effects (font (size 1.27 1.27)) hide)
-    )
-    (property "Manufacturer" "" (at 125.095 106.68 0)
+    (property "Part" "CL10B104KB8NFN" (at 122.555 109.22 0)
+      (effects (font (size 1.27 1.27)) hide)
+    )
+    (property "Manufacturer" "Samsung" (at 125.095 106.68 0)
       (effects (font (size 1.27 1.27)) hide)
     )
@@
       (effects (font (size 1.27 1.27)) hide)
     )
-    (property "Part" "" (at 160.655 93.98 0)
-      (effects (font (size 1.27 1.27)) hide)
-    )
-    (property "Manufacturer" "" (at 163.195 91.44 0)
+    (property "Part" "CL10B104KB8NFN" (at 160.655 93.98 0)
+      (effects (font (size 1.27 1.27)) hide)
+    )
+    (property "Manufacturer" "Samsung" (at 163.195 91.44 0)
       (effects (font (size 1.27 1.27)) hide)
     )
@@
     )
     (property "Datasheet" "https://www.efinixinc.com/docs/trion8-ds-v4.4.pdf" (at 232.41 74.93 0)
+      (effects (font (size 1.27 1.27)) hide)
+    )
+    (property "Manufacturer" "Efinix" (at 232.41 48.26 0)
+      (effects (font (size 1.27 1.27)) hide)
+    )
+    (property "Part" "T20Q144C4" (at 232.41 48.26 0)
       (effects (font (size 1.27 1.27)) hide)
     )
@@
       (effects (font (size 1.27 1.27)) hide)
     )
+    (property "Manufacturer" "Microchip" (at 149.86 137.16 0)
+      (effects (font (size 1.27 1.27)) hide)
+    )
+    (property "Part" "USB3343-CP" (at 149.86 137.16 0)
+      (effects (font (size 1.27 1.27)) hide)
+    )
     (pin "1")
     (pin "10")
@@
       (effects (font (size 1.27 1.27)) hide)
     )
+    (property "Manufacturer" "Any" (at 113.03 153.67 0)
+      (effects (font (size 1.27 1.27)) hide)
+    )
+    (property "Part" "10p-603" (at 113.03 153.67 0)
+      (effects (font (size 1.27 1.27)) hide)
+    )
     (pin "1")
     (pin "2")
@@
       (effects (font (size 1.27 1.27)) hide)
     )
+    (property "Manufacturer" "Any" (at 100.33 153.67 0)
+      (effects (font (size 1.27 1.27)) hide)
+    )
+    (property "Part" "10p-603" (at 100.33 153.67 0)
+      (effects (font (size 1.27 1.27)) hide)
+    )
     (pin "1")
     (pin "2")
@@
       (effects (font (size 1.27 1.27)) hide)
     )
+    (property "Manufacturer" "TDK" (at 152.4 99.06 0)
+      (effects (font (size 1.27 1.27)) hide)
+    )
+    (property "Part" "CGA3E3X5R1H105K080AB" (at 152.4 99.06 0)
+      (effects (font (size 1.27 1.27)) hide)
+    )
     (pin "1")
     (pin "2")
@@
       (effects (font (size 1.27 1.27)) hide)
     )
+    (property "Manufacturer" "Samsung" (at 220.98 25.4 0)
+      (effects (font (size 1.27 1.27)) hide)
+    )
+    (property "Part" "CL10B104KB8NFN" (at 220.98 25.4 0)
+      (effects (font (size 1.27 1.27)) hide)
+    )
