File: ulpi.kicad_sch (KiCad schematic)
At the start: 20 parts, among them J2 USB_C_Receptacle_USB2.0, U16 USB3343, U8 T20Q144xx, Y1 26MHz

Commit message: reconnected fpgaGpio[0] from pin 36 -> 32 (REF_RES is *not* a GPIO!)
Changed lines of the file:
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@@
     )
   )
-  (global_label "ULPI_NXT" (shape input) (at 198.12 154.94 0) (fields_autoplaced)
+  (global_label "ULPI_NXT" (shape output) (at 198.12 154.94 0) (fields_autoplaced)
     (effects (font (size 1.27 1.27)) (justify left))
     (property "Intersheetrefs" "${INTERSHEET_REFS}" (at 209.8138 154.94 0)
@@
     )
   )
-  (global_label "ULPI_DIR" (shape input) (at 198.12 149.86 0) (fields_autoplaced)
+  (global_label "ULPI_DIR" (shape output) (at 198.12 149.86 0) (fields_autoplaced)
     (effects (font (size 1.27 1.27)) (justify left))
     (property "Intersheetrefs" "${INTERSHEET_REFS}" (at 209.451 149.86 0)
@@
     )
   )
-  (global_label "ULPI_CLK" (shape input) (at 198.12 127 0) (fields_autoplaced)
+  (global_label "ULPI_CLK" (shape output) (at 198.12 127 0) (fields_autoplaced)
     (effects (font (size 1.27 1.27)) (justify left))
     (property "Intersheetrefs" "${INTERSHEET_REFS}" (at 209.8743 127 0)
