File: ethernet.kicad_sch (KiCad schematic)
At the start: 50 parts, among them J1 RJ45_Amphenol_RJMG1BD3B8K1ANR, J2 T8_JTAG, J5 ETH GPIO, U2 dp83640, X1 ECS-2520MV-120-CM

Commit message: Some BOM clarifications and updates
Parts:
- U2: Manufacturer (none) -> Texas Instruments
- X1: value ECS-2520MV-120-CM -> ECS-2520MV-250-CM
Other:
- note added: "JTAG for DP83640 (optional) DNL R54 if JTAG controller does not support TRST"
- note removed: "DNL if JTAG controller does not support TRST"
Changed lines of the file:
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@@
     (effects (font (size 1.27 1.27)) (justify left bottom))
   )
-  (text "DNL if JTAG controller does not\nsupport TRST" (at 132.715 163.83 0)
+  (text "JTAG for DP83640 (optional)\nDNL R54 if JTAG controller does not\nsupport TRST"
+    (at 127.635 163.83 0)
     (effects (font (size 1.27 1.27)) (justify left bottom))
   )
@@
       (effects (font (size 1.27 1.27)))
     )
-    (property "Value" "ECS-2520MV-120-CM" (at 99.695 57.15 0)
+    (property "Value" "ECS-2520MV-250-CM" (at 99.695 57.15 0)
       (effects (font (size 1.27 1.27)))
     )
@@
       (effects (font (size 1.27 1.27)) hide)
     )
+    (property "Manufacturer" "Texas Instruments" (at 95.25 129.54 0)
+      (effects (font (size 1.27 1.27)) hide)
+    )

Commit message: Added Manufacturer + Part info for most components.
Parts:
- C16, C17, C18, C19, C20, C24, C25, C26, C47, C55, C56, C73: Manufacturer (none) -> Samsung; Part (none) -> CL10B104KB8NFN
- C23, C46: Manufacturer (none) -> TDK; Part (none) -> 2012X5R1C475K125AC
- C58, C60: Manufacturer (none) -> Any; Part (none) -> 1n-603
- D11: value LED -> LED-GRN; Manufacturer (none) -> Wurth; Part (none) -> 150060GS75000
- J1: Manufacturer (none) -> Amphenol; Part (none) -> RJMG1BD3B8K1ANR
- J2: Manufacturer (none) -> Adam Tech; Part (none) -> 2PH2-14-UA
- J5: Manufacturer (none) -> Adam Tech; Part (none) -> PH2-20-UA
- L2: Manufacturer (none) -> Laird; Part (none) -> MI0603J601R-10
- U2: Part (none) -> DP83640
- X1: Manufacturer (none) -> ECS; Part (none) -> ECS-2520MV-250-CL-TR
Other:
- note added: "Master-clock mode: load R10, X1, DNL R9 Slave-clock mode: load R9, DNL R10, DNL X1"
- note removed: "Master: load R10, DNL R9 Slave: load R9, DNL R10, X1"
Changed lines of the file:
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@@
     (effects (font (size 1.27 1.27)) (justify left bottom))
   )
-  (text "Master: load R10, DNL R9\nSlave: load R9, DNL R10, X1"
+  (text "Master-clock mode: load R10, X1, DNL R9\nSlave-clock mode: load R9, DNL R10, DNL X1"
     (at 114.3 83.82 0)
     (effects (font (size 1.27 1.27)) (justify left bottom))
@@
       (effects (font (size 1.27 1.27)) hide)
     )
+    (property "Manufacturer" "Samsung" (at 185.42 34.29 0)
+      (effects (font (size 1.27 1.27)) hide)
+    )
+    (property "Part" "CL10B104KB8NFN" (at 185.42 34.29 0)
+      (effects (font (size 1.27 1.27)) hide)
+    )
     (pin "1")
     (pin "2")
@@
       (effects (font (size 1.27 1.27)) hide)
     )
+    (property "Manufacturer" "Any" (at 236.22 62.23 0)
+      (effects (font (size 1.27 1.27)) hide)
+    )
+    (property "Part" "1n-603" (at 236.22 62.23 0)
+      (effects (font (size 1.27 1.27)) hide)
+    )
     (pin "1")
     (pin "2")
@@
       (effects (font (size 1.27 1.27)) hide)
     )
+    (property "Manufacturer" "Samsung" (at 232.41 62.23 0)
+      (effects (font (size 1.27 1.27)) hide)
+    )
+    (property "Part" "CL10B104KB8NFN" (at 232.41 62.23 0)
+      (effects (font (size 1.27 1.27)) hide)
+    )
     (pin "1")
     (pin "2")
@@
       (effects (font (size 1.27 1.27)) hide)
     )
+    (property "Manufacturer" "Samsung" (at 49.53 162.56 0)
+      (effects (font (size 1.27 1.27)) hide)
+    )
+    (property "Part" "CL10B104KB8NFN" (at 49.53 162.56 0)
+      (effects (font (size 1.27 1.27)) hide)
+    )
     (pin "1")
     (pin "2")
@@
     )
     (property "Datasheet" "~" (at 143.51 102.87 0)
+      (effects (font (size 1.27 1.27)) hide)
+    )
+    (property "Manufacturer" "Samsung" (at 143.51 102.87 0)
+      (effects (font (size 1.27 1.27)) hide)
+    )
+    (property "Part" "CL10B104KB8NFN" (at 143.51 102.87 0)
       (effects (font (size 1.27 1.27)) hide)
     )
@@
       (effects (font (size 1.27 1.27)) hide)
     )
+    (property "Manufacturer" "Samsung" (at 214.63 62.23 0)
+      (effects (font (size 1.27 1.27)) hide)
+    )
+    (property "Part" "CL10B104KB8NFN" (at 214.63 62.23 0)
+      (effects (font (size 1.27 1.27)) hide)
+    )
     (pin "1")
     (pin "2")
@@
       (effects (font (size 1.27 1.27)) hide)
     )
+    (property "Manufacturer" "Samsung" (at 166.37 34.29 0)
+      (effects (font (size 1.27 1.27)) hide)
+    )
+    (property "Part" "CL10B104KB8NFN" (at 166.37 34.29 0)
+      (effects (font (size 1.27 1.27)) hide)
+    )
     (pin "1")
     (pin "2")
@@
     )
     (property "Datasheet" "~" (at 40.64 153.67 0)
+      (effects (font (size 1.27 1.27)) hide)
+    )
+    (property "Manufacturer" "Laird" (at 40.64 153.67 0)
+      (effects (font (size 1.27 1.27)) hide)
+    )
+    (property "Part" "MI0603J601R-10" (at 40.64 153.67 0)
       (effects (font (size 1.27 1.27)) hide)
     )
@@
       (effects (font (size 1.27 1.27)) hide)
     )
+    (property "Manufacturer" "Samsung" (at 74.93 95.25 0)
+      (effects (font (size 1.27 1.27)) hide)
+    )
+    (property "Part" "CL10B104KB8NFN" (at 74.93 95.25 0)
+      (effects (font (size 1.27 1.27)) hide)
+    )
     (pin "1")
     (pin "2")
@@
       (effects (font (size 1.27 1.27)))
     )
-    (property "Value" "LED" (at 253.0475 67.7601 0)
+    (property "Value" "LED-GRN" (at 253.0475 67.7601 0)
       (effects (font (size 1.27 1.27)))
     )
@@
     )
     (property "Datasheet" "~" (at 251.46 64.77 0)
+      (effects (font (size 1.27 1.27)) hide)
+    )
+    (property "Manufacturer" "Wurth" (at 251.46 64.77 0)
+      (effects (font (size 1.27 1.27)) hide)
+    )
+    (property "Part" "150060GS75000" (at 251.46 64.77 0)
       (effects (font (size 1.27 1.27)) hide)
     )
@@
       (effects (font (size 1.27 1.27)) hide)
     )
+    (property "Manufacturer" "Samsung" (at 190.5 62.23 0)
+      (effects (font (size 1.27 1.27)) hide)
+    )
+    (property "Part" "CL10B104KB8NFN" (at 190.5 62.23 0)
+      (effects (font (size 1.27 1.27)) hide)
+    )
     (pin "1")
     (pin "2")
@@
     )
     (property "Datasheet" "~" (at 40.64 162.56 0)
+      (effects (font (size 1.27 1.27)) hide)
+    )
+    (property "Manufacturer" "TDK" (at 40.64 162.56 0)
+      (effects (font (size 1.27 1.27)) hide)
+    )
+    (property "Part" "2012X5R1C475K125AC" (at 40.64 162.56 0)
       (effects (font (size 1.27 1.27)) hide)
     )
@@
       (effects (font (size 1.27 1.27)) hide)
     )
+    (property "Manufacturer" "ECS" (at 110.49 43.18 0)
+      (effects (font (size 1.27 1.27)) hide)
+    )
+    (property "Part" "ECS-2520MV-250-CL-TR" (at 110.49 43.18 0)
+      (effects (font (size 1.27 1.27)) hide)
+    )
     (pin "1")
     (pin "2")
@@
       (effects (font (size 1.27 1.27)) hide)
     )
+    (property "Manufacturer" "Samsung" (at 58.42 162.56 0)
+      (effects (font (size 1.27 1.27)) hide)
+    )
+    (property "Part" "CL10B104KB8NFN" (at 58.42 162.56 0)
+      (effects (font (size 1.27 1.27)) hide)
+    )
     (pin "1")
     (pin "2")
@@
     )
     (property "Manufacturer" "Texas Instruments" (at 95.25 129.54 0)
+      (effects (font (size 1.27 1.27)) hide)
+    )
+    (property "Part" "DP83640" (at 95.25 129.54 0)
       (effects (font (size 1.27 1.27)) hide)
     )
@@
       (effects (font (size 1.27 1.27)) hide)
     )
+    (property "Manufacturer" "Samsung" (at 66.04 95.25 0)
+      (effects (font (size 1.27 1.27)) hide)
+    )
+    (property "Part" "CL10B104KB8NFN" (at 66.04 95.25 0)
+      (effects (font (size 1.27 1.27)) hide)
+    )
     (pin "1")
     (pin "2")
@@
       (effects (font (size 1.27 1.27)) hide)
     )
+    (property "Manufacturer" "Samsung" (at 124.46 41.91 0)
+      (effects (font (size 1.27 1.27)) hide)
+    )
+    (property "Part" "CL10B104KB8NFN" (at 124.46 41.91 0)
+      (effects (font (size 1.27 1.27)) hide)
+    )
     (pin "1")
     (pin "2")
@@
       (effects (font (size 1.27 1.27)) hide)
     )
+    (property "Manufacturer" "Any" (at 218.44 62.23 0)
+      (effects (font (size 1.27 1.27)) hide)
+    )
+    (property "Part" "1n-603" (at 218.44 62.23 0)
+      (effects (font (size 1.27 1.27)) hide)
+    )
     (pin "1")
     (pin "2")
@@
       (effects (font (size 1.27 1.27)) hide)
     )
+    (property "Manufacturer" "Samsung" (at 199.39 62.23 0)
+      (effects (font (size 1.27 1.27)) hide)
+    )
+    (property "Part" "CL10B104KB8NFN" (at 199.39 62.23 0)
+      (effects (font (size 1.27 1.27)) hide)
+    )
     (pin "1")
     (pin "2")
@@
     )
     (property "Datasheet" "https://www.amphenol-cs.com/media/wysiwyg/files/drawing/rjmg1bd3b8k1anr.pdf" (at 223.52 31.75 0)
+      (effects (font (size 1.27 1.27)) hide)
+    )
+    (property "Manufacturer" "Amphenol" (at 223.52 46.99 0)
+      (effects (font (size 1.27 1.27)) hide)
+    )
+    (property "Part" "RJMG1BD3B8K1ANR" (at 223.52 46.99 0)
       (effects (font (size 1.27 1.27)) hide)
     )
@@
       (effects (font (size 1.27 1.27)) hide)
     )
+    (property "Manufacturer" "Adam Tech" (at 143.51 179.07 0)
+      (effects (font (size 1.27 1.27)) hide)
+    )
+    (property "Part" "2PH2-14-UA" (at 143.51 179.07 0)
+      (effects (font (size 1.27 1.27)) hide)
+    )
     (pin "3")
     (pin "5")
@@
     )
     (property "Datasheet" "~" (at 36.195 42.545 0)
+      (effects (font (size 1.27 1.27)) hide)
+    )
+    (property "Manufacturer" "Adam Tech" (at 36.195 42.545 0)
+      (effects (font (size 1.27 1.27)) hide)
+    )
+    (property "Part" "PH2-20-UA" (at 36.195 42.545 0)
       (effects (font (size 1.27 1.27)) hide)
     )
@@
       (effects (font (size 1.27 1.27)) hide)
     )
+    (property "Manufacturer" "TDK" (at 57.15 95.25 0)
+      (effects (font (size 1.27 1.27)) hide)
+    )
+    (property "Part" "2012X5R1C475K125AC" (at 57.15 95.25 0)
+      (effects (font (size 1.27 1.27)) hide)
+    )

Commit message: Added GPS receiver; increased board size
including battery supply; made board bigger
and added edge connectors for ETH GPIO, PPS
and antenna.
Parts:
- removed J2: T8_JTAG, Connector_PinHeader_2.00mm:PinHeader_2x07_P2.00mm_Vertical, symbol Connector_Generic:Conn_02x07_Odd_Even
- removed R54: 0, Resistor_SMD:R_0603_1608Metric, symbol Device:R_Small
- removed R55: 10k, Resistor_SMD:R_0603_1608Metric, symbol Device:R_Small
- added J11: IO1, proj_footprints:LEMO+SMA_molex_732515460, symbol Connector:Conn_Coaxial_Small
- added J12: IO2, proj_footprints:LEMO+SMA_molex_732515460, symbol Connector:Conn_Coaxial_Small
- added J13: IO3, proj_footprints:LEMO+SMA_molex_732515460, symbol Connector:Conn_Coaxial_Small
- added J14: IO4, proj_footprints:LEMO+SMA_molex_732515460, symbol Connector:Conn_Coaxial_Small
- added J15: IO8, proj_footprints:LEMO+SMA_molex_732515460, symbol Connector:Conn_Coaxial_Small
- added J16: CLK, proj_footprints:LEMO+SMA_molex_732515460, symbol Connector:Conn_Coaxial_Small
Connections:
- net ETH0_CLK_OUT: now also J16.1 (In)
- net ETH0_GPIO_1: now also J11.1 (In)
- net ETH0_GPIO_2: now also J12.1 (In)
- net ETH0_GPIO_3: now also J13.1 (In)
- net ETH0_GPIO_4: now also J14.1 (In)
- net ETH0_GPIO_8: now also J15.1 (In)
- net GND: now also J11.2 (Ext), J12.2 (Ext), J13.2 (Ext), J14.2 (Ext), J15.2 (Ext), J16.2 (Ext); no longer J5.16 (Pin_16)
- net ETH0_TCK: no longer names the net of U2.8 (TCK)
- net ETH0_TDI renamed GPS_PPS
- net ETH0_TDO renamed ETH0_GPIO_10
- net ETH0_GPIO_10: now also J5.16 (Pin_16)
- net ETH0_TMS: no longer names the net of U2.10 (TMS)
- net ETH0_TRSTb: no longer names the net of U2.11 (TRST#)
- net ETH0_TXD_2: no longer names the net of U2.5 (TXD_2)
- no-connect marks 4 -> 6
Other:
- note removed: "JTAG for DP83640 (optional) DNL R54 if JTAG controller does not support TRST"
- moved on the sheet: C18, X1
