File: ethernet.kicad_sch (KiCad schematic)
At the start: 53 parts, among them J1 RJ45_Amphenol_RJMG1BD3B8K1ANR, J11 IO1, J12 IO2, J13 IO3, J14 IO4, J15 IO8, J16 CLK, J5 ETH GPIO, U2 dp83640, X1 ECS-2520MV-250-CM

Commit message: bumped version to 2.1
updated several values;

* added AC-coupling cap on RF_IN
Parts:
- D11: Part 150060GS75000 -> 155060VS73200
- R6, R7: value 680 -> 249
Changed lines of the file:
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@@
       (effects (font (size 1.27 1.27)) (justify left))
     )
-    (property "Value" "680" (at 252.73 46.99 90)
+    (property "Value" "249" (at 252.73 46.99 90)
       (effects (font (size 1.27 1.27)) (justify left))
     )
@@
       (effects (font (size 1.27 1.27)) hide)
     )
-    (property "Part" "150060GS75000" (at 251.46 64.77 0)
+    (property "Part" "155060VS73200" (at 251.46 64.77 0)
       (effects (font (size 1.27 1.27)) hide)
     )
@@
       (effects (font (size 1.27 1.27)) (justify left))
     )
-    (property "Value" "680" (at 252.73 36.83 90)
-      (effects (font (size 1.27 1.27)) (justify left))
-    )
+    (property "Value" "249" (at 252.73 36.83 90)
+      (effects (font (size 1.27 1.27)) (justify left))
+    )

Commit message: small fixes; prettified the fab layer and added DNP on schematic
Parts:
- R9: now not fitted; now left out of the parts list
Changed lines of the file:
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@@
   )
   (symbol (lib_id "Device:R_Small") (at 115.57 93.98 90) (unit 1)
-    (in_bom yes) (on_board yes) (dnp no)
+    (in_bom no) (on_board yes) (dnp yes)
     (property "Reference" "R9" (at 118.11 91.44 90)
       (effects (font (size 1.27 1.27)) (justify left))
