File: led.kicad_sch (KiCad schematic)
At the start: 19 parts, among them U8 T8Q144xx

Commit message: Fixed V1.0 errata
- added feedback resistor for ulpi transceiver clock oscillator
- removed SS_N connection
Parts:
- renumbered C14 to C57, C14 to C64, D1 to D2, D1 to D3, D1 to D4, D1 to D5, D1 to D6, D1 to D7, D1 to D8, D1 to D9

Commit message: sdram layout done - COMPLETE REWORK NEEDED
cannot mix LVDS and GPIO banks due to too different timing
Parts:
- removed C64: 100n, Capacitor_SMD:C_0603_1608Metric, symbol Device:C_Small
- removed unit 7 of U8
Connections:
- net LED0: now also U8.106 (GPIOR_94_CDI27); no longer U8.100 (GPIOR_113_CDI22)
- net LED1: now also U8.105 (GPIOR_95_CDI26); no longer U8.99 (GPIOR_116_CTRL15)
- net LED2: now also U8.103 (GPIOR_104_CDI25)
- net LED3: now also U8.102 (GPIOR_105_CDI24)
- net LED4: now also U8.101 (GPIOR_112_CDI23)
- net LED5: now also U8.100 (GPIOR_113_CDI22)
- net LED6: now also U8.99 (GPIOR_116_CTRL15)
- net LED7: now also U8.98 (GPIOR_117_CTRL14)
- no-connect marks 12 -> 2
Other:
- moved on the sheet: D2, D3, D4, D5, D6, D7, D8, D9, R4, U8F

Commit message: layout finished; passed all checks...
Parts:
- removed C57: 100n, Capacitor_SMD:C_0603_1608Metric, symbol Device:C_Small
- removed U8: T8Q144xx, Package_QFP:LQFP-144_20x20mm_P0.5mm, symbol FPGA_Efinix_Trion:T8Q144xx
Connections:
- no-connect marks 2 -> 0

Commit message: Added Manufacturer + Part info for most components.
Parts:
- D2, D4, D6, D8: value LED -> LED-GRN; Manufacturer (none) -> Wurth; Part (none) -> 150060GS75000
- D3, D5, D7, D9: value LED -> LED-RED; Manufacturer (none) -> Wurth; Part (none) -> 150060RS75000
Changed lines of the file:
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@@
       (effects (font (size 1.27 1.27)))
     )
-    (property "Value" "LED" (at 126.6825 112.5799 0)
+    (property "Value" "LED-GRN" (at 126.6825 112.5799 0)
       (effects (font (size 1.27 1.27)))
     )
@@
       (effects (font (size 1.27 1.27)) hide)
     )
+    (property "Manufacturer" "Wurth" (at 128.27 115.57 0)
+      (effects (font (size 1.27 1.27)) hide)
+    )
+    (property "Part" "150060GS75000" (at 128.27 115.57 0)
+      (effects (font (size 1.27 1.27)) hide)
+    )
     (pin "1")
     (pin "2")
@@
       (effects (font (size 1.27 1.27)))
     )
-    (property "Value" "LED" (at 126.6825 102.4199 0)
+    (property "Value" "LED-RED" (at 126.6825 102.4199 0)
       (effects (font (size 1.27 1.27)))
     )
@@
       (effects (font (size 1.27 1.27)) hide)
     )
+    (property "Manufacturer" "Wurth" (at 128.27 105.41 0)
+      (effects (font (size 1.27 1.27)) hide)
+    )
+    (property "Part" "150060RS75000" (at 128.27 105.41 0)
+      (effects (font (size 1.27 1.27)) hide)
+    )
     (pin "1")
     (pin "2")
@@
       (effects (font (size 1.27 1.27)))
     )
-    (property "Value" "LED" (at 126.6825 71.9399 0)
+    (property "Value" "LED-GRN" (at 126.6825 71.9399 0)
       (effects (font (size 1.27 1.27)))
     )
@@
       (effects (font (size 1.27 1.27)) hide)
     )
+    (property "Manufacturer" "Wurth" (at 128.27 74.93 0)
+      (effects (font (size 1.27 1.27)) hide)
+    )
+    (property "Part" "150060GS75000" (at 128.27 74.93 0)
+      (effects (font (size 1.27 1.27)) hide)
+    )
     (pin "1")
     (pin "2")
@@
       (effects (font (size 1.27 1.27)))
     )
-    (property "Value" "LED" (at 126.6825 121.4699 0)
+    (property "Value" "LED-RED" (at 126.6825 121.4699 0)
       (effects (font (size 1.27 1.27)))
     )
@@
       (effects (font (size 1.27 1.27)) hide)
     )
+    (property "Manufacturer" "Wurth" (at 128.27 124.46 0)
+      (effects (font (size 1.27 1.27)) hide)
+    )
+    (property "Part" "150060RS75000" (at 128.27 124.46 0)
+      (effects (font (size 1.27 1.27)) hide)
+    )
     (pin "1")
     (pin "2")
@@
       (effects (font (size 1.27 1.27)))
     )
-    (property "Value" "LED" (at 126.6825 132.8999 0)
+    (property "Value" "LED-GRN" (at 126.6825 132.8999 0)
       (effects (font (size 1.27 1.27)))
     )
@@
       (effects (font (size 1.27 1.27)) hide)
     )
+    (property "Manufacturer" "Wurth" (at 128.27 135.89 0)
+      (effects (font (size 1.27 1.27)) hide)
+    )
+    (property "Part" "150060GS75000" (at 128.27 135.89 0)
+      (effects (font (size 1.27 1.27)) hide)
+    )
     (pin "1")
     (pin "2")
@@
       (effects (font (size 1.27 1.27)))
     )
-    (property "Value" "LED" (at 126.6825 92.2599 0)
+    (property "Value" "LED-GRN" (at 126.6825 92.2599 0)
       (effects (font (size 1.27 1.27)))
     )
@@
       (effects (font (size 1.27 1.27)) hide)
     )
+    (property "Manufacturer" "Wurth" (at 128.27 95.25 0)
+      (effects (font (size 1.27 1.27)) hide)
+    )
+    (property "Part" "150060GS75000" (at 128.27 95.25 0)
+      (effects (font (size 1.27 1.27)) hide)
+    )
     (pin "1")
     (pin "2")
@@
       (effects (font (size 1.27 1.27)))
     )
-    (property "Value" "LED" (at 126.6825 83.3699 0)
+    (property "Value" "LED-RED" (at 126.6825 83.3699 0)
       (effects (font (size 1.27 1.27)))
     )
@@
       (effects (font (size 1.27 1.27)) hide)
     )
+    (property "Manufacturer" "Wurth" (at 128.27 86.36 0)
+      (effects (font (size 1.27 1.27)) hide)
+    )
+    (property "Part" "150060RS75000" (at 128.27 86.36 0)
+      (effects (font (size 1.27 1.27)) hide)
+    )
     (pin "1")
     (pin "2")
@@
       (effects (font (size 1.27 1.27)))
     )
-    (property "Value" "LED" (at 126.6825 143.0599 0)
+    (property "Value" "LED-RED" (at 126.6825 143.0599 0)
       (effects (font (size 1.27 1.27)))
     )
@@
       (effects (font (size 1.27 1.27)) hide)
     )
+    (property "Manufacturer" "Wurth" (at 128.27 146.05 0)
+      (effects (font (size 1.27 1.27)) hide)
+    )
+    (property "Part" "150060RS75000" (at 128.27 146.05 0)
+      (effects (font (size 1.27 1.27)) hide)
+    )

Commit message: Added GPS receiver; increased board size
including battery supply; made board bigger
and added edge connectors for ETH GPIO, PPS
and antenna.
Parts:
- removed D2, D4, D6, D8: LED-GRN, LED_SMD:LED_0603_1608Metric, symbol Device:LED
- removed D3, D5, D7, D9: LED-RED, LED_SMD:LED_0603_1608Metric, symbol Device:LED
- added D1, D2, D3, D4: LED_Dual_RAG, proj_footprints:LED_Wuerth_Sideview, symbol Device:LED_Dual_KAK
Connections:
- net +3V3: now also D1.2 (A), D2.2 (A), D3.2 (A), D4.2 (A); no longer R4.2, R4.2, R4.2, R4.2, R4.2, R4.2, R4.2, R4.2
- net LED0: now also R4.1
- net LED1: now also R4.1
- net LED2: now also R4.1
- net LED3: now also R4.1
- net LED4: now also R4.1
- net LED5: now also R4.1
- net LED6: now also R4.1
- net LED7: now also R4.1
- new net: D1.1 (K1), R4.2
- new net: D1.3 (K2), R4.2
- new net: D3.3 (K2), R4.2
- new net: D4.1 (K1), R4.2
- new net: D4.3 (K2), R4.2
- new net: D2.3 (K2), R4.2
- new net: D2.1 (K1), R4.2
- new net: D3.1 (K1), R4.2
Other:
- note added: "GRN"
- note added: "RED"
- moved on the sheet: R4
