File: power.kicad_sch (KiCad schematic)
At the start: 18 parts, among them U3 RT8096B

Commit message: sdram layout done - COMPLETE REWORK NEEDED
cannot mix LVDS and GPIO banks due to too different timing
Other:
- moved on the sheet: C16, C3, D1, L3, R1, R4, R72, R8, U3

Commit message: Some BOM clarifications and updates
Other:
- note added: "LED: power-good indicator"
Changed lines of the file:
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@@
     (stroke (width 0) (type default))
+  )
+  (text "LED: power-good indicator" (at 100.33 115.57 0)
+    (effects (font (size 1.27 1.27)) (justify left bottom))
   )
   (symbol (lib_id "Device:R_Small") (at 129.54 46.99 90) (unit 1)

Commit message: Added Manufacturer + Part info for most components.
Parts:
- C16, C3: Manufacturer (none) -> Samsung; Part (none) -> CL31A106KPHNNNE
- D1: value LED -> LED-GRN; Manufacturer (none) -> Wurth; Part (none) -> 150060GS75000
- L3: Manufacturer (none) -> Murata; Part (none) -> 1239AS-H-1R5M=P2
Other:
- note added: "NOTE - regarding zero-Ohm resistors: I usually load these only *after* building the board and verifying that the voltages are correct and that no short-circuit is present downstream of these jumpers."
Changed lines of the file:
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@@
+    (effects (font (size 1.27 1.27)) (justify left bottom))
+  )
+  (text "NOTE - regarding zero-Ohm resistors:\nI usually load these only *after*\nbuilding the board and verifying that\nthe voltages are correct and that no\nshort-circuit is present downstream\nof these jumpers."
+    (at 124.46 72.39 0)
     (effects (font (size 1.27 1.27)) (justify left bottom))
   )
@@
       (effects (font (size 1.27 1.27)) hide)
     )
-    (property "Part" "" (at 67.31 87.63 0)
-      (effects (font (size 1.27 1.27)) hide)
-    )
-    (property "Manufacturer" "" (at 67.31 87.63 0)
+    (property "Part" "CL31A106KPHNNNE" (at 67.31 87.63 0)
+      (effects (font (size 1.27 1.27)) hide)
+    )
+    (property "Manufacturer" "Samsung" (at 67.31 87.63 0)
       (effects (font (size 1.27 1.27)) hide)
     )
@@
       (effects (font (size 1.27 1.27)) hide)
     )
-    (property "Part" "" (at 120.65 52.07 0)
-      (effects (font (size 1.27 1.27)) hide)
-    )
-    (property "Manufacturer" "" (at 120.65 52.07 0)
+    (property "Part" "CL31A106KPHNNNE" (at 120.65 52.07 0)
+      (effects (font (size 1.27 1.27)) hide)
+    )
+    (property "Manufacturer" "Samsung" (at 120.65 52.07 0)
       (effects (font (size 1.27 1.27)) hide)
     )
@@
       (effects (font (size 1.27 1.27)) hide)
     )
-    (property "Part" "" (at 111.76 52.07 0)
-      (effects (font (size 1.27 1.27)) hide)
-    )
-    (property "Manufacturer" "" (at 111.76 52.07 0)
+    (property "Part" "CL31A106KPHNNNE" (at 111.76 52.07 0)
+      (effects (font (size 1.27 1.27)) hide)
+    )
+    (property "Manufacturer" "Samsung" (at 111.76 52.07 0)
       (effects (font (size 1.27 1.27)) hide)
     )
@@
       (effects (font (size 1.27 1.27)) hide)
     )
-    (property "Part" "" (at 97.79 46.99 90)
-      (effects (font (size 1.27 1.27)) hide)
-    )
-    (property "Manufacturer" "" (at 97.79 46.99 90)
+    (property "Part" "1239AS-H-1R5M=P2" (at 97.79 46.99 90)
+      (effects (font (size 1.27 1.27)) hide)
+    )
+    (property "Manufacturer" "Murata" (at 97.79 46.99 90)
       (effects (font (size 1.27 1.27)) hide)
     )
@@
       (effects (font (size 1.27 1.27)) hide)
     )
-    (property "Part" "" (at 111.76 90.17 0)
-      (effects (font (size 1.27 1.27)) hide)
-    )
-    (property "Manufacturer" "" (at 111.76 90.17 0)
+    (property "Part" "CL31A106KPHNNNE" (at 111.76 90.17 0)
+      (effects (font (size 1.27 1.27)) hide)
+    )
+    (property "Manufacturer" "Samsung" (at 111.76 90.17 0)
       (effects (font (size 1.27 1.27)) hide)
     )
@@
       (effects (font (size 1.27 1.27)))
     )
-    (property "Value" "LED" (at 110.1725 103.6899 0)
+    (property "Value" "LED-GRN" (at 110.1725 103.6899 0)
       (effects (font (size 1.27 1.27)))
     )
@@
       (effects (font (size 1.27 1.27)) hide)
     )
+    (property "Manufacturer" "Wurth" (at 111.76 106.68 0)
+      (effects (font (size 1.27 1.27)) hide)
+    )
+    (property "Part" "150060GS75000" (at 111.76 106.68 0)
+      (effects (font (size 1.27 1.27)) hide)
+    )
     (pin "1")
     (pin "2")
@@
       (effects (font (size 1.27 1.27)) hide)
     )
-    (property "Part" "" (at 67.31 49.53 0)
-      (effects (font (size 1.27 1.27)) hide)
-    )
-    (property "Manufacturer" "" (at 67.31 49.53 0)
+    (property "Part" "CL31A106KPHNNNE" (at 67.31 49.53 0)
+      (effects (font (size 1.27 1.27)) hide)
+    )
+    (property "Manufacturer" "Samsung" (at 67.31 49.53 0)
       (effects (font (size 1.27 1.27)) hide)
     )
@@
       (effects (font (size 1.27 1.27)) hide)
     )
-    (property "Part" "" (at 97.79 85.09 90)
-      (effects (font (size 1.27 1.27)) hide)
-    )
-    (property "Manufacturer" "" (at 97.79 85.09 90)
-      (effects (font (size 1.27 1.27)) hide)
-    )
+    (property "Part" "1239AS-H-1R5M=P2" (at 97.79 85.09 90)
+      (effects (font (size 1.27 1.27)) hide)
+    )
+    (property "Manufacturer" "Murata" (at 97.79 85.09 90)
+      (effects (font (size 1.27 1.27)) hide)
+    )

Commit message: Added GPS receiver; increased board size
including battery supply; made board bigger
and added edge connectors for ETH GPIO, PPS
and antenna.
Parts:
- removed D1: LED-GRN, LED_SMD:LED_0603_1608Metric, symbol Device:LED
- removed R4: 1k, Resistor_SMD:R_0603_1608Metric, symbol Device:R_Small
Connections:
- net POWER_GOOD: now reaches U3.5 (PG)
- no-connect marks 1 -> 0
Other:
- note removed: "LED: power-good indicator"
Changed lines of the file:
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@@
   (junction (at 111.76 46.99) (diameter 0) (color 0 0 0 0)
   )
-  (junction (at 90.17 96.52) (diameter 0) (color 0 0 0 0)
-  )
   (junction (at 93.98 58.42) (diameter 0) (color 0 0 0 0)
   )
@@
   (junction (at 67.31 85.09) (diameter 0) (color 0 0 0 0)
   )
-  (no_connect (at 90.17 90.17))
   (wire (pts (xy 67.31 90.17) (xy 67.31 96.52))
     (stroke (width 0) (type default))
@@
     (stroke (width 0) (type default))
   )
-  (wire (pts (xy 120.65 106.68) (xy 115.57 106.68))
-    (stroke (width 0) (type default))
-  )
   (wire (pts (xy 132.08 85.09) (xy 137.16 85.09))
     (stroke (width 0) (type default))
@@
     (stroke (width 0) (type default))
   )
-  (wire (pts (xy 82.55 96.52) (xy 90.17 96.52))
+  (wire (pts (xy 82.55 96.52) (xy 93.98 96.52))
     (stroke (width 0) (type default))
   )
@@
     (stroke (width 0) (type default))
   )
+  (wire (pts (xy 90.17 90.17) (xy 90.17 102.87))
+    (stroke (width 0) (type default))
+  )
   (wire (pts (xy 71.12 71.12) (xy 71.12 68.58))
     (stroke (width 0) (type default))
@@
     (stroke (width 0) (type default))
   )
-  (wire (pts (xy 90.17 96.52) (xy 90.17 106.68))
-    (stroke (width 0) (type default))
-  )
   (wire (pts (xy 71.12 87.63) (xy 74.93 87.63))
     (stroke (width 0) (type default))
@@
     (stroke (width 0) (type default))
   )
-  (wire (pts (xy 90.17 106.68) (xy 102.87 106.68))
-    (stroke (width 0) (type default))
-  )
   (wire (pts (xy 67.31 46.99) (xy 63.5 46.99))
     (stroke (width 0) (type default))
@@
     (stroke (width 0) (type default))
   )
-  (wire (pts (xy 120.65 104.14) (xy 120.65 106.68))
-    (stroke (width 0) (type default))
-  )
-  (wire (pts (xy 90.17 96.52) (xy 93.98 96.52))
-    (stroke (width 0) (type default))
-  )
   (wire (pts (xy 93.98 95.25) (xy 93.98 96.52))
     (stroke (width 0) (type default))
@@
   (wire (pts (xy 120.65 46.99) (xy 127 46.99))
     (stroke (width 0) (type default))
-  )
-  (text "LED: power-good indicator" (at 100.33 115.57 0)
-    (effects (font (size 1.27 1.27)) (justify left bottom))
   )
   (text "NOTE - regarding zero-Ohm resistors:\nI usually load these only *after*\nbuilding the board and verifying that\nthe voltages are correct and that no\nshort-circuit is present downstream\nof these jumpers."
@@
     (effects (font (size 1.27 1.27)) (justify left bottom))
   )
+  (global_label "POWER_GOOD" (shape output) (at 90.17 102.87 270) (fields_autoplaced)
+    (effects (font (size 1.27 1.27)) (justify right))
+    (property "Intersheetrefs" "${INTERSHEET_REFS}" (at 90.17 118.4947 90)
+      (effects (font (size 1.27 1.27)) (justify right) hide)
+    )
+  )
   (symbol (lib_id "Device:R_Small") (at 129.54 46.99 90) (unit 1)
     (in_bom yes) (on_board yes) (dnp no)
@@
         (path "/8c6e15e3-1804-4f03-8a4f-3cb8420d9169/156952d1-5d11-4286-b02e-ddefbba25fea"
           (reference "R59") (unit 1)
-        )
-      )
-    )
-  )
-  (symbol (lib_id "Device:R_Small") (at 105.41 106.68 90) (unit 1)
-    (in_bom yes) (on_board yes) (dnp no)
-    (property "Reference" "R4" (at 104.2416 105.1814 0)
-      (effects (font (size 1.27 1.27)) (justify left))
-    )
-    (property "Value" "1k" (at 106.553 105.1814 0)
-      (effects (font (size 1.27 1.27)) (justify left))
-    )
-    (property "Footprint" "Resistor_SMD:R_0603_1608Metric" (at 105.41 106.68 0)
-      (effects (font (size 1.27 1.27)) hide)
-    )
-    (property "Datasheet" "~" (at 105.41 106.68 0)
-      (effects (font (size 1.27 1.27)) hide)
-    )
-    (property "Part" "" (at 105.41 106.68 0)
-      (effects (font (size 1.27 1.27)) hide)
-    )
-    (property "Manufacturer" "" (at 105.41 106.68 0)
-      (effects (font (size 1.27 1.27)) hide)
-    )
-    (pin "1")
-    (pin "2")
-    (instances
-      (project "usbadc"
-        (path "/7c8a1f8d-8834-4c9b-aaae-1f231e9b09a1/00000000-0000-0000-0000-00006086f2e3"
-          (reference "R4") (unit 1)
-        )
-      )
-      (project "trion-8-test"
-        (path "/8c6e15e3-1804-4f03-8a4f-3cb8420d9169/156952d1-5d11-4286-b02e-ddefbba25fea"
-          (reference "R64") (unit 1)
         )
       )
@@
     )
   )
-  (symbol (lib_id "power:+3V3") (at 120.65 104.14 0) (mirror y) (unit 1)
-    (in_bom yes) (on_board yes) (dnp no) (fields_autoplaced)
-    (property "Reference" "#PWR0118" (at 120.65 107.95 0)
-      (effects (font (size 1.27 1.27)) hide)
-    )
-    (property "Value" "+3V3" (at 120.65 100.0069 0)
-      (effects (font (size 1.27 1.27)))
-    )
-    (property "Footprint" "" (at 120.65 104.14 0)
-      (effects (font (size 1.27 1.27)) hide)
-    )
-    (property "Datasheet" "" (at 120.65 104.14 0)
-      (effects (font (size 1.27 1.27)) hide)
-    )
-    (pin "1")
-    (instances
-      (project "trion-8-test"
-        (path "/8c6e15e3-1804-4f03-8a4f-3cb8420d9169/156952d1-5d11-4286-b02e-ddefbba25fea"
-          (reference "#PWR0118") (unit 1)
-        )
-      )
-    )
-  )
   (symbol (lib_id "Regulator_Switching:TLV62569DDC") (at 82.55 49.53 0) (unit 1)
     (in_bom yes) (on_board yes) (dnp no)
@@
         )
       )
-    )
-  )
-  (symbol (lib_id "Device:LED") (at 111.76 106.68 0) (unit 1)
-    (in_bom yes) (on_board yes) (dnp no) (fields_autoplaced)
-    (property "Reference" "D1" (at 110.1725 101.2657 0)
-      (effects (font (size 1.27 1.27)))
-    )
-    (property "Value" "LED-GRN" (at 110.1725 103.6899 0)
-      (effects (font (size 1.27 1.27)))
-    )
-    (property "Footprint" "LED_SMD:LED_0603_1608Metric" (at 111.76 106.68 0)
-      (effects (font (size 1.27 1.27)) hide)
-    )
-    (property "Datasheet" "~" (at 111.76 106.68 0)
-      (effects (font (size 1.27 1.27)) hide)
-    )
-    (property "Manufacturer" "Wurth" (at 111.76 106.68 0)
-      (effects (font (size 1.27 1.27)) hide)
-    )
-    (property "Part" "150060GS75000" (at 111.76 106.68 0)
-      (effects (font (size 1.27 1.27)) hide)
-    )
-    (pin "1")
-    (pin "2")
-    (instances
-      (project "trion-8-test"
-        (path "/8c6e15e3-1804-4f03-8a4f-3cb8420d9169/156952d1-5d11-4286-b02e-ddefbba25fea"
-          (reference "D1") (unit 1)
-        )
-      )
