File: sdram.kicad_sch (KiCad schematic)
At the start: 20 parts, among them U1 MT48LC16M16A2P, U8 T8Q144xx

Commit message: layout finished; passed all checks...
Parts:
- removed unit 10 of U8
- removed unit 9 of U8
- added C15, C3, C57: 100n, Capacitor_SMD:C_0603_1608Metric, symbol Device:C_Small
- added R1: 10k, Resistor_SMD:R_0603_1608Metric, symbol Device:R_Small
- added unit 6 of U8
- added unit 3 of U8
- added unit 4 of U8
- added unit 2 of U8
- added X2: ECS-2520MV-120-CM, Oscillator:Oscillator_SMD_ECS_2520MV-xxx-xx-4Pin_2.5x2.0mm, symbol Oscillator:ECS-2520MV-xxx-xx
Connections:
- net +3V3: now also C15.1, C3.1, C57.1, R1.1, U8.12 (VCCIO1C_1D), U8.143 (VCCIO1E), U8.21 (VCCIO1B), U8.95 (VCCIO3B_3C), X2.1 (Tri-State), X2.4 (VDD)
- net A0: now also U8.137 (GPIOL_70_CBSEL0); no longer U8.86 (GPIOR_133_CDI18)
- net A1: now also U8.134 (GPIOL_73_EXTFB1_CDI15); no longer U8.84 (GPIOR_135_CDI17)
- net A10: now also U8.131 (GPIOL_75_PLLIN1); no longer U8.87 (GPIOR_132_CDI19)
- net A11: now also U8.101 (GPIOR_112_CDI23)
- net A12: now also U8.100 (GPIOR_113_CDI22)
- net A2: now also U8.135 (GPIOL_72_EXTFB0_CDI14); no longer U8.83 (GPIOR_136_CDI16)
- net A3: now also U8.136 (GPIOL_71_NSTATUS); no longer U8.82 (GPIOR_138)
- net A6: now also U8.106 (GPIOR_94_CDI27); no longer U8.75 (GPIOR_157_PLLIN)
- net A7: now also U8.105 (GPIOR_95_CDI26)
- net A8: now also U8.103 (GPIOR_104_CDI25); no longer R30.2, U8.74 (GPIOR_158_TEST_N)
- net A9: now also U8.102 (GPIOR_105_CDI24)
- net BA0: now also U8.4 (GPIOL_54_CDI11); no longer U8.81 (GPIOR_139)
- net BA1: now also U8.3 (GPIOL_53_CDI10); no longer U8.89 (GPIOR_129_CTRL10)
- net CASb: now also U8.8 (GPIOL_40_CDI8)
- net CKE: now also U8.99 (GPIOR_116_CTRL15)
- net CLK: now also U8.98 (GPIOR_117_CTRL14)
- net CSb: now also R1.2, U8.6 (GPIOL_46); no longer R22.2, U8.80 (GPIOR_149_CBUS2)
- net DQ1: now also U8.20 (GPIOL_12_CDI2)
- net DQ10: now also U8.89 (GPIOR_129_CTRL10)
- net DQ11: now also U8.87 (GPIOR_132_CDI19)
- net DQ12: now also U8.86 (GPIOR_133_CDI18)
- net DQ13: now also U8.81 (GPIOR_139)
- net DQ14: now also U8.77 (GPIOR_154)
- net DQ15: now also U8.76 (GPIOR_155)
- net DQ2: now also U8.19 (GPIOL_13_CDI3)
- net DQ3: now also U8.18 (GPIOL_20_CTRL0_CDI4)
- net DQ4: now also U8.17 (GPIOL_21_CTRL1_CDI5)
- net DQ5: now also U8.16 (GPIOL_22_CTRL2)
- net DQ6: now also U8.15 (GPIOL_24_CLK0)
- net DQ7: now also U8.14 (GPIOL_25_CLK1)
- net DQ8: now also U8.93 (GPIOR_123_CLK12_CDI20)
- net DQ9: now also U8.90 (GPIOR_128_CTRL11)
- net DQMH: now also U8.97 (GPIOR_122_CLK13_CDI21)
- net DQML: now also U8.11 (GPIOL_31_CLK7_CDI6)
- net GND: now also C15.2, C3.2, C57.2, X2.2 (GND)
- net RASb: now also U8.7 (GPIOL_41_CDI9); no longer R23.2, U8.79 (GPIOR_150_CBUS1)
- net WEb: now also U8.10 (GPIOL_32_CTRL4_CDI7)
- net LED6: now reaches R24.2, U8.78 (GPIOR_151_CBUS0)
- net LED0: now reaches U8.92 (GPIOR_125_CLK10)
- net A4 renamed SDRAM_A4
- net SDRAM_A4: no longer U8.76 (GPIOR_155)
- net A5 renamed SDRAM_A5
- net SDRAM_A5: no longer U8.77 (GPIOR_154)
- net DQ0 renamed SDRAM_DQ0
- new net: U8.75 (GPIOR_157_PLLIN), X2.3 (OUT)
- new net LED1: U8.84 (GPIOR_135_CDI17)
- new net LED2: U8.83 (GPIOR_136_CDI16)
- new net LED3: U8.82 (GPIOR_138)
- new net LED4: R22.2, U8.80 (GPIOR_149_CBUS2)
- new net LED5: R23.2, U8.79 (GPIOR_150_CBUS1)
- new net LED7: R30.2, U8.74 (GPIOR_158_TEST_N)
- new net ULPI_RSTb: U8.138 (GPIOL_69_CBSEL1)
- new net ULPI_STP: U8.132 (GPIOL_74_PLLIN0)
- no-connect marks 3 -> 5
Other:
- moved on the sheet: R30, U8G

Commit message: rerouted some SDRAM pins to 139,140,141,142,144
Preparation for moving ULPI to free up some DDIO pins
on the other side of the package...
Connections:
- net A0: now also U8.144 (GPIOL_64); no longer U8.137 (GPIOL_70_CBSEL0)
- net A1: now also U8.139 (GPIOL_68); no longer U8.134 (GPIOL_73_EXTFB1_CDI15)
- net A10: now also U8.142 (GPIOL_66_CDI12); no longer U8.131 (GPIOL_75_PLLIN1)
- net A2: now also U8.140 (GPIOL_67_CDI13); no longer U8.135 (GPIOL_72_EXTFB0_CDI14)
- net A3: now also U8.141 (GPIOL_65); no longer U8.136 (GPIOL_71_NSTATUS)
Changed lines of the file:
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@@
   (junction (at 74.93 40.64) (diameter 0) (color 0 0 0 0)
   )
-  (no_connect (at 158.75 110.49))
-  (no_connect (at 158.75 113.03))
-  (no_connect (at 158.75 118.11))
-  (no_connect (at 158.75 120.65))
-  (no_connect (at 158.75 115.57))
+  (no_connect (at 219.71 123.19))
+  (no_connect (at 219.71 113.03))
+  (no_connect (at 219.71 115.57))
+  (no_connect (at 219.71 118.11))
+  (no_connect (at 219.71 110.49))
   (wire (pts (xy 107.95 168.91) (xy 128.27 168.91))
     (stroke (width 0) (type default))
@@
     (effects (font (size 1.27 1.27)) (justify left bottom))
   )
-  (label "A1" (at 219.71 118.11 0) (fields_autoplaced)
-    (effects (font (size 1.27 1.27)) (justify left bottom))
+  (label "A1" (at 158.75 120.65 180) (fields_autoplaced)
+    (effects (font (size 1.27 1.27)) (justify right bottom))
   )
   (label "A3" (at 44.45 73.66 180) (fields_autoplaced)
@@
     (effects (font (size 1.27 1.27)) (justify right bottom))
   )
-  (label "A10" (at 219.71 123.19 0) (fields_autoplaced)
-    (effects (font (size 1.27 1.27)) (justify left bottom))
+  (label "A10" (at 158.75 115.57 180) (fields_autoplaced)
+    (effects (font (size 1.27 1.27)) (justify right bottom))
   )
   (label "DQ12" (at 160.02 156.21 180) (fields_autoplaced)
@@
     (effects (font (size 1.27 1.27)) (justify right bottom))
   )
-  (label "A2" (at 219.71 115.57 0) (fields_autoplaced)
-    (effects (font (size 1.27 1.27)) (justify left bottom))
+  (label "A2" (at 158.75 118.11 180) (fields_autoplaced)
+    (effects (font (size 1.27 1.27)) (justify right bottom))
   )
   (label "A11" (at 44.45 93.98 180) (fields_autoplaced)
@@
     (effects (font (size 1.27 1.27)) (justify right bottom))
   )
-  (label "A3" (at 219.71 113.03 0) (fields_autoplaced)
-    (effects (font (size 1.27 1.27)) (justify left bottom))
+  (label "A3" (at 158.75 113.03 180) (fields_autoplaced)
+    (effects (font (size 1.27 1.27)) (justify right bottom))
   )
   (label "BA0" (at 215.9 87.63 0) (fields_autoplaced)
@@
     (effects (font (size 1.27 1.27)) (justify right bottom))
   )
-  (label "A0" (at 219.71 110.49 0) (fields_autoplaced)
-    (effects (font (size 1.27 1.27)) (justify left bottom))
+  (label "A0" (at 158.75 110.49 180) (fields_autoplaced)
+    (effects (font (size 1.27 1.27)) (justify right bottom))
   )
   (label "DQ14" (at 52.07 173.99 180) (fields_autoplaced)

Commit message: added ethernet phy
Connections:
- net A11: no longer U8.101 (GPIOR_112_CDI23)
- net A12: no longer U8.100 (GPIOR_113_CDI22)
- net CKE: no longer U8.99 (GPIOR_116_CTRL15)
- net DQ10: now also U8.97 (GPIOR_122_CLK13_CDI21); no longer U8.89 (GPIOR_129_CTRL10)
- net DQ15: now also R30.2, U8.74 (GPIOR_158_TEST_N); no longer U8.76 (GPIOR_155)
- net DQ8: now also U8.100 (GPIOR_113_CDI22); no longer U8.93 (GPIOR_123_CLK12_CDI20)
- net DQ9: now also U8.99 (GPIOR_116_CTRL15); no longer U8.90 (GPIOR_128_CTRL11)
- net DQMH: now also U8.101 (GPIOR_112_CDI23); no longer U8.97 (GPIOR_122_CLK13_CDI21)
- net LED7: now also U8.76 (GPIOR_155); no longer R30.2, U8.74 (GPIOR_158_TEST_N)
- net ULPI_STP: now also U8.135 (GPIOL_72_EXTFB0_CDI14); no longer U8.132 (GPIOL_74_PLLIN0)
- net ULPI_NXT: now reaches U8.131 (GPIOL_75_PLLIN1)
- net ULPI_DIR: now reaches U8.134 (GPIOL_73_EXTFB1_CDI15)
- new net FPGA_B3_IO_0: U8.93 (GPIOR_123_CLK12_CDI20)
- new net FPGA_B3_IO_1: U8.90 (GPIOR_128_CTRL11)
- new net FPGA_B3_IO_2: U8.89 (GPIOR_129_CTRL10)
- new net ULPI_CLK: U8.132 (GPIOL_74_PLLIN0)
- no-connect marks 5 -> 2
Changed lines of the file:
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@@
   (junction (at 74.93 40.64) (diameter 0) (color 0 0 0 0)
   )
-  (no_connect (at 219.71 123.19))
   (no_connect (at 219.71 113.03))
-  (no_connect (at 219.71 115.57))
-  (no_connect (at 219.71 118.11))
   (no_connect (at 219.71 110.49))
   (wire (pts (xy 107.95 168.91) (xy 128.27 168.91))
@@
     (stroke (width 0) (type default))
   )
+  (wire (pts (xy 116.84 166.37) (xy 107.95 166.37))
+    (stroke (width 0) (type default))
+  )
   (wire (pts (xy 74.93 40.64) (xy 80.01 40.64))
     (stroke (width 0) (type default))
@@
     (effects (font (size 1.27 1.27)) (justify right bottom))
   )
-  (label "CKE" (at 148.59 90.17 0) (fields_autoplaced)
-    (effects (font (size 1.27 1.27)) (justify left bottom))
-  )
   (label "DQ11" (at 160.02 153.67 180) (fields_autoplaced)
     (effects (font (size 1.27 1.27)) (justify right bottom))
@@
     (effects (font (size 1.27 1.27)) (justify right bottom))
   )
-  (label "A11" (at 44.45 93.98 180) (fields_autoplaced)
-    (effects (font (size 1.27 1.27)) (justify right bottom))
-  )
   (label "DQMH" (at 44.45 111.76 180) (fields_autoplaced)
     (effects (font (size 1.27 1.27)) (justify right bottom))
   )
-  (label "DQ10" (at 160.02 151.13 180) (fields_autoplaced)
-    (effects (font (size 1.27 1.27)) (justify right bottom))
+  (label "DQ10" (at 148.59 95.25 0) (fields_autoplaced)
+    (effects (font (size 1.27 1.27)) (justify left bottom))
   )
   (label "DQ13" (at 215.9 153.67 0) (fields_autoplaced)
     (effects (font (size 1.27 1.27)) (justify left bottom))
   )
-  (label "DQ9" (at 160.02 148.59 180) (fields_autoplaced)
-    (effects (font (size 1.27 1.27)) (justify right bottom))
-  )
-  (label "CKE" (at 44.45 104.14 180) (fields_autoplaced)
-    (effects (font (size 1.27 1.27)) (justify right bottom))
+  (label "DQ9" (at 148.59 90.17 0) (fields_autoplaced)
+    (effects (font (size 1.27 1.27)) (justify left bottom))
   )
   (label "DQ4" (at 69.85 68.58 0) (fields_autoplaced)
@@
     (effects (font (size 1.27 1.27)) (justify right bottom))
   )
-  (label "A11" (at 87.63 97.79 180) (fields_autoplaced)
-    (effects (font (size 1.27 1.27)) (justify right bottom))
-  )
   (label "A3" (at 158.75 113.03 180) (fields_autoplaced)
     (effects (font (size 1.27 1.27)) (justify right bottom))
@@
     (effects (font (size 1.27 1.27)) (justify left bottom))
   )
-  (label "DQ15" (at 107.95 166.37 0) (fields_autoplaced)
+  (label "DQ15" (at 116.84 171.45 0) (fields_autoplaced)
     (effects (font (size 1.27 1.27)) (justify left bottom))
   )
@@
     (effects (font (size 1.27 1.27)) (justify right bottom))
   )
-  (label "A12" (at 148.59 87.63 0) (fields_autoplaced)
-    (effects (font (size 1.27 1.27)) (justify left bottom))
-  )
   (label "DQ7" (at 215.9 54.61 0) (fields_autoplaced)
     (effects (font (size 1.27 1.27)) (justify left bottom))
   )
-  (label "DQ8" (at 148.59 97.79 0) (fields_autoplaced)
+  (label "DQ8" (at 148.59 87.63 0) (fields_autoplaced)
     (effects (font (size 1.27 1.27)) (justify left bottom))
   )
@@
     (effects (font (size 1.27 1.27)) (justify left bottom))
   )
-  (label "A12" (at 44.45 96.52 180) (fields_autoplaced)
-    (effects (font (size 1.27 1.27)) (justify right bottom))
-  )
   (label "A6" (at 44.45 81.28 180) (fields_autoplaced)
     (effects (font (size 1.27 1.27)) (justify right bottom))
   )
-  (label "DQMH" (at 148.59 95.25 0) (fields_autoplaced)
-    (effects (font (size 1.27 1.27)) (justify left bottom))
+  (label "DQMH" (at 87.63 97.79 180) (fields_autoplaced)
+    (effects (font (size 1.27 1.27)) (justify right bottom))
   )
   (label "DQ14" (at 69.85 93.98 0) (fields_autoplaced)
@@
     )
   )
-  (global_label "LED7" (shape output) (at 116.84 171.45 0) (fields_autoplaced)
-    (effects (font (size 1.27 1.27)) (justify left))
-    (property "Intersheetrefs" "${INTERSHEET_REFS}" (at 124.4818 171.45 0)
+  (global_label "ULPI_NXT" (shape input) (at 219.71 123.19 0) (fields_autoplaced)
+    (effects (font (size 1.27 1.27)) (justify left))
+    (property "Intersheetrefs" "${INTERSHEET_REFS}" (at 231.4038 123.19 0)
+      (effects (font (size 1.27 1.27)) (justify left) hide)
+    )
+  )
+  (global_label "FPGA_B3_IO_0" (shape bidirectional) (at 148.59 97.79 0) (fields_autoplaced)
+    (effects (font (size 1.27 1.27)) (justify left))
+    (property "Intersheetrefs" "${INTERSHEET_REFS}" (at 165.9308 97.79 0)
+      (effects (font (size 1.27 1.27)) (justify left) hide)
+    )
+  )
+  (global_label "LED7" (shape output) (at 116.84 166.37 0) (fields_autoplaced)
+    (effects (font (size 1.27 1.27)) (justify left))
+    (property "Intersheetrefs" "${INTERSHEET_REFS}" (at 124.4818 166.37 0)
       (effects (font (size 1.27 1.27)) (justify left) hide)
     )
@@
     )
   )
+  (global_label "ULPI_CLK" (shape input) (at 219.71 120.65 0) (fields_autoplaced)
+    (effects (font (size 1.27 1.27)) (justify left))
+    (property "Intersheetrefs" "${INTERSHEET_REFS}" (at 231.4643 120.65 0)
+      (effects (font (size 1.27 1.27)) (justify left) hide)
+    )
+  )
   (global_label "LED2" (shape output) (at 215.9 148.59 0) (fields_autoplaced)
     (effects (font (size 1.27 1.27)) (justify left))
@@
     )
   )
+  (global_label "FPGA_B3_IO_1" (shape bidirectional) (at 160.02 148.59 180) (fields_autoplaced)
+    (effects (font (size 1.27 1.27)) (justify right))
+    (property "Intersheetrefs" "${INTERSHEET_REFS}" (at 142.6792 148.59 0)
+      (effects (font (size 1.27 1.27)) (justify right) hide)
+    )
+  )
+  (global_label "FPGA_B3_IO_2" (shape bidirectional) (at 160.02 151.13 180) (fields_autoplaced)
+    (effects (font (size 1.27 1.27)) (justify right))
+    (property "Intersheetrefs" "${INTERSHEET_REFS}" (at 142.6792 151.13 0)
+      (effects (font (size 1.27 1.27)) (justify right) hide)
+    )
+  )
+  (global_label "A12" (shape input) (at 44.45 96.52 180) (fields_autoplaced)
+    (effects (font (size 1.27 1.27)) (justify right))
+    (property "Intersheetrefs" "${INTERSHEET_REFS}" (at 37.9572 96.52 0)
+      (effects (font (size 1.27 1.27)) (justify right) hide)
+    )
+  )
   (global_label "LED1" (shape output) (at 215.9 146.05 0) (fields_autoplaced)
     (effects (font (size 1.27 1.27)) (justify left))
@@
     )
   )
-  (global_label "ULPI_STP" (shape output) (at 219.71 120.65 0) (fields_autoplaced)
-    (effects (font (size 1.27 1.27)) (justify left))
-    (property "Intersheetrefs" "${INTERSHEET_REFS}" (at 231.3433 120.65 0)
+  (global_label "ULPI_STP" (shape output) (at 219.71 115.57 0) (fields_autoplaced)
+    (effects (font (size 1.27 1.27)) (justify left))
+    (property "Intersheetrefs" "${INTERSHEET_REFS}" (at 231.3433 115.57 0)
       (effects (font (size 1.27 1.27)) (justify left) hide)
     )
@@
       (effects (font (size 1.27 1.27)) (justify right) hide)
     )
+  )
+  (global_label "CKE" (shape input) (at 44.45 104.14 180) (fields_autoplaced)
+    (effects (font (size 1.27 1.27)) (justify right))
+    (property "Intersheetrefs" "${INTERSHEET_REFS}" (at 37.7758 104.14 0)
+      (effects (font (size 1.27 1.27)) (justify right) hide)
+    )
+  )
+  (global_label "ULPI_DIR" (shape input) (at 219.71 118.11 0) (fields_autoplaced)
+    (effects (font (size 1.27 1.27)) (justify left))
+    (property "Intersheetrefs" "${INTERSHEET_REFS}" (at 231.041 118.11 0)
+      (effects (font (size 1.27 1.27)) (justify left) hide)
+    )
+  )
+  (global_label "A11" (shape input) (at 44.45 93.98 180) (fields_autoplaced)
+    (effects (font (size 1.27 1.27)) (justify right))
+    (property "Intersheetrefs" "${INTERSHEET_REFS}" (at 37.9572 93.98 0)
+      (effects (font (size 1.27 1.27)) (justify right) hide)
+    )

Commit message: Some BOM clarifications and updates
Parts:
- U8: value T8Q144xx -> T20Q144xx
- X2: value ECS-2520MV-120-CM -> ECS-2520MV-250-CM
Other:
- note added: "Backup Clock (optional)"
- note added: "NOTE: SDRAM not used for Ethernet/PTP application. Can be loaded to test the SDRAM controller on the same PCB."
Changed lines of the file:
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@@
     (stroke (width 0) (type default))
+  )
+  (text "Backup Clock (optional)" (at 144.145 181.61 0)
+    (effects (font (size 1.27 1.27)) (justify left bottom))
+  )
+  (text "NOTE:\nSDRAM not used for Ethernet/PTP application.\nCan be loaded to test the SDRAM controller\non the same PCB."
+    (at 62.23 133.985 0)
+    (effects (font (size 1.27 1.27)) (justify left bottom))
   )
   (label "DQML" (at 160.02 82.55 180) (fields_autoplaced)
@@
       (effects (font (size 1.27 1.27)))
     )
-    (property "Value" "T8Q144xx" (at 118.11 104.4743 0)
+    (property "Value" "T20Q144xx" (at 118.11 104.4743 0)
       (effects (font (size 1.27 1.27)))
     )
@@
       (effects (font (size 1.27 1.27)) hide)
     )
-    (property "Value" "T8Q144xx" (at 187.96 99.3943 0)
+    (property "Value" "T20Q144xx" (at 187.96 99.3943 0)
       (effects (font (size 1.27 1.27)) hide)
     )
@@
       (effects (font (size 1.27 1.27)))
     )
-    (property "Value" "T8Q144xx" (at 80.01 183.2143 0)
+    (property "Value" "T20Q144xx" (at 80.01 183.2143 0)
       (effects (font (size 1.27 1.27)))
     )
@@
       (effects (font (size 1.27 1.27)))
     )
-    (property "Value" "T8Q144xx" (at 201.93 132.08 0)
+    (property "Value" "T20Q144xx" (at 201.93 132.08 0)
       (effects (font (size 1.27 1.27)))
     )
@@
       (effects (font (size 1.27 1.27)))
     )
-    (property "Value" "T8Q144xx" (at 187.96 66.3743 0)
+    (property "Value" "T20Q144xx" (at 187.96 66.3743 0)
       (effects (font (size 1.27 1.27)))
     )
@@
       (effects (font (size 1.27 1.27)))
     )
-    (property "Value" "T8Q144xx" (at 200.66 162.56 0)
+    (property "Value" "T20Q144xx" (at 200.66 162.56 0)
       (effects (font (size 1.27 1.27)))
     )
@@
       (effects (font (size 1.27 1.27)))
     )
-    (property "Value" "ECS-2520MV-120-CM" (at 127.635 182.88 0)
-      (effects (font (size 1.27 1.27)))
-    )
+    (property "Value" "ECS-2520MV-250-CM" (at 127.635 182.88 0)
+      (effects (font (size 1.27 1.27)))
+    )

Commit message: part-info update
Parts:
- U1: value MT48LC16M16A2P -> NDS36PT5-16ET
Changed lines of the file:
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@@
       (effects (font (size 1.27 1.27)) (justify left))
     )
-    (property "Value" "MT48LC16M16A2P" (at 59.3441 54.1599 0)
+    (property "Value" "NDS36PT5-16ET" (at 59.3441 54.1599 0)
       (effects (font (size 1.27 1.27)) (justify left))
     )
@@
       (effects (font (size 1.27 1.27) italic) hide)
     )
-    (property "Datasheet" "https://www.micron.com/-/media/client/global/documents/products/data-sheet/dram/256mb_sdr.pdf" (at 57.15 95.25 0)
+    (property "Datasheet" "" (at 57.15 95.25 0)
       (effects (font (size 1.27 1.27)) hide)
     )
