File: trion-8-test.kicad_sch (KiCad schematic)
At the start: 4 parts

Commit message: sdram layout done - COMPLETE REWORK NEEDED
cannot mix LVDS and GPIO banks due to too different timing
Connections:
- no-connect marks 1 -> 0
Other:
- removed sheet FT-USB-JTAG
- removed sheet usb_fsls
- added sheet sdram (sdram.kicad_sch)
- sheet bank_1a_cfg ports: added none; removed GPIOR_155
- sheet ulpi ports: added none; removed ULPI_RSTb, ULPI_STP
Changed lines of the file:
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@@
 (kicad_sch (version 20230121) (generator eeschema)
   (paper "A4")
-  (no_connect (at 65.405 88.9))
-  (wire (pts (xy 64.77 176.53) (xy 64.77 139.7))
-    (stroke (width 0) (type default))
-  )
-  (wire (pts (xy 66.675 173.355) (xy 66.675 135.89))
-    (stroke (width 0) (type default))
-  )
-  (wire (pts (xy 64.77 139.7) (xy 61.595 139.7))
-    (stroke (width 0) (type default))
-  )
-  (wire (pts (xy 62.23 176.53) (xy 64.77 176.53))
-    (stroke (width 0) (type default))
-  )
-  (wire (pts (xy 62.23 173.355) (xy 66.675 173.355))
-    (stroke (width 0) (type default))
-  )
-  (wire (pts (xy 66.675 135.89) (xy 61.595 135.89))
-    (stroke (width 0) (type default))
-  )
   (symbol (lib_id "Mechanical:MountingHole") (at 191.77 132.08 0) (unit 1)
     (in_bom yes) (on_board yes) (dnp no) (fields_autoplaced)
@@
     )
   )
-  (sheet (at 29.845 160.02) (size 32.385 27.305) (fields_autoplaced)
+  (sheet (at 32.385 161.29) (size 29.21 24.13) (fields_autoplaced)
     (stroke (width 0.1524) (type solid))
     (fill (color 0 0 0 0.0000))
-    (property "Sheetname" "usb_fsls" (at 29.845 159.3084 0)
+    (property "Sheetname" "sdram" (at 32.385 160.5784 0)
       (effects (font (size 1.27 1.27)) (justify left bottom))
     )
-    (property "Sheetfile" "usb_fsls.kicad_sch" (at 29.845 187.9096 0)
+    (property "Sheetfile" "sdram.kicad_sch" (at 32.385 186.0046 0)
       (effects (font (size 1.27 1.27)) (justify left top))
-    )
-    (pin "GPIOL_75" input (at 62.23 176.53 0)
-      (effects (font (size 1.27 1.27)) (justify right))
-    )
-    (pin "GPIOL_73" input (at 62.23 173.355 0)
-      (effects (font (size 1.27 1.27)) (justify right))
     )
     (instances
       (project "trion-8-test"
-        (path "/8c6e15e3-1804-4f03-8a4f-3cb8420d9169" (page "5"))
+        (path "/8c6e15e3-1804-4f03-8a4f-3cb8420d9169" (page "7"))
       )
     )
@@
     (property "Sheetfile" "ulpi.kicad_sch" (at 29.845 147.9046 0)
       (effects (font (size 1.27 1.27)) (justify left top))
-    )
-    (pin "ULPI_RSTb" input (at 61.595 135.89 0)
-      (effects (font (size 1.27 1.27)) (justify right))
-    )
-    (pin "ULPI_STP" input (at 61.595 139.7 0)
-      (effects (font (size 1.27 1.27)) (justify right))
     )
     (instances
@@
     )
   )
-  (sheet (at 41.275 34.925) (size 26.035 24.765) (fields_autoplaced)
-    (stroke (width 0.1524) (type solid))
-    (fill (color 0 0 0 0.0000))
-    (property "Sheetname" "FT-USB-JTAG" (at 41.275 34.2134 0)
-      (effects (font (size 1.27 1.27)) (justify left bottom))
-    )
-    (property "Sheetfile" "FT-USB-JTAG.kicad_sch" (at 41.275 60.2746 0)
-      (effects (font (size 1.27 1.27)) (justify left top))
-    )
-    (instances
-      (project "trion-8-test"
-        (path "/8c6e15e3-1804-4f03-8a4f-3cb8420d9169" (page "2"))
-      )
-    )
-  )
   (sheet (at 27.94 76.2) (size 37.465 27.94) (fields_autoplaced)
     (stroke (width 0.1524) (type solid))
@@
       (effects (font (size 1.27 1.27)) (justify left top))
     )
-    (pin "GPIOR_155" bidirectional (at 65.405 88.9 0)
-      (effects (font (size 1.27 1.27)) (justify right))
-    )
     (instances

Commit message: layout finished; passed all checks...
Changed lines of the file:
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@@
     )
   )
-  (sheet (at 32.385 161.29) (size 29.21 24.13) (fields_autoplaced)
+  (sheet (at 32.131 161.29) (size 30.099 24.13) (fields_autoplaced)
     (stroke (width 0.1524) (type solid))
     (fill (color 0 0 0 0.0000))
-    (property "Sheetname" "sdram" (at 32.385 160.5784 0)
+    (property "Sheetname" "sdram" (at 32.131 160.5784 0)
       (effects (font (size 1.27 1.27)) (justify left bottom))
     )
-    (property "Sheetfile" "sdram.kicad_sch" (at 32.385 186.0046 0)
+    (property "Sheetfile" "sdram.kicad_sch" (at 32.131 186.0046 0)
       (effects (font (size 1.27 1.27)) (justify left top))
     )
@@
     )
   )
-  (sheet (at 29.845 118.745) (size 31.75 28.575) (fields_autoplaced)
+  (sheet (at 31.115 118.745) (size 31.115 28.575) (fields_autoplaced)
     (stroke (width 0.1524) (type solid))
     (fill (color 0 0 0 0.0000))
-    (property "Sheetname" "ulpi" (at 29.845 118.0334 0)
+    (property "Sheetname" "ulpi" (at 31.115 118.0334 0)
       (effects (font (size 1.27 1.27)) (justify left bottom))
     )
-    (property "Sheetfile" "ulpi.kicad_sch" (at 29.845 147.9046 0)
+    (property "Sheetfile" "ulpi.kicad_sch" (at 31.115 147.9046 0)
       (effects (font (size 1.27 1.27)) (justify left top))
     )
@@
     )
   )
-  (sheet (at 27.94 76.2) (size 37.465 27.94) (fields_autoplaced)
+  (sheet (at 28.067 80.772) (size 35.433 27.94) (fields_autoplaced)
     (stroke (width 0.1524) (type solid))
     (fill (color 0 0 0 0.0000))
-    (property "Sheetname" "bank_1a_cfg" (at 27.94 75.4884 0)
+    (property "Sheetname" "bank_1a_cfg" (at 28.067 80.0604 0)
       (effects (font (size 1.27 1.27)) (justify left bottom))
     )
-    (property "Sheetfile" "bank_1a_cfg.kicad_sch" (at 27.94 104.7246 0)
+    (property "Sheetfile" "bank_1a_cfg.kicad_sch" (at 28.067 109.2966 0)
       (effects (font (size 1.27 1.27)) (justify left top))
     )

Commit message: added ethernet phy
Other:
- added sheet Ethernet (ethernet.kicad_sch)
Changed lines of the file:
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@@
+    )
+  )
+  (sheet (at 162.56 44.45) (size 50.8 30.48) (fields_autoplaced)
+    (stroke (width 0.1524) (type solid))
+    (fill (color 0 0 0 0.0000))
+    (property "Sheetname" "Ethernet" (at 162.56 43.7384 0)
+      (effects (font (size 1.27 1.27)) (justify left bottom))
+    )
+    (property "Sheetfile" "ethernet.kicad_sch" (at 162.56 75.5146 0)
+      (effects (font (size 1.27 1.27)) (justify left top))
+    )
+    (instances
+      (project "trion-8-test"
+        (path "/8c6e15e3-1804-4f03-8a4f-3cb8420d9169" (page "8"))
+      )
     )
   )

Commit message: Some BOM clarifications and updates
Parts:
- H1, H2, H3, H4: value Foot -> Foot FF-13-P3.5X5.5B; Manufacturer (none) -> Essentra; Part (none) -> FF-13-P3.5X5.5B
Other:
- sheet unused renamed GPIO
Changed lines of the file:
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@@
   (paper "A4")
   (symbol (lib_id "Mechanical:MountingHole") (at 191.77 132.08 0) (unit 1)
-    (in_bom yes) (on_board yes) (dnp no) (fields_autoplaced)
+    (in_bom yes) (on_board yes) (dnp no)
     (property "Reference" "H3" (at 194.31 130.8679 0)
       (effects (font (size 1.27 1.27)) (justify left))
     )
-    (property "Value" "Foot" (at 194.31 133.2921 0)
+    (property "Value" "Foot FF-13-P3.5X5.5B" (at 180.34 142.24 0)
       (effects (font (size 1.27 1.27)) (justify left))
     )
@@
     )
     (property "Datasheet" "~" (at 191.77 132.08 0)
+      (effects (font (size 1.27 1.27)) hide)
+    )
+    (property "Part" "FF-13-P3.5X5.5B" (at 191.77 132.08 0)
+      (effects (font (size 1.27 1.27)) hide)
+    )
+    (property "Manufacturer" "Essentra" (at 191.77 132.08 0)
       (effects (font (size 1.27 1.27)) hide)
     )
@@
   )
   (symbol (lib_id "Mechanical:MountingHole") (at 171.45 132.08 0) (unit 1)
-    (in_bom yes) (on_board yes) (dnp no) (fields_autoplaced)
+    (in_bom yes) (on_board yes) (dnp no)
     (property "Reference" "H1" (at 173.99 130.8679 0)
       (effects (font (size 1.27 1.27)) (justify left))
     )
-    (property "Value" "Foot" (at 173.99 133.2921 0)
+    (property "Value" "Foot FF-13-P3.5X5.5B" (at 160.02 136.525 0)
       (effects (font (size 1.27 1.27)) (justify left))
     )
@@
     )
     (property "Datasheet" "~" (at 171.45 132.08 0)
+      (effects (font (size 1.27 1.27)) hide)
+    )
+    (property "Part" "FF-13-P3.5X5.5B" (at 171.45 132.08 0)
+      (effects (font (size 1.27 1.27)) hide)
+    )
+    (property "Manufacturer" "Essentra" (at 171.45 132.08 0)
       (effects (font (size 1.27 1.27)) hide)
     )
@@
   )
   (symbol (lib_id "Mechanical:MountingHole") (at 201.295 132.08 0) (unit 1)
-    (in_bom yes) (on_board yes) (dnp no) (fields_autoplaced)
+    (in_bom yes) (on_board yes) (dnp no)
     (property "Reference" "H4" (at 203.835 130.8679 0)
       (effects (font (size 1.27 1.27)) (justify left))
     )
-    (property "Value" "Foot" (at 203.835 133.2921 0)
+    (property "Value" "Foot FF-13-P3.5X5.5B" (at 189.865 144.78 0)
       (effects (font (size 1.27 1.27)) (justify left))
     )
@@
     )
     (property "Datasheet" "~" (at 201.295 132.08 0)
+      (effects (font (size 1.27 1.27)) hide)
+    )
+    (property "Part" "FF-13-P3.5X5.5B" (at 201.295 132.08 0)
+      (effects (font (size 1.27 1.27)) hide)
+    )
+    (property "Manufacturer" "Essentra" (at 201.295 132.08 0)
       (effects (font (size 1.27 1.27)) hide)
     )
@@
   )
   (symbol (lib_id "Mechanical:MountingHole") (at 182.245 132.08 0) (unit 1)
-    (in_bom yes) (on_board yes) (dnp no) (fields_autoplaced)
+    (in_bom yes) (on_board yes) (dnp no)
     (property "Reference" "H2" (at 184.785 130.8679 0)
       (effects (font (size 1.27 1.27)) (justify left))
     )
-    (property "Value" "Foot" (at 184.785 133.2921 0)
+    (property "Value" "Foot FF-13-P3.5X5.5B" (at 170.815 139.7 0)
       (effects (font (size 1.27 1.27)) (justify left))
     )
@@
     )
     (property "Datasheet" "~" (at 182.245 132.08 0)
+      (effects (font (size 1.27 1.27)) hide)
+    )
+    (property "Part" "FF-13-P3.5X5.5B" (at 182.245 132.08 0)
+      (effects (font (size 1.27 1.27)) hide)
+    )
+    (property "Manufacturer" "Essentra" (at 182.245 132.08 0)
       (effects (font (size 1.27 1.27)) hide)
     )
@@
     (stroke (width 0.1524) (type solid))
     (fill (color 0 0 0 0.0000))
-    (property "Sheetname" "unused" (at 92.075 161.2134 0)
+    (property "Sheetname" "GPIO" (at 92.075 161.2134 0)
       (effects (font (size 1.27 1.27)) (justify left bottom))
     )

Commit message: Added GPS receiver; increased board size
including battery supply; made board bigger
and added edge connectors for ETH GPIO, PPS
and antenna.
Other:
- added sheet GPS (gps.kicad_sch)
Changed lines of the file:
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@@
     )
   )
-  (sheet (at 32.131 161.29) (size 30.099 24.13) (fields_autoplaced)
+  (sheet (at 31.75 161.29) (size 30.48 24.13) (fields_autoplaced)
     (stroke (width 0.1524) (type solid))
     (fill (color 0 0 0 0.0000))
-    (property "Sheetname" "sdram" (at 32.131 160.5784 0)
+    (property "Sheetname" "sdram" (at 31.75 160.5784 0)
       (effects (font (size 1.27 1.27)) (justify left bottom))
     )
-    (property "Sheetfile" "sdram.kicad_sch" (at 32.131 186.0046 0)
+    (property "Sheetfile" "sdram.kicad_sch" (at 31.75 186.0046 0)
       (effects (font (size 1.27 1.27)) (justify left top))
     )
@@
     )
   )
-  (sheet (at 31.115 118.745) (size 31.115 28.575) (fields_autoplaced)
+  (sheet (at 163.195 85.725) (size 49.53 32.385) (fields_autoplaced)
+    (stroke (width 0.1524) (type solid))
+    (fill (color 0 0 0 0.0000))
+    (property "Sheetname" "GPS" (at 163.195 85.0134 0)
+      (effects (font (size 1.27 1.27)) (justify left bottom))
+    )
+    (property "Sheetfile" "gps.kicad_sch" (at 163.195 118.6946 0)
+      (effects (font (size 1.27 1.27)) (justify left top))
+    )
+    (instances
+      (project "trion-8-test"
+        (path "/8c6e15e3-1804-4f03-8a4f-3cb8420d9169" (page "9"))
+      )
+    )
+  )
+  (sheet (at 31.115 118.745) (size 30.48 19.05) (fields_autoplaced)
     (stroke (width 0.1524) (type solid))
     (fill (color 0 0 0 0.0000))
@@
       (effects (font (size 1.27 1.27)) (justify left bottom))
     )
-    (property "Sheetfile" "ulpi.kicad_sch" (at 31.115 147.9046 0)
+    (property "Sheetfile" "ulpi.kicad_sch" (at 31.115 138.3796 0)
       (effects (font (size 1.27 1.27)) (justify left top))
     )
@@
     )
   )
-  (sheet (at 28.067 80.772) (size 35.433 27.94) (fields_autoplaced)
+  (sheet (at 32.385 80.772) (size 27.94 19.558) (fields_autoplaced)
     (stroke (width 0.1524) (type solid))
     (fill (color 0 0 0 0.0000))
-    (property "Sheetname" "bank_1a_cfg" (at 28.067 80.0604 0)
+    (property "Sheetname" "bank_1a_cfg" (at 32.385 80.0604 0)
       (effects (font (size 1.27 1.27)) (justify left bottom))
     )
-    (property "Sheetfile" "bank_1a_cfg.kicad_sch" (at 28.067 109.2966 0)
+    (property "Sheetfile" "bank_1a_cfg.kicad_sch" (at 32.385 100.9146 0)
       (effects (font (size 1.27 1.27)) (justify left top))
     )
