File: bank_1a_cfg.kicad_sch (KiCad schematic)
At the start: 54 parts, among them J2 T8_JTAG, Q1 SSM3K37MFV, SW1 Reset, U8 T8Q144xx, U9 AT25FF081A-SSHN-B, X1 ECS-2520MV-120-CM

Commit message: Fixed V1.0 errata
- added feedback resistor for ulpi transceiver clock oscillator
- removed SS_N connection
Parts:
- renumbered C13 to C27, C14 to C28, C14 to C29, C2 to C3, C13 to C30, C14 to C31, C13 to C32, C14 to C33, C14 to C34, C14 to C35, C14 to C36, C14 to C37, C14 to C38, C14 to C39, C14 to C40, C14 to C41, C14 to C42, C14 to C43, C14 to C44, C14 to C45, C23 to C65, C23 to C66, C23 to C67, C23 to C69, C23 to C70, C23 to C71, D1 to D10, J2 to J3, L2 to L3, L2 to L4, L2 to L5, R3 to R22, R3 to R23, R3 to R24, R3 to R30, R3 to R31, R3 to R32, R3 to R33, R3 to R34, R3 to R35, R3 to R36, R3 to R37, R3 to R40, R3 to R41, R3 to R42, R3 to R43, X1 to X2

Commit message: sdram layout done - COMPLETE REWORK NEEDED
cannot mix LVDS and GPIO banks due to too different timing
Parts:
- removed C3, C42: 100n, Capacitor_SMD:C_0603_1608Metric, symbol Device:C_Small
- removed R22, R23, R24, R30: 10k, Resistor_SMD:R_0603_1608Metric, symbol Device:R_Small
- removed unit 8 of U8
- removed X2: ECS-2520MV-120-CM, Oscillator:Oscillator_SMD_ECS_2520MV-xxx-xx-4Pin_2.5x2.0mm, symbol Oscillator:ECS-2520MV-xxx-xx
Connections:
- no-connect marks 3 -> 2
Other:
- moved on the sheet: C16, C27, C28, C29, C30, C31, C32, C43, C44, C66, C69, C71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

Commit message: layout finished; passed all checks...
Connections:
- net SDRAM_DQ0: now reaches U8.33 (GPIOL_05_CSO)
- no-connect marks 2 -> 1
Changed lines of the file:
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@@
   )
   (no_connect (at 22.86 66.04))
-  (no_connect (at 132.08 55.88))
   (wire (pts (xy 115.57 162.56) (xy 115.57 139.7))
     (stroke (width 0) (type default))
@@
     (stroke (width 0) (type default))
   )
+  (global_label "SDRAM_DQ0" (shape bidirectional) (at 132.08 55.88 0) (fields_autoplaced)
+    (effects (font (size 1.27 1.27)) (justify left))
+    (property "Intersheetrefs" "${INTERSHEET_REFS}" (at 147.2436 55.88 0)
+      (effects (font (size 1.27 1.27)) (justify left) hide)
+    )
+  )
   (symbol (lib_id "Device:R_Small") (at 134.62 34.29 0) (unit 1)

Commit message: Some BOM clarifications and updates
Parts:
- U8: value T8Q144xx -> T20Q144xx
Other:
- note added: "Green LED (indicating FPGA configuration is complete)"
Changed lines of the file:
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@@
     (stroke (width 0) (type default))
+  )
+  (text "Green LED (indicating FPGA\nconfiguration is complete)"
+    (at 121.92 90.805 0)
+    (effects (font (size 1.27 1.27)) (justify left bottom))
   )
   (global_label "SDRAM_DQ0" (shape bidirectional) (at 132.08 55.88 0) (fields_autoplaced)
@@
       (effects (font (size 1.27 1.27)) (justify left))
     )
-    (property "Value" "T8Q144xx" (at 123.952 176.4721 0)
+    (property "Value" "T20Q144xx" (at 123.952 176.4721 0)
       (effects (font (size 1.27 1.27)) (justify left))
     )
@@
       (effects (font (size 1.27 1.27)))
     )
-    (property "Value" "T8Q144xx" (at 109.22 75.2643 0)
-      (effects (font (size 1.27 1.27)))
-    )
+    (property "Value" "T20Q144xx" (at 109.22 75.2643 0)
+      (effects (font (size 1.27 1.27)))
+    )

Commit message: Added Manufacturer + Part info for most components.
Parts:
- C16, C45: Manufacturer (none) -> Samsung; Part (none) -> CL31A106KPHNNNE
- C27, C30, C32: Manufacturer (none) -> TDK; Part (none) -> 2012X5R1C475K125AC
- C28, C29, C31, C33, C34, C35, C36, C37, C38, C39, C40, C41, C43, C44: Manufacturer (none) -> Samsung; Part (none) -> CL10B104KB8NFN
- C65, C66, C67, C69, C70, C71: Manufacturer (none) -> TDK; Part (none) -> CGA4J2X7R1C105K125AA
- D10: value LED -> LED-GRN; Manufacturer (none) -> Wurth; Part (none) -> 150060GS75000
- J3: Manufacturer (none) -> Adam Tech; Part (none) -> 2PH2-14-UA
- L3, L4, L5: Manufacturer (none) -> Laird; Part (none) -> MI0603J601R-10
- Q1: Manufacturer (none) -> Toshiba; Part (none) -> SSM3K37MFV
- SW1: Manufacturer (none) -> C&K; Part (none) -> PTS810
- U8: Manufacturer (none) -> Efinix; Part (none) -> T20Q144C4
- U9: Manufacturer (none) -> Renesas; Part (none) -> AT25FF081A-SSHN-B

Commit message: Added GPS receiver; increased board size
including battery supply; made board bigger
and added edge connectors for ETH GPIO, PPS
and antenna.
Parts:
- removed D10: LED-GRN, LED_SMD:LED_0603_1608Metric, symbol Device:LED
- removed SW1: Reset, Button_Switch_SMD:SW_SPST_PTS810, symbol Switch:SW_Push
- added D5: LED_Dual_RAG, proj_footprints:LED_Wuerth_Sideview, symbol Device:LED_Dual_KAK
- added R51: 1k, Resistor_SMD:R_0603_1608Metric, symbol Device:R_Small
- added SW1: Reconfig, proj_footprints:SW_SPST_PTS810_and_PTS841, symbol fmc:SW_Push_Shielded
Connections:
- net +3V3: now also D5.2 (A); no longer R4.2
- net GND: now also SW1.1, SW1.3 (Shield)
- net at Q1.3 (D): now also R4.2
- net at R4.1: now also D5.3 (K2)
- net at C45.1, J3.3 (Pin_3), R35.2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: now also SW1.2
- net at Q1.1 (G), R36.2, U8.34 (CDONE): now also R51.1
- new net: D5.1 (K1), R51.2
Other:
- note added: "Bi-color LED indicating power and FPGA config. complete: red: power, not configured grn: power, configured"
- note added: "GRN"
- note added: "RED"
- note removed: "Green LED (indicating FPGA configuration is complete)"
- moved on the sheet: Q1, R4

Commit message: finalizing...
Changed lines of the file:
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@@
     (effects (font (size 1.27 1.27)) (justify left bottom))
   )
-  (text "GRN" (at 113.03 90.805 0)
+  (text "GRN" (at 113.03 97.79 0)
     (effects (font (size 1.27 1.27)) (justify left bottom))
   )
-  (text "RED" (at 113.03 97.79 0)
+  (text "RED" (at 113.03 90.805 0)
     (effects (font (size 1.27 1.27)) (justify left bottom))
   )
