File: unused.kicad_sch (KiCad schematic)
At the start: 1 part, among them U8 T8Q144xx

Commit message: sdram layout done - COMPLETE REWORK NEEDED
cannot mix LVDS and GPIO banks due to too different timing
Parts:
- removed unit 9 of U8
- removed unit 10 of U8
Connections:
- no-connect marks 41 -> 14
Other:
- moved on the sheet: U8B

Commit message: layout finished; passed all checks...
Parts:
- removed U8: T8Q144xx, Package_QFP:LQFP-144_20x20mm_P0.5mm, symbol FPGA_Efinix_Trion:T8Q144xx
- added C11, C14: 100n, Capacitor_SMD:C_0603_1608Metric, symbol Device:C_Small
- added U8: T8Q144xx, Package_QFP:LQFP-144_20x20mm_P0.5mm, symbol FPGA_Efinix_Trion:T8Q144xx
Connections:
- net +3V3: now also C11.1, C14.1, U8.51 (VCCIO4B), U8.52 (VCCIO4B), U8.62 (VCCIO4A), U8.63 (VCCIO4A)
- new net GND: C11.2, C14.2
- no-connect marks 14 -> 27

Commit message: added ethernet phy
Parts:
- added C74, C75: 100n, Capacitor_SMD:C_0603_1608Metric, symbol Device:C_Small
- added J6: FPGA GPIO, Connector_PinHeader_2.54mm:PinHeader_2x10_P2.54mm_Vertical, symbol Connector_Generic:Conn_02x10_Odd_Even
- added J7: FPGA_B3_GPIO, Connector_PinHeader_2.54mm:PinHeader_2x04_P2.54mm_Vertical, symbol Connector_Generic:Conn_02x04_Odd_Even
Connections:
- net +3V3: now also C74.1, C75.1, J6.2 (Pin_2), J6.20 (Pin_20), J7.8 (Pin_8)
- net GND: now also C74.2, C75.2, J6.1 (Pin_1), J6.11 (Pin_11), J6.13 (Pin_13), J6.15 (Pin_15), J6.17 (Pin_17), J6.19 (Pin_19), J6.3 (Pin_3), J6.5 (Pin_5), J6.7 (Pin_7), J6.9 (Pin_9), J7.1 (Pin_1), J7.3 (Pin_3), J7.5 (Pin_5), J7.7 (Pin_7)
- net FPGA_GPIO_0: now reaches U8.36 (REF_RES)
- net FPGA_GPIO_0: now also J6.4 (Pin_4)
- net FPGA_GPIO_1: now reaches U8.38 (GPIOB_TXP00)
- net FPGA_GPIO_1: now also J6.6 (Pin_6)
- net FPGA_GPIO_2: now reaches U8.39 (GPIOB_TXN00)
- net FPGA_GPIO_2: now also J6.8 (Pin_8)
- net FPGA_GPIO_3: now reaches U8.40 (GPIOB_TXP02)
- net FPGA_GPIO_3: now also J6.10 (Pin_10)
- net FPGA_GPIO_4: now reaches U8.41 (GPIOB_TXN02)
- net FPGA_GPIO_4: now also J6.12 (Pin_12)
- net FPGA_GPIO_5: now reaches U8.42 (GPIOB_TXP04)
- net FPGA_GPIO_5: now also J6.14 (Pin_14)
- net FPGA_GPIO_6: now reaches U8.43 (GPIOB_TXN04)
- net FPGA_GPIO_6: now also J6.16 (Pin_16)
- net FPGA_GPIO_7: now reaches U8.45 (GPIOB_TXP06)
- net FPGA_GPIO_7: now also J6.18 (Pin_18)
- net ETH0_RSTb: now reaches U8.46 (GPIOB_TXN06)
- net ETH0_MDIO: now reaches U8.47 (GPIOB_TXP09)
- net ETH0_MDC: now reaches U8.48 (GPIOB_TXN09)
- net ETH0_PWRDWN_IRQ: now reaches U8.53 (GPIOB_TXP11)
- net ETH0_TXD_3: now reaches U8.54 (GPIOB_TXN11)
- net ETH0_TXD_2: now reaches U8.55 (GPIOB_RXP00)
- net ETH0_TXD_1: now reaches U8.56 (GPIOB_RXN00)
- net ETH0_TXD_0: now reaches U8.58 (GPIOB_RXP02)
- net ETH0_TX_EN: now reaches U8.59 (GPIOB_RXN02)
- net ETH0_RXD_0: now reaches U8.60 (GPIOB_RXN03)
- net ETH0_RXD_1: now reaches U8.61 (GPIOB_RXP03)
- net ETH0_RXD_2: now reaches U8.65 (GPIOB_RXN07)
- net ETH0_RXD_3: now reaches U8.66 (GPIOB_RXP07)
- net ETH0_COL: now reaches U8.67 (GPIOB_RXP10)
- net ETH0_RX_ER: now reaches U8.68 (GPIOB_RXN10)
- net ETH0_CRS_DV: now reaches U8.69 (GPIOB_RXN12_EXTFB0)
- net ETH0_RX_DV: now reaches U8.70 (GPIOB_RXP12_EXTFB0)
- net ETH0_RX_CLK: now reaches U8.71 (GPIOB_CLKP0)
- net ETH0_GPIO_9: now reaches U8.72 (GPIOB_CLKN0)
- new net FPGA_B3_IO_0: J7.2 (Pin_2)
- new net FPGA_B3_IO_1: J7.4 (Pin_4)
- new net FPGA_B3_IO_2: J7.6 (Pin_6)
- no-connect marks 27 -> 0
Other:
- note added: "Bank 4 is not really unused anymore..."

Commit message: Some BOM clarifications and updates
Parts:
- U8: value T8Q144xx -> T20Q144xx
Other:
- note added: "The filename is 'unused' for legacy reasons."
Changed lines of the file:
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@@
     (stroke (width 0) (type default))
+  )
+  (text "The filename is 'unused' for legacy reasons." (at 179.705 178.435 0)
+    (effects (font (size 1.27 1.27)) (justify left bottom))
   )
   (text "Bank 4 is not really unused anymore..." (at 59.69 36.83 0)
@@
       (effects (font (size 1.27 1.27)))
     )
-    (property "Value" "T8Q144xx" (at 194.31 145.1143 0)
+    (property "Value" "T20Q144xx" (at 194.31 145.1143 0)
       (effects (font (size 1.27 1.27)))
     )
@@
       (effects (font (size 1.27 1.27)))
     )
-    (property "Value" "T8Q144xx" (at 191.77 95.5843 0)
-      (effects (font (size 1.27 1.27)))
-    )
+    (property "Value" "T20Q144xx" (at 191.77 95.5843 0)
+      (effects (font (size 1.27 1.27)))
+    )

Commit message: Added Manufacturer + Part info for most components.
Parts:
- C11, C14, C74, C75: Manufacturer (none) -> Samsung; Part (none) -> CL10B104KB8NFN
- J6: Manufacturer (none) -> Adam Tech; Part (none) -> PH2-20-UA
- J7: Manufacturer (none) -> Adam Tech; Part (none) -> PH2-08-UA
- U8: Manufacturer (none) -> Efinix; Part (none) -> T20Q144C4
Changed lines of the file:
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@@
+      (effects (font (size 1.27 1.27)) hide)
+    )
+    (property "Manufacturer" "Samsung" (at 88.9 97.79 0)
+      (effects (font (size 1.27 1.27)) hide)
+    )
+    (property "Part" "CL10B104KB8NFN" (at 88.9 97.79 0)
       (effects (font (size 1.27 1.27)) hide)
     )
@@
     )
     (property "Datasheet" "~" (at 86.36 173.99 0)
+      (effects (font (size 1.27 1.27)) hide)
+    )
+    (property "Manufacturer" "Adam Tech" (at 86.36 173.99 0)
+      (effects (font (size 1.27 1.27)) hide)
+    )
+    (property "Part" "PH2-08-UA" (at 86.36 173.99 0)
       (effects (font (size 1.27 1.27)) hide)
     )
@@
       (effects (font (size 1.27 1.27)) hide)
     )
+    (property "Manufacturer" "Samsung" (at 127 63.5 0)
+      (effects (font (size 1.27 1.27)) hide)
+    )
+    (property "Part" "CL10B104KB8NFN" (at 127 63.5 0)
+      (effects (font (size 1.27 1.27)) hide)
+    )
     (pin "1")
     (pin "2")
@@
     )
     (property "Datasheet" "~" (at 85.725 137.16 0)
+      (effects (font (size 1.27 1.27)) hide)
+    )
+    (property "Manufacturer" "Adam Tech" (at 85.725 137.16 0)
+      (effects (font (size 1.27 1.27)) hide)
+    )
+    (property "Part" "PH2-20-UA" (at 85.725 137.16 0)
       (effects (font (size 1.27 1.27)) hide)
     )
@@
     )
     (property "Datasheet" "https://www.efinixinc.com/docs/trion8-ds-v4.4.pdf" (at 194.31 152.4 0)
+      (effects (font (size 1.27 1.27)) hide)
+    )
+    (property "Manufacturer" "Efinix" (at 194.31 125.73 0)
+      (effects (font (size 1.27 1.27)) hide)
+    )
+    (property "Part" "T20Q144C4" (at 194.31 125.73 0)
       (effects (font (size 1.27 1.27)) hide)
     )
@@
       (effects (font (size 1.27 1.27)) hide)
     )
+    (property "Manufacturer" "Efinix" (at 191.77 76.2 0)
+      (effects (font (size 1.27 1.27)) hide)
+    )
+    (property "Part" "T20Q144C4" (at 191.77 76.2 0)
+      (effects (font (size 1.27 1.27)) hide)
+    )
     (pin "76")
     (pin "141")
@@
       (effects (font (size 1.27 1.27)) hide)
     )
+    (property "Manufacturer" "Samsung" (at 127 97.79 0)
+      (effects (font (size 1.27 1.27)) hide)
+    )
+    (property "Part" "CL10B104KB8NFN" (at 127 97.79 0)
+      (effects (font (size 1.27 1.27)) hide)
+    )
     (pin "1")
     (pin "2")
@@
       (effects (font (size 1.27 1.27)) hide)
     )
+    (property "Manufacturer" "Samsung" (at 105.41 98.425 0)
+      (effects (font (size 1.27 1.27)) hide)
+    )
+    (property "Part" "CL10B104KB8NFN" (at 105.41 98.425 0)
+      (effects (font (size 1.27 1.27)) hide)
+    )

Commit message: Added GPS receiver; increased board size
including battery supply; made board bigger
and added edge connectors for ETH GPIO, PPS
and antenna.
Parts:
- removed J7: FPGA_B3_GPIO, Connector_PinHeader_2.54mm:PinHeader_2x04_P2.54mm_Vertical, symbol Connector_Generic:Conn_02x04_Odd_Even
Connections:
- net ETH0_RXD_2 is gone; now on net FPGA_GPIO_7: U8.65 (GPIOB_RXN07)
- net ETH0_TXD_2 is gone; now on net FPGA_GPIO_6: U8.55 (GPIOB_RXP00)
- net ETH0_TXD_3 is gone; now on net FPGA_GPIO_5: U8.54 (GPIOB_TXN11)
- net FPGA_GPIO_5: no longer U8.42 (GPIOB_TXP04)
- net FPGA_GPIO_6: no longer U8.43 (GPIOB_TXN04)
- net FPGA_GPIO_7: no longer U8.45 (GPIOB_TXP06)
- net ETH0_RXD_3 renamed GPS_RSTb
- new net GPS_PPS: U8.45 (GPIOB_TXP06)
- new net UART_RX: U8.42 (GPIOB_TXP04)
- new net UART_TX: U8.43 (GPIOB_TXN04)

Commit message: finalizing...
Other:
- note removed: "Bank 4 is not really unused anymore..."
Changed lines of the file:
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@@
-    (effects (font (size 1.27 1.27)) (justify left bottom))
-  )
-  (text "Bank 4 is not really unused anymore..." (at 59.69 36.83 0)
     (effects (font (size 1.27 1.27)) (justify left bottom))
   )
