File: gps.kicad_sch (KiCad schematic)
At the start: 28 parts, among them J10 PPS, J2 GPS_GPIO, J8 Antenna, J9 Geofnc, U3 LC76G, U4 TS5A63157DBV

Commit message: bumped version to 2.1
updated several values;

* added AC-coupling cap on RF_IN
Parts:
- added C84: 47p, Capacitor_SMD:C_0402_1005Metric, symbol Device:C_Small
- D12: Manufacturer (none) -> Nexperia; Part (none) -> BAS16J,115
- D13: Manufacturer Littlefuse -> Nexperia; Part SP0402B-ULC-01ETG -> PESD5V5C1BLYL
- L8: value 100n -> 68n; Manufacturer (none) -> Murata; Part (none) -> LQW15AN68NJ00D
- R13: value 210 -> 10
Connections:
- net RF_IN: now also C84.1; no longer U3.11 (RF_IN)
- new net RF_IN_AC: C84.2, U3.11 (RF_IN)
Changed lines of the file:
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@@
   (junction (at 196.215 100.965) (diameter 0) (color 0 0 0 0)
   )
+  (junction (at 211.455 106.045) (diameter 0) (color 0 0 0 0)
+  )
+  (junction (at 114.3 93.345) (diameter 0) (color 0 0 0 0)
+  )
+  (junction (at 148.59 47.625) (diameter 0) (color 0 0 0 0)
+  )
+  (junction (at 138.43 72.39) (diameter 0) (color 0 0 0 0)
+  )
+  (junction (at 82.55 109.22) (diameter 0) (color 0 0 0 0)
+  )
+  (junction (at 248.285 109.855) (diameter 0) (color 0 0 0 0)
+  )
+  (junction (at 196.215 102.235) (diameter 0) (color 0 0 0 0)
+  )
+  (junction (at 146.05 98.425) (diameter 0) (color 0 0 0 0)
+  )
+  (junction (at 148.59 50.165) (diameter 0) (color 0 0 0 0)
+  )
+  (junction (at 118.11 101.6) (diameter 0) (color 0 0 0 0)
+  )
+  (junction (at 199.39 83.185) (diameter 0) (color 0 0 0 0)
+  )
+  (junction (at 97.79 93.345) (diameter 0) (color 0 0 0 0)
+  )
+  (junction (at 148.59 52.705) (diameter 0) (color 0 0 0 0)
+  )
+  (junction (at 64.77 93.345) (diameter 0) (color 0 0 0 0)
+  )
+  (junction (at 211.455 102.235) (diameter 0) (color 0 0 0 0)
+  )
+  (junction (at 149.86 98.425) (diameter 0) (color 0 0 0 0)
+  )
+  (junction (at 105.41 101.6) (diameter 0) (color 0 0 0 0)
+  )
   (junction (at 232.41 98.425) (diameter 0) (color 0 0 0 0)
-  )
-  (junction (at 211.455 106.045) (diameter 0) (color 0 0 0 0)
-  )
-  (junction (at 114.3 93.345) (diameter 0) (color 0 0 0 0)
-  )
-  (junction (at 148.59 47.625) (diameter 0) (color 0 0 0 0)
-  )
-  (junction (at 138.43 72.39) (diameter 0) (color 0 0 0 0)
-  )
-  (junction (at 82.55 109.22) (diameter 0) (color 0 0 0 0)
-  )
-  (junction (at 248.285 109.855) (diameter 0) (color 0 0 0 0)
-  )
-  (junction (at 196.215 102.235) (diameter 0) (color 0 0 0 0)
-  )
-  (junction (at 146.05 98.425) (diameter 0) (color 0 0 0 0)
-  )
-  (junction (at 148.59 50.165) (diameter 0) (color 0 0 0 0)
-  )
-  (junction (at 118.11 101.6) (diameter 0) (color 0 0 0 0)
-  )
-  (junction (at 199.39 83.185) (diameter 0) (color 0 0 0 0)
-  )
-  (junction (at 97.79 93.345) (diameter 0) (color 0 0 0 0)
-  )
-  (junction (at 148.59 52.705) (diameter 0) (color 0 0 0 0)
-  )
-  (junction (at 64.77 93.345) (diameter 0) (color 0 0 0 0)
-  )
-  (junction (at 211.455 102.235) (diameter 0) (color 0 0 0 0)
-  )
-  (junction (at 149.86 98.425) (diameter 0) (color 0 0 0 0)
-  )
-  (junction (at 105.41 101.6) (diameter 0) (color 0 0 0 0)
   )
   (junction (at 167.64 50.165) (diameter 0) (color 0 0 0 0)
@@
     (stroke (width 0) (type default))
   )
+  (wire (pts (xy 194.31 98.425) (xy 215.9 98.425))
+    (stroke (width 0) (type default))
+  )
   (wire (pts (xy 49.53 93.345) (xy 64.77 93.345))
     (stroke (width 0) (type default))
@@
     (stroke (width 0) (type default))
   )
+  (wire (pts (xy 220.98 98.425) (xy 232.41 98.425))
+    (stroke (width 0) (type default))
+  )
   (wire (pts (xy 144.145 98.425) (xy 146.05 98.425))
     (stroke (width 0) (type default))
@@
   )
   (wire (pts (xy 156.845 110.49) (xy 149.86 110.49))
-    (stroke (width 0) (type default))
-  )
-  (wire (pts (xy 194.31 98.425) (xy 232.41 98.425))
     (stroke (width 0) (type default))
   )
@@
   (text "NOTES:\n - 4u7 capacitor used\n   elsewhere has >20M\n   isolation res. which\n   is not great for\n   battery!\n - TS5A63157 has very\n   low leakage."
     (at 35.56 167.64 0)
+    (effects (font (size 1.27 1.27)) (justify left bottom))
+  )
+  (label "RF_IN_AC" (at 201.295 98.425 0) (fields_autoplaced)
     (effects (font (size 1.27 1.27)) (justify left bottom))
   )
@@
       (effects (font (size 1.27 1.27)) hide)
     )
-    (property "Datasheet" "https://www.littelfuse.com/media?resourcetype=datasheets&itemid=54962f33-9d87-4d79-919d-dac7ef6a0067&filename=littelfuse-tvs-diode-array-ultra-low-capacitance-discrete-tvs-datasheet" (at 248.285 103.505 0)
-      (effects (font (size 1.27 1.27)) hide)
-    )
-    (property "Part" "SP0402B-ULC-01ETG" (at 248.285 103.505 0)
-      (effects (font (size 1.27 1.27)) hide)
-    )
-    (property "Manufacturer" "Littlefuse" (at 248.285 103.505 0)
+    (property "Datasheet" "" (at 248.285 103.505 0)
+      (effects (font (size 1.27 1.27)) hide)
+    )
+    (property "Part" "PESD5V5C1BLYL" (at 248.285 103.505 0)
+      (effects (font (size 1.27 1.27)) hide)
+    )
+    (property "Manufacturer" "Nexperia" (at 248.285 103.505 0)
       (effects (font (size 1.27 1.27)) hide)
     )
@@
       (effects (font (size 1.27 1.27)) (justify left))
     )
-    (property "Value" "210" (at 213.995 90.805 90)
+    (property "Value" "10" (at 213.995 90.805 90)
       (effects (font (size 1.27 1.27)) (justify left))
     )
@@
       (effects (font (size 1.27 1.27)) hide)
     )
+    (property "Part" "BAS16J,115" (at 82.55 102.87 90)
+      (effects (font (size 1.27 1.27)) hide)
+    )
+    (property "Manufacturer" "Nexperia" (at 82.55 102.87 90)
+      (effects (font (size 1.27 1.27)) hide)
+    )
     (pin "1")
     (pin "2")
@@
         (path "/8c6e15e3-1804-4f03-8a4f-3cb8420d9169/82d47f49-82af-402b-b162-0356b73b8b45"
           (reference "#PWR069") (unit 1)
+        )
+      )
+    )
+  )
+  (symbol (lib_id "Device:C_Small") (at 218.44 98.425 270) (mirror x) (unit 1)
+    (in_bom yes) (on_board yes) (dnp no)
+    (property "Reference" "C84" (at 216.535 95.25 90)
+      (effects (font (size 1.27 1.27)) (justify left))
+    )
+    (property "Value" "47p" (at 216.535 102.235 90)
+      (effects (font (size 1.27 1.27)) (justify left))
+    )
+    (property "Footprint" "Capacitor_SMD:C_0402_1005Metric" (at 218.44 98.425 0)
+      (effects (font (size 1.27 1.27)) hide)
+    )
+    (property "Datasheet" "~" (at 218.44 98.425 0)
+      (effects (font (size 1.27 1.27)) hide)
+    )
+    (property "Manufacturer" "" (at 218.44 98.425 0)
+      (effects (font (size 1.27 1.27)) hide)
+    )
+    (property "Part" "" (at 218.44 98.425 0)
+      (effects (font (size 1.27 1.27)) hide)
+    )
+    (pin "1")
+    (pin "2")
+    (instances
+      (project "tic-nic"
+        (path "/8c6e15e3-1804-4f03-8a4f-3cb8420d9169/82d47f49-82af-402b-b162-0356b73b8b45"
+          (reference "C84") (unit 1)
         )
       )
@@
       (effects (font (size 1.27 1.27)) (justify left))
     )
-    (property "Value" "100n" (at 233.5508 104.0821 0)
+    (property "Value" "68n" (at 233.5508 104.0821 0)
       (effects (font (size 1.27 1.27)) (justify left))
     )
@@
       (effects (font (size 1.27 1.27)) hide)
     )
+    (property "Part" "LQW15AN68NJ00D" (at 232.41 102.87 0)
+      (effects (font (size 1.27 1.27)) hide)
+    )
+    (property "Manufacturer" "Murata" (at 232.41 102.87 0)
+      (effects (font (size 1.27 1.27)) hide)
+    )
