File: gps.kicad_sch (KiCad schematic)
At the start: 29 parts, among them J10 PPS, J2 GPS_GPIO, J8 Antenna, J9 Geofnc, U3 LC76G, U4 TS5A63157DBV

Commit message: small fixes; prettified the fab layer and added DNP on schematic
Parts:
- D12: value D -> BAS16J
- D13: value ~ -> PESD5V5C1
- R14, R15, R16, R20: now not fitted; now left out of the parts list
Other:
- note added: "Bat. retainer: Keystone 3034 alt. holder: Adam Tech BH-74K-5 Install JP7 1-2 to enable battery- backup; 2-3 when no battery is present or to disable battery."
- note added: "JP6 controls power-supply of active antenna; install for active antenna, remove for passive antenna."
- note added: "Use I2C instead of UART: DNL R29, DNL R38 but load R14, R15, R16 and R20."
- note removed: "Bat. retainer: Keystone 3034 alt. holder: Adam Tech BH-74K-5"
Changed lines of the file:
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@@
     (stroke (width 0) (type default))
   )
-  (text "Bat. retainer: Keystone 3034\nalt. holder: Adam Tech BH-74K-5"
-    (at 64.135 142.24 0)
+  (text "Bat. retainer: Keystone 3034\nalt. holder: Adam Tech BH-74K-5\n\nInstall JP7 1-2 to enable battery-\nbackup; 2-3 when no battery is\npresent or to disable battery."
+    (at 65.405 147.955 0)
+    (effects (font (size 1.27 1.27)) (justify left bottom))
+  )
+  (text "Use I2C instead of UART: DNL R29, DNL R38\nbut load R14, R15, R16 and R20."
+    (at 212.09 71.755 0)
     (effects (font (size 1.27 1.27)) (justify left bottom))
   )
   (text "NOTES:\n - 4u7 capacitor used\n   elsewhere has >20M\n   isolation res. which\n   is not great for\n   battery!\n - TS5A63157 has very\n   low leakage."
     (at 35.56 167.64 0)
+    (effects (font (size 1.27 1.27)) (justify left bottom))
+  )
+  (text "JP6 controls power-supply of active\nantenna; install for active antenna,\nremove for passive antenna."
+    (at 194.945 121.92 0)
     (effects (font (size 1.27 1.27)) (justify left bottom))
   )
@@
   )
   (symbol (lib_id "Diode:ESD9B5.0ST5G") (at 248.285 103.505 90) (unit 1)
-    (in_bom yes) (on_board yes) (dnp no) (fields_autoplaced)
+    (in_bom yes) (on_board yes) (dnp no)
     (property "Reference" "D13" (at 250.2916 103.505 90)
       (effects (font (size 1.27 1.27)) (justify right))
     )
-    (property "Value" "~" (at 245.3203 103.505 0)
+    (property "Value" "PESD5V5C1" (at 245.11 104.775 0)
       (effects (font (size 1.27 1.27)))
     )
@@
   )
   (symbol (lib_id "Device:R_Small") (at 199.39 79.375 0) (unit 1)
-    (in_bom yes) (on_board yes) (dnp no)
+    (in_bom no) (on_board yes) (dnp yes)
     (property "Reference" "R14" (at 196.85 80.645 90)
       (effects (font (size 1.27 1.27)) (justify left))
@@
   )
   (symbol (lib_id "Device:R_Small") (at 213.36 85.725 270) (mirror x) (unit 1)
-    (in_bom yes) (on_board yes) (dnp no)
+    (in_bom no) (on_board yes) (dnp yes)
     (property "Reference" "R16" (at 213.995 88.265 90)
       (effects (font (size 1.27 1.27)) (justify left))
@@
       (effects (font (size 1.27 1.27)) (justify left))
     )
-    (property "Value" "D" (at 84.582 104.0821 90)
+    (property "Value" "BAS16J" (at 84.582 104.0821 90)
       (effects (font (size 1.27 1.27)) (justify left))
     )
@@
   )
   (symbol (lib_id "Device:R_Small") (at 205.74 79.375 0) (unit 1)
-    (in_bom yes) (on_board yes) (dnp no)
+    (in_bom no) (on_board yes) (dnp yes)
     (property "Reference" "R15" (at 203.2 80.645 90)
       (effects (font (size 1.27 1.27)) (justify left))
@@
   )
   (symbol (lib_id "Device:R_Small") (at 213.36 83.185 270) (unit 1)
-    (in_bom yes) (on_board yes) (dnp no)
+    (in_bom no) (on_board yes) (dnp yes)
     (property "Reference" "R20" (at 213.995 80.645 90)
       (effects (font (size 1.27 1.27)) (justify left))
