File: gpio.kicad_sch (KiCad schematic)
At the start: 6 parts, among them J6 FPGA GPIO, U8 T20Q144xx

Commit message: reconnected fpgaGpio[0] from pin 36 -> 32 (REF_RES is *not* a GPIO!)
Connections:
- net FPGA_GPIO_0: no longer U8.36 (REF_RES)
- no-connect marks 0 -> 1
Changed lines of the file:
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@@
   (junction (at 77.47 129.54) (diameter 0) (color 0 0 0 0)
   )
+  (no_connect (at 171.45 135.89))
   (wire (pts (xy 222.25 73.66) (xy 225.425 73.66))
     (stroke (width 0) (type default))
@@
   )
   (wire (pts (xy 95.25 124.46) (xy 95.25 127))
-    (stroke (width 0) (type default))
-  )
-  (wire (pts (xy 168.402 135.89) (xy 171.45 135.89))
     (stroke (width 0) (type default))
   )
@@
       (effects (font (size 1.27 1.27)) (justify right) hide)
     )
-  )
-  (global_label "FPGA_GPIO_0" (shape bidirectional) (at 168.402 135.89 180) (fields_autoplaced)
-    (effects (font (size 1.27 1.27)) (justify right))
-    (property "Intersheetrefs" "${INTERSHEET_REFS}" (at 151.9683 135.89 0)
-      (effects (font (size 1.27 1.27)) (justify right) hide)
-    )
