File: tic-nic.kicad_sch (KiCad schematic)
At the start: 4 parts

Commit message: bumped version to 2.1
updated several values;

* added AC-coupling cap on RF_IN
Parts:
- H1, H2, H3, H4: Part FF-13-P3.5X5.5B -> FSR-1
Changed lines of the file:
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@@
       (effects (font (size 1.27 1.27)) hide)
     )
-    (property "Part" "FF-13-P3.5X5.5B" (at 191.77 132.08 0)
+    (property "Part" "FSR-1" (at 191.77 132.08 0)
       (effects (font (size 1.27 1.27)) hide)
     )
@@
       (effects (font (size 1.27 1.27)) hide)
     )
-    (property "Part" "FF-13-P3.5X5.5B" (at 171.45 132.08 0)
+    (property "Part" "FSR-1" (at 171.45 132.08 0)
       (effects (font (size 1.27 1.27)) hide)
     )
@@
       (effects (font (size 1.27 1.27)) hide)
     )
-    (property "Part" "FF-13-P3.5X5.5B" (at 201.295 132.08 0)
+    (property "Part" "FSR-1" (at 201.295 132.08 0)
       (effects (font (size 1.27 1.27)) hide)
     )
@@
       (effects (font (size 1.27 1.27)) hide)
     )
-    (property "Part" "FF-13-P3.5X5.5B" (at 182.245 132.08 0)
+    (property "Part" "FSR-1" (at 182.245 132.08 0)
       (effects (font (size 1.27 1.27)) hide)
     )

Commit message: more fab updates
Parts:
- H1, H2, H3, H4: value Foot FF-13-P3.5X5.5B -> Foot
Changed lines of the file:
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@@
       (effects (font (size 1.27 1.27)) (justify left))
     )
-    (property "Value" "Foot FF-13-P3.5X5.5B" (at 180.34 142.24 0)
+    (property "Value" "Foot" (at 190.246 137.16 0)
       (effects (font (size 1.27 1.27)) (justify left))
     )
@@
       (effects (font (size 1.27 1.27)) (justify left))
     )
-    (property "Value" "Foot FF-13-P3.5X5.5B" (at 160.02 136.525 0)
+    (property "Value" "Foot" (at 169.672 137.16 0)
       (effects (font (size 1.27 1.27)) (justify left))
     )
@@
       (effects (font (size 1.27 1.27)) (justify left))
     )
-    (property "Value" "Foot FF-13-P3.5X5.5B" (at 189.865 144.78 0)
+    (property "Value" "Foot" (at 199.39 137.16 0)
       (effects (font (size 1.27 1.27)) (justify left))
     )
@@
       (effects (font (size 1.27 1.27)) (justify left))
     )
-    (property "Value" "Foot FF-13-P3.5X5.5B" (at 170.815 139.7 0)
+    (property "Value" "Foot" (at 180.594 137.16 0)
       (effects (font (size 1.27 1.27)) (justify left))
     )
